File: v2-rf-frontend-board.sch (EAGLE design)
At the start: 155 parts, among them J3 ROCKETNET-CONNECTOR-16M, Q1 NTR4101P, T1 ALT4532, T2 ALT4532, U1 MAX2769, U11 LM3480IM4, U2 SAW_1.4X1.1, U3 LAN8710A-EZC, U4 7Q-16.368MBG-T, U5 XC2401, U6 SAW_1.4X1.1, X1 25 MHz, X3 BU-SMA-H

Commit message: Cleaned up part packages. Added exported partslist.
Parts:
- removed LED37: RGB, LED_RGB_PLCC6:LED_RGB_PLCC-6
- added LED2: BLUE, led:LEDCHIP-LED0603
- added LED3: GREEN, led:LEDCHIP-LED0603
- added LED4: RED, led:LEDCHIP-LED0603
- C1, C21, C23, C27, C28, C33, C36, C40: device rcl_custom:C-EU1206-B -> rcl:C-EUC1206
- C10, C26, C29, C30, C31, C32, C34, C35, C45, C46, C47, C48, C49, C50, C53: device rcl_custom:C-EU0402-B -> rcl:C-EUC0402
- C20, C51, C52: device rcl_custom:C-EU0603-B -> rcl:C-EUC0603
- C37, C38, C39, C41, C42, C44: device rcl_custom:C-EU0402-B-NOSILK -> rcl:C-EUC0402
- C43: device rcl3:C-EUC0402 -> rcl:C-EUC0402
- C59: device rcl_custom:C-EU0402-B-NOSILK -> rcl:C-EUC0603
- D1: value (none) -> 25V 1A
- LED1: value (none) -> GREEN
- R1, R12, R18, R3, R38, R39, R40: device rcl_custom:R-US_0402-B -> rcl:R-US_R0402
- R10, R11, R15, R20, R22, R23, R24, R25, R27, R28, R29, R42, R43, R44, R45, R46, R47, R48: device rcl_custom:R-US_0402-B-NOSILK -> rcl:R-US_R0402
- R16: device rcl:R-EU_R0402 -> rcl:R-US_R0402
- R6: value 500 -> 750; device rcl_custom:R-US_0402-B -> rcl:R-US_R0402
- U8: value STM32F4V_100PIN_GPSBOARD -> STM32F4V
- renumbered U$1 to U7, U$3 to U8, U$5 to J2, U11 to U9, USB_MICRO to J1, X3 to X2
Connections:
- net N$11: now also LED2.C; no longer LED37B.A
- net N$12: now also LED3.C; no longer LED37G.A
- net N$18: now also LED4.C; no longer LED37R.A
- net N$23: now also LED4.A; no longer LED37R.K
- net N$24: now also LED3.A; no longer LED37G.K
- net N$25: now also LED2.A; no longer LED37B.K

Commit message: Moved all parts onto the board in rough groupings.
Parts:
- removed TP22: TPTP06R, testpad:TPTP06R
Connections:
- net 3.3VA: no longer TP22.TP
Changed lines of the file:
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@@
 <part name="U$7" library="SparkFun-Aesthetics" deviceset="3.3VD" device=""/>
 <part name="U$10" library="SparkFun-Aesthetics" deviceset="3.3VD" device=""/>
-<part name="TP22" library="testpad" deviceset="TP" device="TP06R"/>
 <part name="TP26" library="testpad" deviceset="TP" device="TP06R"/>
 <part name="GND3" library="supply1" deviceset="GND" device="" value=""/>
@@
 <instance part="BAR_GND" gate="1" x="248.92" y="71.12"/>
 <instance part="U$32" gate="3.3VD" x="287.02" y="195.58"/>
-<instance part="TP22" gate="G$1" x="220.98" y="220.98" rot="MR0"/>
 <instance part="TP26" gate="G$1" x="153.67" y="101.6"/>
 <instance part="U1" gate="G$1" x="248.92" y="116.84" smashed="yes">
@@
 <wire x1="220.98" y1="218.44" x2="220.98" y2="215.9" width="0.1524" layer="91"/>
 <junction x="233.68" y="218.44"/>
-<pinref part="TP22" gate="G$1" pin="TP"/>
-<junction x="220.98" y="218.44"/>
 <pinref part="U1" gate="G$1" pin="VCCVCO"/>
 </segment>

Commit message: Laid the RF part. Four layers, AVDD and DVDD good where they meet.
Parts:
- L6, U2: value SAW_1.4X1.1 -> SAW
- renumbered U6 to L6
Connections:
- net N$13 renamed LNAOUT
- net N$21 renamed XTAL
- net N$22 renamed MIXIN
- net N$37 renamed LNA1CHIP
- removed net BAR_GND: C10.1, C17.2, C9.2, R4.2, R8.1, R9.1, X2G$1.GND, X2G2.GND, X2G3.GND, X2G4.GND
- removed net N$1: C22.1, L2.1, L6.RFIN, X2G$1.1
- new net LNA2CHIP: C22.2, U1.LNA2
- net GND: now also C10.1, C17.2, C9.2, R4.2, R8.1, R9.1, X2G$1.GND, X2G2.GND, X2G3.GND, X2G4.GND
- net LNA2: now also C22.1, L2.1, L6.RFIN, X2G$1.1; no longer C22.2, U1.LNA2
Changed lines of the file:
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@@
 <part name="U$7" library="SparkFun-Aesthetics" deviceset="3.3VD" device=""/>
 <part name="U$10" library="SparkFun-Aesthetics" deviceset="3.3VD" device=""/>
-<part name="TP26" library="testpad" deviceset="TP" device="TP06R"/>
+<part name="TP26" library="testpad" deviceset="TP" device="TP06R" value=""/>
 <part name="GND3" library="supply1" deviceset="GND" device="" value=""/>
 <part name="R42" library="rcl" deviceset="R-US_" device="R0402" value="4.7k"/>
@@
 <part name="U1" library="max2769" deviceset="MAX2769" device=""/>
 <part name="C11" library="rcl" deviceset="C-EU" device="C0402" value="DNP"/>
-<part name="U2" library="swift-nav" deviceset="SAW_1.4X1.1" device=""/>
+<part name="U2" library="swift-nav" deviceset="SAW_1.4X1.1" device="" value="SAW"/>
 <part name="BAR_GND1" library="supply" deviceset="GND_BAR" device="" value="GND"/>
 <part name="U4" library="swift-nav" deviceset="7Q-16.368MBG-T" device=""/>
@@
 <part name="DIG_GND19" library="supply" deviceset="GND_BAR" device="" value="GND"/>
 <part name="U5" library="swift-nav" deviceset="XC2401" device=""/>
-<part name="U6" library="swift-nav" deviceset="SAW_1.4X1.1" device=""/>
+<part name="L6" library="swift-nav" deviceset="SAW_1.4X1.1" device="" value="SAW"/>
 <part name="BAR_GND2" library="supply" deviceset="GND_BAR" device="" value="GND"/>
 <part name="C56" library="rcl" deviceset="C-EU" device="C0402" value="100pF"/>
@@
 <part name="BAR_GND3" library="supply" deviceset="GND_BAR" device="" value="GND"/>
 <part name="U$15" library="SparkFun-Aesthetics" deviceset="3.3VD" device=""/>
-<part name="TP23" library="testpad" deviceset="TP" device="TP06R"/>
+<part name="TP23" library="testpad" deviceset="TP" device="TP06R" value=""/>
 <part name="DIG_GND8" library="supply" deviceset="GND_BAR" device="" value="GND"/>
 <part name="R4" library="rcl" deviceset="R-US_" device="R0402" value="0"/>
@@
 <wire x1="167.64" y1="175.26" x2="162.56" y2="175.26" width="0.15" layer="91"/>
 <pinref part="DIG_GND24" gate="1" pin="BAR_GND"/>
+</segment>
+<segment>
+<pinref part="C10" gate="G$1" pin="1"/>
+<pinref part="DIG_GND17" gate="1" pin="BAR_GND"/>
+<wire x1="86.36" y1="99.06" x2="86.36" y2="100.33" width="0.1524" layer="91"/>
 </segment>
 </net>
@@
 </segment>
 </net>
-<net name="BAR_GND" class="0">
-<segment>
-<pinref part="C10" gate="G$1" pin="1"/>
-<pinref part="DIG_GND17" gate="1" pin="BAR_GND"/>
-<wire x1="86.36" y1="99.06" x2="86.36" y2="100.33" width="0.1524" layer="91"/>
-</segment>
-</net>
 </nets>
 </sheet>
@@
 <attribute name="VALUE" x="106.68" y="96.52" size="2.54" layer="96"/>
 </instance>
-<instance part="U6" gate="U1" x="69.85" y="99.06"/>
+<instance part="L6" gate="U1" x="69.85" y="99.06"/>
 <instance part="BAR_GND2" gate="1" x="71.12" y="86.36"/>
 <instance part="C56" gate="G$1" x="85.09" y="121.92"/>
@@
 </segment>
 <segment>
-<pinref part="U6" gate="U1" pin="GND1"/>
+<pinref part="L6" gate="U1" pin="GND1"/>
 <wire x1="66.04" y1="88.9" x2="71.12" y2="88.9" width="0.15" layer="91"/>
 <wire x1="71.12" y1="88.9" x2="76.2" y2="88.9" width="0.15" layer="91"/>
-<pinref part="U6" gate="U1" pin="GND2"/>
-<pinref part="U6" gate="U1" pin="GND3"/>
+<pinref part="L6" gate="U1" pin="GND2"/>
+<pinref part="L6" gate="U1" pin="GND3"/>
 <junction x="71.12" y="88.9"/>
 <pinref part="BAR_GND2" gate="1" pin="BAR_GND"/>
@@
 <pinref part="C58" gate="G$1" pin="2"/>
 <pinref part="DIG_GND28" gate="1" pin="BAR_GND"/>
+</segment>
+<segment>
+<pinref part="C9" gate="G$1" pin="2"/>
+<pinref part="DIG_GND9" gate="1" pin="BAR_GND"/>
+</segment>
+<segment>
+<pinref part="C17" gate="G$1" pin="2"/>
+<pinref part="DIG_GND15" gate="1" pin="BAR_GND"/>
+</segment>
+<segment>
+<pinref part="X2" gate="G$1" pin="GND"/>
+<pinref part="BAR_GND3" gate="1" pin="BAR_GND"/>
+<wire x1="45.72" y1="63.5" x2="45.72" y2="66.04" width="0.1524" layer="91"/>
+<junction x="45.72" y="71.12"/>
+<wire x1="45.72" y1="66.04" x2="45.72" y2="68.58" width="0.1524" layer="91"/>
+<wire x1="45.72" y1="68.58" x2="45.72" y2="71.12" width="0.1524" layer="91"/>
+<wire x1="45.72" y1="71.12" x2="45.72" y2="76.2" width="0.1524" layer="91"/>
+<junction x="45.72" y="68.58"/>
+<junction x="45.72" y="66.04"/>
+<pinref part="X2" gate="G3" pin="GND"/>
+<pinref part="X2" gate="G2" pin="GND"/>
+<pinref part="X2" gate="G4" pin="GND"/>
+</segment>
+<segment>
+<pinref part="DIG_GND8" gate="1" pin="BAR_GND"/>
+<pinref part="R4" gate="G$1" pin="2"/>
+<wire x1="210.82" y1="134.62" x2="210.82" y2="129.54" width="0.1524" layer="91"/>
+</segment>
+<segment>
+<pinref part="R8" gate="G$1" pin="1"/>
+<pinref part="DIG_GND30" gate="1" pin="BAR_GND"/>
+<wire x1="137.16" y1="124.46" x2="139.7" y2="124.46" width="0.1524" layer="91"/>
+<pinref part="R9" gate="G$1" pin="1"/>
+<wire x1="139.7" y1="124.46" x2="142.24" y2="124.46" width="0.1524" layer="91"/>
+<junction x="139.7" y="124.46"/>
 </segment>
 </net>
@@
 </segment>
 </net>
-<net name="LNA2" class="0">
+<net name="LNA2CHIP" class="0">
 <segment>
 <wire x1="223.52" y1="93.98" x2="213.36" y2="93.98" width="0.1524" layer="91"/>
@@
 </segment>
 </net>
-<net name="N$21" class="0">
+<net name="XTAL" class="0">
 <segment>
 <pinref part="U1" gate="G$1" pin="XTAL"/>
@@
 </segment>
 </net>
-<net name="N$13" class="0">
+<net name="LNAOUT" class="0">
 <segment>
 <pinref part="U2" gate="U1" pin="RFIN"/>
@@
 </segment>
 </net>
-<net name="N$22" class="0">
+<net name="MIXIN" class="0">
 <segment>
 <pinref part="U2" gate="U1" pin="RFOUT"/>
@@
 <net name="N$3" class="0">
 <segment>
-<pinref part="U6" gate="U1" pin="RFOUT"/>
+<pinref part="L6" gate="U1" pin="RFOUT"/>
 <pinref part="U5" gate="U1" pin="RFIN"/>
 <wire x1="85.09" y1="104.14" x2="86.36" y2="104.14" width="0.15" layer="91"/>
 </segment>
 </net>
-<net name="N$37" class="0">
+<net name="LNA1CHIP" class="0">
 <segment>
 <pinref part="C19" gate="G$1" pin="1"/>
@@
 </segment>
 </net>
-<net name="BAR_GND" class="0">
-<segment>
-<pinref part="C9" gate="G$1" pin="2"/>
-<pinref part="DIG_GND9" gate="1" pin="BAR_GND"/>
-</segment>
-<segment>
-<pinref part="C17" gate="G$1" pin="2"/>
-<pinref part="DIG_GND15" gate="1" pin="BAR_GND"/>
-</segment>
-<segment>
-<pinref part="X2" gate="G$1" pin="GND"/>
-<pinref part="BAR_GND3" gate="1" pin="BAR_GND"/>
-<wire x1="45.72" y1="63.5" x2="45.72" y2="66.04" width="0.1524" layer="91"/>
-<junction x="45.72" y="71.12"/>
-<wire x1="45.72" y1="66.04" x2="45.72" y2="68.58" width="0.1524" layer="91"/>
-<wire x1="45.72" y1="68.58" x2="45.72" y2="71.12" width="0.1524" layer="91"/>
-<wire x1="45.72" y1="71.12" x2="45.72" y2="76.2" width="0.1524" layer="91"/>
-<junction x="45.72" y="68.58"/>
-<junction x="45.72" y="66.04"/>
-<pinref part="X2" gate="G3" pin="GND"/>
-<pinref part="X2" gate="G2" pin="GND"/>
-<pinref part="X2" gate="G4" pin="GND"/>
-</segment>
-<segment>
-<pinref part="DIG_GND8" gate="1" pin="BAR_GND"/>
-<pinref part="R4" gate="G$1" pin="2"/>
-<wire x1="210.82" y1="134.62" x2="210.82" y2="129.54" width="0.1524" layer="91"/>
-</segment>
-<segment>
-<pinref part="R8" gate="G$1" pin="1"/>
-<pinref part="DIG_GND30" gate="1" pin="BAR_GND"/>
-<wire x1="137.16" y1="124.46" x2="139.7" y2="124.46" width="0.1524" layer="91"/>
-<pinref part="R9" gate="G$1" pin="1"/>
-<wire x1="139.7" y1="124.46" x2="142.24" y2="124.46" width="0.1524" layer="91"/>
-<junction x="139.7" y="124.46"/>
-</segment>
-</net>
 <net name="ANTFLAG" class="0">
 <segment>
@@
 </segment>
 </net>
-<net name="N$1" class="0">
+<net name="LNA2" class="0">
 <segment>
 <pinref part="C22" gate="G$1" pin="1"/>
@@
 <wire x1="129.54" y1="81.28" x2="129.54" y2="78.74" width="0.1524" layer="91"/>
 <wire x1="129.54" y1="78.74" x2="193.04" y2="78.74" width="0.1524" layer="91"/>
-<pinref part="U6" gate="U1" pin="RFIN"/>
+<pinref part="L6" gate="U1" pin="RFIN"/>
 <wire x1="57.15" y1="104.14" x2="55.88" y2="104.14" width="0.15" layer="91"/>
 <wire x1="55.88" y1="104.14" x2="55.88" y2="78.74" width="0.15" layer="91"/>

Commit message: Testpoint breakouts matched to stm32. Other peripheral components grouped better.
Connections:
- net N$23 renamed LED4
- net N$24 renamed LED3
- net N$25 renamed LED2
Changed lines of the file:
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@@
 <part name="DIG_GND10" library="supply" deviceset="GND_BAR" device="" value="GND"/>
 <part name="R18" library="rcl" deviceset="R-US_" device="R0402" value="10k"/>
-<part name="TP2" library="testpad" deviceset="TP" device="TP06R"/>
+<part name="TP2" library="testpad" deviceset="TP" device="TP06R" value=""/>
 <part name="R38" library="rcl" deviceset="R-US_" device="R0402" value="750"/>
 <part name="R39" library="rcl" deviceset="R-US_" device="R0402" value="750"/>
@@
 <part name="U$17" library="SparkFun-Aesthetics" deviceset="3.3VD" device=""/>
 <part name="3.3VD1" library="SparkFun-Aesthetics" deviceset="3.3VD" device=""/>
-<part name="TP1" library="testpad" deviceset="TP" device="TP06R"/>
+<part name="TP1" library="testpad" deviceset="TP" device="TP06R" value=""/>
 <part name="TP4" library="Tova" deviceset="TEST-POINT" device=""/>
 <part name="TP5" library="Tova" deviceset="TEST-POINT" device=""/>
@@
 </segment>
 </net>
-<net name="N$23" class="0">
+<net name="LED4" class="0">
 <segment>
 <pinref part="U8" gate="G$1" pin="PD14"/>
@@
 </segment>
 </net>
-<net name="N$24" class="0">
+<net name="LED3" class="0">
 <segment>
 <pinref part="U8" gate="G$1" pin="PD13"/>
@@
 </segment>
 </net>
-<net name="N$25" class="0">
+<net name="LED2" class="0">
 <segment>
 <pinref part="U8" gate="G$1" pin="PD11"/>

Commit message: Took a first try at Ethernet section. Tight but a little worried about trace widths.
Parts:
- R20: value 0R(board_mounted) -> 0R
Connections:
- net N$59 renamed VDDA
Changed lines of the file:
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@@
 <setting verticaltext="up"/>
 </settings>
-<grid distance="1.27" unitdist="mm" unit="mm" style="lines" multiple="2" display="no" altdistance="0.01" altunitdist="inch" altunit="inch"/>
+<grid distance="0.0125" unitdist="inch" unit="inch" style="dots" multiple="2" display="yes" altdistance="0.01" altunitdist="inch" altunit="inch"/>
 <layers>
 <layer number="1" name="Top" color="4" fill="1" visible="no" active="no"/>
@@
 <part name="C28" library="rcl" deviceset="C-EU" device="C1206" value="22uF/6.3V"/>
 <part name="GND20" library="supply1" deviceset="GND" device="" value=""/>
-<part name="R20" library="rcl" deviceset="R-US_" device="R0402" value="0R(board_mounted)"/>
+<part name="R20" library="rcl" deviceset="R-US_" device="R0402" value="0R"/>
 <part name="GND131" library="supply1" deviceset="GND" device="" value=""/>
 <part name="C35" library="rcl" deviceset="C-EU" device="C0402" value="100nF"/>
@@
 </segment>
 </net>
-<net name="N$59" class="0">
+<net name="VDDA" class="0">
 <segment>
 <wire x1="193.04" y1="152.4" x2="185.42" y2="152.4" width="0.1524" layer="91"/>

Commit message: Ethernet basically done.
Connections:
- net N$34 renamed PE0
Changed lines of the file:
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@@
 </segment>
 </net>
-<net name="N$34" class="0">
+<net name="PE0" class="0">
 <segment>
 <pinref part="Q1" gate="G$1" pin="G"/>

Commit message: Finished board layout. Removed some test pads. Needs review.
Parts:
- removed TP26, TP36, TP37, TP38, TP42: TPTP06R, testpad:TPTP06R
Connections:
- net N$17 renamed VFB2
- net +5V: no longer TP37.TP
- net 3.3VA: no longer TP42.TP
- net 3.3VD: no longer TP38.TP
- net ANTBIAS: no longer TP26.TP
- net GND: no longer TP36.TP
Changed lines of the file:
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@@
 <part name="U$7" library="SparkFun-Aesthetics" deviceset="3.3VD" device=""/>
 <part name="U$10" library="SparkFun-Aesthetics" deviceset="3.3VD" device=""/>
-<part name="TP26" library="testpad" deviceset="TP" device="TP06R" value=""/>
 <part name="GND3" library="supply1" deviceset="GND" device="" value=""/>
 <part name="R42" library="rcl" deviceset="R-US_" device="R0402" value="4.7k"/>
@@
 <part name="C1" library="rcl" deviceset="C-EU" device="C1206" value="10u"/>
 <part name="C21" library="rcl" deviceset="C-EU" device="C1206" value="10u"/>
-<part name="TP16" library="testpad" deviceset="TP" device="TP06R"/>
-<part name="TP17" library="testpad" deviceset="TP" device="TP06R"/>
+<part name="TP16" library="testpad" deviceset="TP" device="TP06R" value=""/>
+<part name="TP17" library="testpad" deviceset="TP" device="TP06R" value=""/>
 <part name="R1" library="rcl" deviceset="R-US_" device="R0402" value="11.5k"/>
 <part name="GND2" library="SparkFun-Aesthetics" deviceset="GND" device=""/>
-<part name="TP18" library="testpad" deviceset="TP" device="TP06R"/>
+<part name="TP18" library="testpad" deviceset="TP" device="TP06R" value=""/>
 <part name="C26" library="rcl" deviceset="C-EU" device="C0402" value="22p"/>
 <part name="C33" library="rcl" deviceset="C-EU" device="C1206" value="100u"/>
@@
 <part name="D1" library="SparkFun-DiscreteSemi" deviceset="DIODE" device="SMA-ALT" value="25V 1A"/>
 <part name="VIN" library="dp_devices" deviceset="SUPPLY_+5V" device="" value="VIN"/>
-<part name="TP34" library="testpad" deviceset="TP" device="TP06R"/>
-<part name="TP35" library="testpad" deviceset="TP" device="TP06R"/>
-<part name="TP36" library="testpad" deviceset="TP" device="TP06R"/>
-<part name="TP37" library="testpad" deviceset="TP" device="TP06R"/>
-<part name="TP38" library="testpad" deviceset="TP" device="TP06R"/>
+<part name="TP34" library="testpad" deviceset="TP" device="TP06R" value=""/>
+<part name="TP35" library="testpad" deviceset="TP" device="TP06R" value=""/>
 <part name="C42" library="rcl" deviceset="C-EU" device="C0402" value="10n"/>
 <part name="C43" library="rcl" deviceset="C-EU" device="C0402" value="10n"/>
@@
 <part name="GND13" library="SparkFun-Aesthetics" deviceset="GND" device=""/>
 <part name="GND14" library="SparkFun-Aesthetics" deviceset="GND" device=""/>
-<part name="GND15" library="SparkFun-Aesthetics" deviceset="GND" device=""/>
 <part name="GND16" library="SparkFun-Aesthetics" deviceset="GND" device=""/>
-<part name="TP27" library="testpad" deviceset="TP" device="TP06R"/>
+<part name="TP27" library="testpad" deviceset="TP" device="TP06R" value=""/>
 <part name="GND17" library="SparkFun-Aesthetics" deviceset="GND" device=""/>
 <part name="GND18" library="SparkFun-Aesthetics" deviceset="GND" device=""/>
@@
 <part name="GND21" library="SparkFun-Aesthetics" deviceset="GND" device=""/>
 <part name="GND22" library="SparkFun-Aesthetics" deviceset="GND" device=""/>
-<part name="TP42" library="testpad" deviceset="TP" device="TP06R"/>
 <part name="BAR_GND3" library="supply" deviceset="GND_BAR" device="" value="GND"/>
 <part name="U$15" library="SparkFun-Aesthetics" deviceset="3.3VD" device=""/>
@@
 <instance part="BAR_GND" gate="1" x="248.92" y="71.12"/>
 <instance part="U$32" gate="3.3VD" x="287.02" y="195.58"/>
-<instance part="TP26" gate="G$1" x="153.67" y="101.6"/>
 <instance part="U1" gate="G$1" x="248.92" y="116.84" smashed="yes">
 <attribute name="NAME" x="228.6" y="76.2" size="2.54" layer="95" font="vector"/>
@@
 <junction x="153.67" y="99.06"/>
 <junction x="143.51" y="99.06"/>
-<pinref part="TP26" gate="G$1" pin="TP"/>
 <pinref part="C54" gate="G$1" pin="1"/>
 <wire x1="163.83" y1="99.06" x2="163.83" y2="96.52" width="0.1524" layer="91"/>
@@
 <instance part="C40" gate="G$1" x="187.96" y="134.62"/>
 <instance part="C41" gate="G$1" x="162.56" y="127" smashed="yes">
-<attribute name="NAME" x="167.259" y="127.254" size="1.778" layer="95" rot="R90"/>
-<attribute name="VALUE" x="166.751" y="125.476" size="1.778" layer="96" rot="R270"/>
+<attribute name="NAME" x="163.449" y="127.381" size="1.778" layer="95"/>
+<attribute name="VALUE" x="163.1315" y="122.301" size="1.778" layer="96"/>
 </instance>
 <instance part="U$4" gate="3.3VD" x="187.96" y="142.24"/>
 <instance part="TP34" gate="G$1" x="167.64" y="177.8"/>
 <instance part="TP35" gate="G$1" x="167.64" y="149.86"/>
-<instance part="TP36" gate="G$1" x="73.66" y="137.16"/>
-<instance part="TP37" gate="G$1" x="180.34" y="168.91"/>
-<instance part="TP38" gate="G$1" x="180.34" y="140.97"/>
 <instance part="C42" gate="G$1" x="276.86" y="149.86" smashed="yes">
 <attribute name="NAME" x="278.384" y="150.241" size="1.778" layer="95"/>
@@
 <instance part="GND13" gate="1" x="101.6" y="124.46"/>
 <instance part="GND14" gate="1" x="96.52" y="127"/>
-<instance part="GND15" gate="1" x="73.66" y="129.54"/>
 <instance part="GND16" gate="1" x="76.2" y="154.94"/>
 <instance part="TP27" gate="G$1" x="91.44" y="160.02"/>
@@
 <instance part="GND21" gate="1" x="162.56" y="148.59"/>
 <instance part="GND22" gate="1" x="175.26" y="149.86"/>
-<instance part="TP42" gate="G$1" x="320.04" y="160.02"/>
 </instances>
 <busses>
@@
 <pinref part="C60" gate="G$1" pin="2"/>
 <wire x1="269.24" y1="142.24" x2="269.24" y2="144.78" width="0.1524" layer="91"/>
-</segment>
-<segment>
-<pinref part="TP36" gate="G$1" pin="TP"/>
-<pinref part="GND15" gate="1" pin="GND"/>
-<wire x1="73.66" y1="132.08" x2="73.66" y2="134.62" width="0.1524" layer="91"/>
 </segment>
 <segment>
@@
 <wire x1="167.64" y1="166.37" x2="180.34" y2="166.37" width="0.15" layer="91"/>
 <junction x="167.64" y="166.37"/>
-<pinref part="TP37" gate="G$1" pin="TP"/>
 <wire x1="180.34" y1="166.37" x2="187.96" y2="166.37" width="0.1524" layer="91"/>
-<junction x="180.34" y="166.37"/>
 <junction x="187.96" y="166.37"/>
 </segment>
@@
 <pinref part="C59" gate="G$1" pin="1"/>
 <wire x1="320.04" y1="154.94" x2="320.04" y2="152.4" width="0.1524" layer="91"/>
-<pinref part="TP42" gate="G$1" pin="TP"/>
-<wire x1="320.04" y1="157.48" x2="320.04" y2="154.94" width="0.1524" layer="91"/>
-<junction x="320.04" y="154.94"/>
 </segment>
 </net>
@@
 <wire x1="167.64" y1="138.43" x2="180.34" y2="138.43" width="0.15" layer="91"/>
 <junction x="167.64" y="138.43"/>
-<pinref part="TP38" gate="G$1" pin="TP"/>
 <pinref part="U7" gate="G$1" pin="VOUT2"/>
 <wire x1="180.34" y1="138.43" x2="187.96" y2="138.43" width="0.1524" layer="91"/>
-<junction x="180.34" y="138.43"/>
 <junction x="187.96" y="138.43"/>
 </segment>
@@
 </segment>
 </net>
-<net name="N$17" class="0">
+<net name="VFB2" class="0">
 <segment>
 <pinref part="TP35" gate="G$1" pin="TP"/>

Commit message: BOM done. Board done. All parts reviewed. Ready for review & ship.
Parts:
- R38, R39, R6: value 750 -> 68
- R40: value 300 -> 27
Changed lines of the file:
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@@
 <setting verticaltext="up"/>
 </settings>
-<grid distance="0.0125" unitdist="inch" unit="inch" style="dots" multiple="2" display="yes" altdistance="0.01" altunitdist="inch" altunit="inch"/>
+<grid distance="0.0125" unitdist="inch" unit="inch" style="dots" multiple="2" display="yes" altdistance="0.025" altunitdist="inch" altunit="inch"/>
 <layers>
 <layer number="1" name="Top" color="4" fill="1" visible="no" active="no"/>
@@
 <part name="R18" library="rcl" deviceset="R-US_" device="R0402" value="10k"/>
 <part name="TP2" library="testpad" deviceset="TP" device="TP06R" value=""/>
-<part name="R38" library="rcl" deviceset="R-US_" device="R0402" value="750"/>
-<part name="R39" library="rcl" deviceset="R-US_" device="R0402" value="750"/>
-<part name="R40" library="rcl" deviceset="R-US_" device="R0402" value="300"/>
+<part name="R38" library="rcl" deviceset="R-US_" device="R0402" value="68"/>
+<part name="R39" library="rcl" deviceset="R-US_" device="R0402" value="68"/>
+<part name="R40" library="rcl" deviceset="R-US_" device="R0402" value="27"/>
 <part name="3.3VD3" library="SparkFun-Aesthetics" deviceset="3.3VD" device=""/>
 <part name="U$7" library="SparkFun-Aesthetics" deviceset="3.3VD" device=""/>
@@
 <part name="C43" library="rcl" deviceset="C-EU" device="C0402" value="10n"/>
 <part name="LED1" library="led" deviceset="LED" device="CHIP-LED0603" value="GREEN"/>
-<part name="R6" library="rcl" deviceset="R-US_" device="R0402" value="750"/>
+<part name="R6" library="rcl" deviceset="R-US_" device="R0402" value="68"/>
 <part name="R10" library="rcl" deviceset="R-US_" device="R0402" value="75"/>
 <part name="R11" library="rcl" deviceset="R-US_" device="R0402" value="75"/>
