File: v2-rf-frontend-board.sch (EAGLE design)
At the start: 151 parts, among them J1 USB_MICROB, J2 MICROSD, J3 ROCKETNET-CONNECTOR-16M, Q1 NTR4101P, T1 ALT4532, T2 ALT4532, U1 MAX2769, U2 SAW, U3 LAN8710A-EZC, U4 7Q-16.368MBG-T, U5 XC2401, U7 LT4619_REDUCED, U8 STM32F4V, U9 LM3480IM4, X1 25 MHz, X2 BU-SMA-H

Commit message: Fixes as per design review. microUSB footprint needs help but symbol and signals OK. RF side placement adjusted but impedance 50 ohms wants 14mm wide trace. help.
Parts:
- removed J2: MICROSD, adafruit:MICROSD
- removed JP1: AUX HDR, SparkFun-Connectors:M04LOCK
- added R7: 100k, rcl:R-US_R0402
- added SD: CON_HIROSE_DM3D(MICROSD), con-usd-hirose-dm3-gpsboard:CON_HIROSE_DM3D(MICROSD)
- added TP22, TP26, TP32, TP33: TEST-POINT, Tova:TEST-POINT
- C33, C40: device rcl:C-EUC1206 -> SparkFun-Passives:CAP_POL6032
- J1: device SparkFun:USB_MICROB_PLUG-PTH -> con-hirose-microusb:ZX62D-B-5P8
- JTAG1: value (none) -> M05X2PTH; device microbuilder:JTAG-CORTEXM3 -> SparkFun-Connectors:M05X2PTH
- U9: value LM3480IM4 -> LM3480IM3
Connections:
- removed net N$4: TP27.TP, U7.PGOOD
- removed net N$46: J3.AUX1, JP1.1
- removed net N$47: J3.AUX2, JP1.2
- removed net N$48: J3.AUX3, JP1.3
- removed net N$50: J3.AUX4, JP1.4
- new net AUX1: J3.AUX1, TP22.1
- new net AUX2: J3.AUX2, TP26.1
- new net AUX3: J3.AUX3, TP32.1
- new net AUX4: J3.AUX4, TP33.1
- new net PGOOD: R7.1, TP27.TP, U7.PGOOD
- net +5V: now also C33.+; no longer C33.1
- net 3.3VD: now also C40.+; no longer C40.1
- net GND: now also C33.-, C40.-, J1.GND1, J1.GND2, J1.GND3, J1.GND4, J1.GND5, J1.GND6, SD$.6, SDCD.0, SDCD.1, SDG1.PAD, SDG2.PAD, SDG3.PAD, SDG4.PAD, U8.PA4; no longer C33.2, C40.2, J2.CARD_DETECT, J2.CARD_DETECT1, J2.GND, J2.GND1, J2.VSS
- net N$6: now also R7.2
- net SDIO_CLK: now also SD$.5; no longer J2.SCLK
- net SDIO_CMD: now also SD$.3; no longer J2.DATA_IN
- net SDIO_D0: now also SD$.7; no longer J2.DATA_OUT
- net SDIO_D1: now also SD$.8; no longer J2.DAT1
- net SDIO_D2: now also SD$.1; no longer J2.DAT2
- net SDIO_D3: now also SD$.2; no longer J2.CS
- net VDD: now also SD$.4; no longer J2.VDD
Other:
- note added: "3-wire faux-SPI serial config bus"
- note added: "4.5 - 26 Vin"
- note added: "CONFIG 2: EXT LNA = DNP L6, U5, C57, C56"
- note added: "CONFIG 3: EXT POWERED LNA = DNP L6, U5, L2, C57, C56, C24, C25, C54, C55"
- note added: "MICROSD"
- note added: "SEE CONFIG 1, CONFIG 3"
- note added: "SEE CONFIG 2, CONFIG 3"
- note added: "actual-SPI I/Q data out"
- note removed: "3-wire serial config register"
- note removed: "5 - 20 Vin"
- note removed: "CONFIG 2: EXT LNA = DNP U5,U6"
- note removed: "CONFIG 3: EXT POWERED LNA = DNP L6,L2"
- note removed: "TODO: CURRENT FOR MAX2769?"
- moved on the sheet: C1, C10, C11, C2, C20, C21, C26, C38, C39, C41, C42, C43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

Commit message: Updated microUSB symbol and library. Package not finalized.
Parts:
- removed J1: USB_MICROB, con-hirose-microusb:ZX62D-B-5P8
- added C62: 100n, rcl:C-EUC0402
- added U$1: ZX62D-B-5P8, con-hirose-microusb:ZX62D-B-5P8
Connections:
- new net SHLD: C62.2, U$1.SHLD@1, U$1.SHLD@2, U$1.SHLD@3, U$1.SHLD@4
- net GND: now also C62.1, U$1.GND; no longer J1.GND, J1.GND1, J1.GND2, J1.GND3, J1.GND4, J1.GND5, J1.GND6
- net OTG_FS_DM: now also U$1.D-; no longer J1.D-
- net OTG_FS_DP: now also U$1.D+; no longer J1.D+
- net OTG_FS_VBUS: now also U$1.VCC; no longer J1.VCC
Other:
- moved on the sheet: R12

Commit message: Major changes to to PWR and GPS sheets. No change to board layout yet, waiting on feedback.
Parts:
- removed C57: 0.047uF, rcl:C-EUC0402
- removed TP16, TP17, TP27, TP34, TP35: TPTP06R, testpad:TPTP06R
- removed U9: LM3480IM3, SparkFun-PowerIC:LM3480IM4
- added L5: 9.1nH, SparkFun-Passives:INDUCTOR0402
- added R13: 470, rcl:R-US_R0402
- added U10: LMZ12001, SparkFun-PowerIC:LMZ12001
- added U6: MAX8510EXK29+T, SparkFun-PowerIC:V_REG_LDOSMD2
- C1: value 10u -> 1uF; device rcl:C-EUC1206 -> rcl:C-EUC0603
- C21: value 10u -> 220nF; device rcl:C-EUC1206 -> rcl:C-EUC0402
- C24, C54: value 0.47uF -> 100pF
- C26: value 22p -> 220nF
- C33: value 100u -> 10uF; device SparkFun-Passives:CAP_POL6032 -> rcl:C-EUC0805
- C38: value 100n -> 100u; device rcl:C-EUC0402 -> SparkFun-Passives:CAP_POL6032
- C39: value 22p -> 1uF; device rcl:C-EUC0402 -> rcl:C-EUC0603
- C40: value 100u -> 1uF; device SparkFun-Passives:CAP_POL6032 -> rcl:C-EUC0603
- C41: value 100n -> 1uF; device rcl:C-EUC0402 -> rcl:C-EUC0603
- C42, C43: value 10n -> 1uF; device rcl:C-EUC0402 -> rcl:C-EUC0603
- C56: value 100pF -> 10nF
- C59, C60: value 1u -> 1uF
- L2: value 3.3nH -> 6.2nH
- R1: value 11.5k -> 10k
- R3: value 19.1k -> 3.3k
- R7: value 100k -> 240k
- U7: value LT4619_REDUCED -> MAX8510EXK29+T; device LT4619:LT4619_REDUCED -> SparkFun-PowerIC:V_REG_LDOSMD2
Connections:
- net LNA2CHIP renamed N$1
- removed net +5V: C26.2, C33.+, C42.1, C60.1, U7.VOUT1, U9.IN
- removed net 3.3VA: C12.1, C13.1, C15.1, C16.1, C18.1, C43.1, C5.1, C56.1, C57.1, C59.1, C6.1, C8.1, U1.VCCCP, U1.VCCIF, U1.VCCRF, U1.VCCVCO, U5.VDD, U9.OUT
- removed net ANTBIAS: C24.1, C25.1, C54.1, C55.1, L2.2, U1.ANTBIAS
- removed net LNA1: C19.2, U5.RFOUT
- removed net LNA1CHIP: C19.1, U1.LNA1
- removed net PGOOD: R7.1, TP27.TP, U7.PGOOD
- removed net VFB2: C39.1, R3.1, TP35.TP, U7.VFB2
- new net 2.85VA: C12.1, C13.1, C15.1, C16.1, C18.1, C42.1, C43.2, C5.1, C6.1, C8.1, U1.VCCCP, U1.VCCIF, U1.VCCRF, U1.VCCVCO, U7.OUT
- new net 2.85VD: C14.1, C17.1, C58.1, C59.1, C60.2, C7.1, C9.1, R5.2, U1.VCCADC, U1.VCCD, U4.VDD, U6.OUT
- new net N$10: R7.2, U10.RON
- new net N$13: C43.1, U7.BP
- new net N$17: C19.1, C22.1, C24.2, C25.2
- new net N$21: C54.1, C55.1, L6.RFOUT
- new net N$22: C55.2, L2.1, L5.2
- new net N$23: R13.1, U1.ANTBIAS
- new net N$4: C56.1, R13.2, U5.VDD
- net 3.3VD: now also C26.1, C38.+, C39.1, C40.1, C41.1, R1.2, U10.VOUT, U6.EN, U6.IN, U7.EN, U7.IN; no longer C14.1, C17.1, C39.2, C40.+, C58.1, C7.1, C9.1, R5.2, U1.VCCADC, U1.VCCD, U4.VDD, U7.VOUT2
- net GND: now also C33.2, C38.-, C39.2, C40.2, L5.1, R3.1, U10.EP, U10.GND, U6.GND, U7.GND; no longer C24.2, C25.2, C33.-, C38.2, C40.-, C43.2, C54.2, C55.2, C57.2, C60.2, R1.2, R3.2, U7.MODE/PLLIN, U7.PGND, U7.SGND, U9.GND
- net LNA2: no longer C22.1, L2.1
- net N$14: now also L2.2, U5.RFIN; no longer C41.1, U7.TK/SS2
- net N$16: now also C60.1, U6.BP; no longer C38.1, U7.TK/SS1
- net N$2: now also C19.2, U1.LNA1; no longer TP17.TP, U7.SW1
- net N$3: now also C25.1, U5.RFOUT; no longer L6.RFOUT, U5.RFIN
- net N$5: now also C24.1, C54.2; no longer C26.1, R1.1, TP34.TP, U7.VFB1
- net N$6: now also C21.1, U10.SS; no longer R7.2, U7.FREQ/PLL/FLTR, U7.INTVCC
- net N$7: now also C26.2, R1.1, R3.2, U10.FB; no longer TP16.TP, U7.SW2
- net VIN: now also C33.1, R7.1, U10.VIN; no longer C21.1, U7.EXTVCC, U7.VIN
Other:
- note added: "2.85V Analog and Digital to MAX2769 GPS Receiver"
- note added: "CHOICE #1: - POPULATE C19 FOR LNA1 - POPULATE C22 FOR LNA2 CHOICE #2: - POPULATE C55, U5, R13, C56, L2, L5 - POPULATE C54"
- note added: "Vsys to 3.3V"
- note added: "actual-SPI I/Q data in"
- note removed: "CONFIG 1: CPA ONLY = DNP L2"
- note removed: "CONFIG 2: EXT LNA = DNP L6, U5, C57, C56"
- note removed: "CONFIG 3: EXT POWERED LNA = DNP L6, U5, L2, C57, C56, C24, C25, C54, C55"
- note removed: "Low noise 3.3V for MAX2769"
- note removed: "SEE CONFIG 1, CONFIG 3"
- note removed: "SEE CONFIG 2, CONFIG 3"
- note removed: "Vsys to 3.3 V and 5.0 V SPS"
- note removed: "actual-SPI I/Q data out"
- moved on the sheet: C1, C11, C12, C13, C14, C15, C16, C17, C18, C19, C2, C21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

Commit message: Made a capacitor options footprint and symbol for the 'do not populate' choice capacitor hack.
Parts:
- removed C25, C54, C55: 100pF, rcl:C-EUC0402
- C19, C22, C24: device rcl:C-EUC0402 -> wicker:CAP-OPTION
Connections:
- removed net N$1: C22.2, U1.LNA2
- new net N$25: C19.2, C22.2
- net N$17: now also C19.3, U1.LNA2; no longer C19.1, C22.1, C24.2, C25.2
- net N$2: now also C19.1; no longer C19.2
- net N$21: now also C24.2; no longer C54.1, C55.1
- net N$22: now also C24.3; no longer C55.2
- net N$3: now also C22.1; no longer C25.1
- net N$5: now also C22.3; no longer C54.2
Other:
- moved on the sheet: C56, L2, L5, L6, R13, U5, X2, X2G2, X2G3, X2G4

Commit message: Laid out new LNA1, LNA2, and ANTBIAS sections. Layout done. Passes ERC, DRC. Ready for design review.
Connections:
- net N$23 renamed ANTBIAS
Changed lines of the file:
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@@
 </segment>
 </net>
-<net name="N$23" class="0">
+<net name="ANTBIAS" class="0">
 <segment>
 <pinref part="R13" gate="G$1" pin="1"/>

Commit message: ERC and DRC passed. Added ground vias everywhere. Fixed 0.1in breakout header by making new symbol, should be able to drop in a proper header if we want. Changed order of IO pins on sch to make sense and swapped four of the IO pin signals for ease of routing. Fixed tNames on board so labels align with the right parts. Added voltage to caps in sch. Tidied up. Added board title on tnames layer. Andrew is free to fix voltage 3.3vd, 2.85va, 2.86vd with polygons for OCD & beauty reasons if his heart so desires.
Parts:
- removed TP10, TP11, TP12, TP13, TP14, TP15, TP19, TP20, TP21, TP24, TP25, TP28, TP29, TP3, TP30, TP31, TP4, TP5, TP6, TP7, TP8, TP9: TEST-POINT, Tova:TEST-POINT
- removed U$1: ZX62D-B-5P8, con-hirose-microusb:ZX62D-B-5P8
- added JP1: BREAKOUT, wicker:HEADER-11X02
- added USB: ZX62D-B-5P8, con-hirose-microusb:ZX62D-B-5P8
- C1: value 1uF -> 1uF 50V; device rcl:C-EUC0603 -> rcl_custom:C-EU0603-C-NOSILK
- C10, C2, C62: value 100n -> 100n 10V; device rcl:C-EUC0402 -> rcl_custom:C-EU0402-C-NOSILK
- C11: device rcl:C-EUC0402 -> rcl_custom:C-EU0402-C-NOSILK
- C12, C14, C16, C17, C6, C8: value 100pF -> 100pF 10V; device rcl:C-EUC0402 -> rcl_custom:C-EU0402-C-NOSILK
- C13, C15, C18, C31, C32, C34, C35, C37, C45, C46, C47, C48, C49, C5, C50, C53, C7, C9: value 100nF -> 100nF 10V; device rcl:C-EUC0402 -> rcl_custom:C-EU0402-C-NOSILK
- C19, C22, C24: value 100pF -> 100pF 10V
- C20: value 2.2u -> 2.2u 10V; device rcl:C-EUC0603 -> rcl_custom:C-EU0603-C-NOSILK
- C21, C26: value 220nF -> 220nF 10V; device rcl:C-EUC0402 -> rcl_custom:C-EU0402-C-NOSILK
- C23, C27, C28, C36: device rcl:C-EUC1206 -> rcl_custom:C-EU1206-C
- C29, C30: value 16pF -> 18pF 10V; device rcl:C-EUC0402 -> rcl_custom:C-EU0402-C-NOSILK
- C3: value 27pF -> 27pF 10V; device rcl:C-EUC0402 -> rcl_custom:C-EU0402-C-NOSILK
- C33: value 10uF -> 10uF 50V; device rcl:C-EUC0805 -> rcl_custom:C-EU0805-C-NOSILK
- C38: value 100u -> 100u 10V
- C39, C40, C41, C42, C43, C59, C60: value 1uF -> 1uF 10V; device rcl:C-EUC0603 -> rcl_custom:C-EU0603-C-NOSILK
- C4: value 470pF -> 470pF 10V; device rcl:C-EUC0402 -> rcl_custom:C-EU0402-C-NOSILK
- C44: value 1nF -> 1nF 10V; device rcl:C-EUC0402 -> rcl_custom:C-EU0402-C-NOSILK
- C51, C52: value 2.2uF -> 2.2uF 10V; device rcl:C-EUC0603 -> rcl_custom:C-EU0603-C-NOSILK
- C56: value 10nF -> 10nF 10V; device rcl:C-EUC0402 -> rcl_custom:C-EU0402-C-NOSILK
- C58: value 0.47uF -> 470nF 10V; device rcl:C-EUC0402 -> rcl_custom:C-EU0402-C-NOSILK
- L2, L5: device SparkFun-Passives:INDUCTOR0402 -> rcl_custom:L-US0402-C-NOSILK
- L3: device rcl_custom:L-US0805-B-NOSILK -> rcl_custom:L-US0805-C-NOSILK
- R1, R10, R11, R12, R13, R15, R16, R18, R2, R20, R22, R23, R24, R25, R27, R28, R29, R3, R38, R39, R4, R40, R42, R43, R44, R45, R46, R47, R48, R5, R6, R7, R8, R9: device rcl:R-US_R0402 -> rcl_custom:R-US_0402-C-NOSILK
Connections:
- net 2.85VA: now also C43.1; no longer C43.2
- net 2.85VD: now also C60.1; no longer C60.2
- net ANTFLAG: now also JP1.14, JP1.9; no longer TP4.1, TP5.1
- net GND: now also USB.GND; no longer U$1.GND
- net I0-DATA_OUT: now also JP1.11, JP1.12; no longer TP30.1, TP31.1
- net I1-CLK_SER: now also JP1.10, JP1.13; no longer TP25.1, TP28.1
- net LD: now also JP1.15, JP1.8; no longer TP29.1, TP3.1
- net MAX_!IDLE: now also JP1.19, JP1.4, U8.PE11; no longer TP8.1, TP9.1, U8.PE9
- net MAX_!SHDN: now also JP1.18, JP1.5, U8.PE10; no longer TP6.1, TP7.1, U8.PE7
- net MAX_CFG_!CS: now also JP1.20, JP1.3; no longer TP14.1, TP15.1
- net MAX_CFG_MOSI: now also JP1.1, JP1.22; no longer TP21.1, TP24.1
- net MAX_CFG_SCLK: now also JP1.2, JP1.21; no longer TP19.1, TP20.1
- net N$13: now also C43.2; no longer C43.1
- net N$16: now also C60.2; no longer C60.1
- net OTG_FS_DM: now also USB.D-; no longer U$1.D-
- net OTG_FS_DP: now also USB.D+; no longer U$1.D+
- net OTG_FS_VBUS: now also USB.VCC; no longer U$1.VCC
- net Q0-DATASYNC: now also JP1.16, JP1.7, U8.PE7; no longer TP10.1, TP11.1, U8.PE10
- net Q1-TIMESYNC: now also JP1.17, JP1.6, U8.PE9; no longer TP12.1, TP13.1, U8.PE11
- net SHLD: now also USB.SHLD@1, USB.SHLD@2, USB.SHLD@3, USB.SHLD@4; no longer U$1.SHLD@1, U$1.SHLD@2, U$1.SHLD@3, U$1.SHLD@4
Other:
- note added: "CHOICE #1"
- note added: "CHOICE #2"

Commit message: Fresh libraries export. Sent email to Andrew with notes.
Parts:
- C33: device rcl_custom:C-EU0805-C-NOSILK -> rcl_custom:C-EU1206-C
- C58: device rcl_custom:C-EU0402-C-NOSILK -> rcl_custom:C-EU0603-C-NOSILK
- L6, L7: value SAW -> SAW_1.4X1.1
- R7: value 240k -> 249k
- renumbered SD to SD1, U2 to L7
Changed lines of the file:
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@@
 <part name="U1" library="max2769" deviceset="MAX2769" device=""/>
 <part name="C11" library="rcl_custom" deviceset="C-EU" device="0402-C-NOSILK" value="DNP"/>
-<part name="U2" library="swift-nav" deviceset="SAW_1.4X1.1" device="" value="SAW"/>
+<part name="L7" library="swift-nav" deviceset="SAW_1.4X1.1" device="" value="SAW_1.4X1.1"/>
 <part name="BAR_GND1" library="supply" deviceset="GND_BAR" device="" value="GND"/>
 <part name="U4" library="swift-nav" deviceset="7Q-16.368MBG-T" device=""/>
@@
 <part name="U$6" library="SparkFun-Aesthetics" deviceset="2.85VD" device=""/>
 <part name="U5" library="swift-nav" deviceset="XC2401" device=""/>
-<part name="L6" library="swift-nav" deviceset="SAW_1.4X1.1" device="" value="SAW"/>
+<part name="L6" library="swift-nav" deviceset="SAW_1.4X1.1" device="" value="SAW_1.4X1.1"/>
 <part name="BAR_GND2" library="supply" deviceset="GND_BAR" device="" value="GND"/>
-<part name="C58" library="rcl_custom" deviceset="C-EU" device="0402-C-NOSILK" value="470nF 10V"/>
+<part name="C58" library="rcl_custom" deviceset="C-EU" device="0603-C-NOSILK" value="470nF 10V"/>
 <part name="DIG_GND28" library="supply" deviceset="GND_BAR" device="" value="GND"/>
 <part name="DIG_GND9" library="supply" deviceset="GND_BAR" device="" value="GND"/>
@@
 <part name="TP33" library="Tova" deviceset="TEST-POINT" device=""/>
 <part name="DIG_GND18" library="supply" deviceset="GND_BAR" device="" value="GND"/>
-<part name="SD" library="con-usd-hirose-dm3-gpsboard" deviceset="CON_HIROSE_DM3*" device="D(MICROSD)"/>
+<part name="SD1" library="con-usd-hirose-dm3-gpsboard" deviceset="CON_HIROSE_DM3*" device="D(MICROSD)"/>
 <part name="DIG_GND21" library="supply" deviceset="GND_BAR" device="" value="GND"/>
 <part name="DIG_GND31" library="supply" deviceset="GND_BAR" device="" value="GND"/>
@@
 <part name="R1" library="rcl_custom" deviceset="R-US_" device="0402-C-NOSILK" value="10k"/>
 <part name="R3" library="rcl_custom" deviceset="R-US_" device="0402-C-NOSILK" value="3.3k"/>
-<part name="R7" library="rcl_custom" deviceset="R-US_" device="0402-C-NOSILK" value="240k"/>
+<part name="R7" library="rcl_custom" deviceset="R-US_" device="0402-C-NOSILK" value="249k"/>
 <part name="GND4" library="SparkFun-Aesthetics" deviceset="GND" device=""/>
 <part name="C38" library="SparkFun-Passives" deviceset="CAP_POL" device="6032" value="100u 10V"/>
 <part name="GND15" library="SparkFun-Aesthetics" deviceset="GND" device=""/>
-<part name="C33" library="rcl_custom" deviceset="C-EU" device="0805-C-NOSILK" value="10uF 50V"/>
+<part name="C33" library="rcl_custom" deviceset="C-EU" device="1206-C" value="10uF 50V"/>
 <part name="GND2" library="SparkFun-Aesthetics" deviceset="GND" device=""/>
 <part name="C39" library="rcl_custom" deviceset="C-EU" device="0603-C-NOSILK" value="1uF 10V"/>
@@
 <instance part="LED4" gate="G$1" x="283.21" y="99.06" rot="R90"/>
 <instance part="DIG_GND18" gate="1" x="264.16" y="37.846"/>
-<instance part="SD" gate="$" x="51.562" y="117.094" rot="MR0"/>
-<instance part="SD" gate="G1" x="55.372" y="102.87"/>
-<instance part="SD" gate="G2" x="55.372" y="100.33"/>
-<instance part="SD" gate="G3" x="55.372" y="97.79"/>
-<instance part="SD" gate="G4" x="55.372" y="95.25"/>
-<instance part="SD" gate="CD" x="54.102" y="134.112"/>
+<instance part="SD1" gate="$" x="51.562" y="117.094" rot="MR0"/>
+<instance part="SD1" gate="G1" x="55.372" y="102.87"/>
+<instance part="SD1" gate="G2" x="55.372" y="100.33"/>
+<instance part="SD1" gate="G3" x="55.372" y="97.79"/>
+<instance part="SD1" gate="G4" x="55.372" y="95.25"/>
+<instance part="SD1" gate="CD" x="54.102" y="134.112"/>
 <instance part="DIG_GND21" gate="1" x="65.532" y="131.572"/>
 <instance part="DIG_GND31" gate="1" x="41.656" y="131.572"/>
@@
 <wire x1="65.532" y1="107.696" x2="65.532" y2="102.87" width="0.1524" layer="91"/>
 <junction x="65.532" y="102.87"/>
-<pinref part="SD" gate="G1" pin="PAD"/>
+<pinref part="SD1" gate="G1" pin="PAD"/>
 <wire x1="57.912" y1="102.87" x2="62.992" y2="102.87" width="0.1524" layer="91"/>
-<pinref part="SD" gate="G2" pin="PAD"/>
+<pinref part="SD1" gate="G2" pin="PAD"/>
 <wire x1="62.992" y1="100.33" x2="57.912" y2="100.33" width="0.1524" layer="91"/>
-<pinref part="SD" gate="G3" pin="PAD"/>
+<pinref part="SD1" gate="G3" pin="PAD"/>
 <wire x1="57.912" y1="97.79" x2="65.532" y2="97.79" width="0.1524" layer="91"/>
-<pinref part="SD" gate="G4" pin="PAD"/>
+<pinref part="SD1" gate="G4" pin="PAD"/>
 <wire x1="57.912" y1="95.25" x2="65.532" y2="95.25" width="0.1524" layer="91"/>
 <junction x="65.532" y="95.25"/>
 <junction x="65.532" y="97.79"/>
-<pinref part="SD" gate="$" pin="6"/>
+<pinref part="SD1" gate="$" pin="6"/>
 <wire x1="58.42" y1="107.696" x2="57.15" y2="107.696" width="0.1524" layer="91"/>
 </segment>
 <segment>
-<pinref part="SD" gate="CD" pin="1"/>
+<pinref part="SD1" gate="CD" pin="1"/>
 <pinref part="DIG_GND21" gate="1" pin="BAR_GND"/>
 <wire x1="56.642" y1="134.112" x2="60.706" y2="134.112" width="0.1524" layer="91"/>
@@
 </segment>
 <segment>
-<pinref part="SD" gate="CD" pin="0"/>
+<pinref part="SD1" gate="CD" pin="0"/>
 <pinref part="DIG_GND31" gate="1" pin="BAR_GND"/>
 <wire x1="49.022" y1="134.112" x2="41.656" y2="134.112" width="0.1524" layer="91"/>
@@
 <pinref part="U8" gate="G$1" pin="PC8"/>
 <wire x1="57.15" y1="125.476" x2="167.64" y2="125.73" width="0.1524" layer="91"/>
-<pinref part="SD" gate="$" pin="7"/>
+<pinref part="SD1" gate="$" pin="7"/>
 </segment>
 </net>
@@
 <pinref part="U8" gate="G$1" pin="PC9"/>
 <wire x1="167.64" y1="115.57" x2="57.15" y2="115.316" width="0.1524" layer="91"/>
-<pinref part="SD" gate="$" pin="8"/>
+<pinref part="SD1" gate="$" pin="8"/>
 </segment>
 </net>
@@
 <pinref part="U8" gate="G$1" pin="PC10"/>
 <wire x1="167.64" y1="113.03" x2="57.15" y2="112.776" width="0.1524" layer="91"/>
-<pinref part="SD" gate="$" pin="1"/>
+<pinref part="SD1" gate="$" pin="1"/>
 </segment>
 </net>
@@
 <pinref part="U8" gate="G$1" pin="PC12"/>
 <wire x1="57.15" y1="120.396" x2="167.64" y2="120.65" width="0.1524" layer="91"/>
-<pinref part="SD" gate="$" pin="5"/>
+<pinref part="SD1" gate="$" pin="5"/>
 </segment>
 </net>
@@
 <pinref part="U8" gate="G$1" pin="PD2"/>
 <wire x1="57.15" y1="122.936" x2="167.64" y2="123.19" width="0.1524" layer="91"/>
-<pinref part="SD" gate="$" pin="3"/>
+<pinref part="SD1" gate="$" pin="3"/>
 </segment>
 </net>
@@
 <pinref part="U8" gate="G$1" pin="PC11"/>
 <wire x1="163.83" y1="118.11" x2="167.64" y2="118.11" width="0.15" layer="91"/>
-<pinref part="SD" gate="$" pin="2"/>
+<pinref part="SD1" gate="$" pin="2"/>
 </segment>
 </net>
@@
 <wire x1="57.15" y1="110.236" x2="73.152" y2="110.236" width="0.1524" layer="91"/>
 <wire x1="73.152" y1="110.236" x2="73.152" y2="107.188" width="0.1524" layer="91"/>
-<pinref part="SD" gate="$" pin="4"/>
+<pinref part="SD1" gate="$" pin="4"/>
 <label x="63.5" y="110.49" size="1.778" layer="95"/>
 <wire x1="73.152" y1="110.236" x2="89.154" y2="110.236" width="0.1524" layer="91"/>
@@
 <attribute name="VALUE" x="208.28" y="143.002" size="1.778" layer="96"/>
 </instance>
-<instance part="U2" gate="U1" x="204.47" y="88.646"/>
+<instance part="L7" gate="U1" x="204.47" y="88.646" smashed="yes">
+<attribute name="NAME" x="197.358" y="97.028" size="1.27" layer="95"/>
+<attribute name="VALUE" x="214.122" y="97.028" size="1.27" layer="96" align="bottom-right"/>
+</instance>
 <instance part="BAR_GND1" gate="1" x="205.74" y="73.914"/>
 <instance part="U4" gate="U$1" x="170.942" y="142.748"/>
@@
 </segment>
 <segment>
-<pinref part="U2" gate="U1" pin="GND1"/>
-<pinref part="U2" gate="U1" pin="GND3"/>
+<pinref part="L7" gate="U1" pin="GND1"/>
+<pinref part="L7" gate="U1" pin="GND3"/>
 <wire x1="200.66" y1="78.486" x2="205.74" y2="78.486" width="0.15" layer="91"/>
 <wire x1="205.74" y1="78.486" x2="210.82" y2="78.486" width="0.15" layer="91"/>
-<pinref part="U2" gate="U1" pin="GND2"/>
+<pinref part="L7" gate="U1" pin="GND2"/>
 <pinref part="BAR_GND1" gate="1" pin="BAR_GND"/>
 <junction x="205.74" y="78.486"/>
@@
 <net name="LNAOUT" class="0">
 <segment>
-<pinref part="U2" gate="U1" pin="RFIN"/>
+<pinref part="L7" gate="U1" pin="RFIN"/>
 <pinref part="U1" gate="G$1" pin="LNAOUT"/>
 <wire x1="191.77" y1="93.726" x2="191.77" y2="111.506" width="0.15" layer="91"/>
@@
 <net name="MIXIN" class="0">
 <segment>
-<pinref part="U2" gate="U1" pin="RFOUT"/>
+<pinref part="L7" gate="U1" pin="RFOUT"/>
 <pinref part="U1" gate="G$1" pin="MIXIN"/>
 <wire x1="219.71" y1="93.726" x2="219.71" y2="106.426" width="0.1524" layer="91"/>

Commit message: Cleanup on Jenner's fine work. Mostly adding polygons to power signals, some additional caps, moving parts around for optimal placement, added mounting holes, made polygon lines consistent. NOT DONE YET, still have RF cleanup and Ethernet cleanup to do.
Parts:
- removed D1: 25V 1A, SparkFun-DiscreteSemi:DIODESMA-ALT
- removed JTAG1: M05X2PTH, SparkFun-Connectors:M05X2PTH
- removed TP18, TP2: TPTP06R, testpad:TPTP06R
- added C25, C54, C55: 100n, rcl_custom:C-EU0402-B-NOSILK
- added D2: DIODE-0603, diode-0603:DIODE-0603
- added J1: 1.27MM-SWD-CONNECTOR, con-swd:1.27MM-SWD-CONNECTOR
- added U$1, U$12, U$14, U$18: #4-BARE_MOUNTING_HOLE/.300, mount:#4-BARE_MOUNTING_HOLE/.300
- C1: device rcl_custom:C-EU0603-C-NOSILK -> rcl_custom:C-EU0805-B-NOSILK
- C26: value 220nF 10V -> 220nF
- C38: value 100u 10V -> 100u
- C39: value 1uF 10V -> 1uF; device rcl_custom:C-EU0603-C-NOSILK -> rcl_custom:C-EU0603-B-NOSILK
- C40, C41, C42, C59: value 1uF 10V -> 1u; device rcl_custom:C-EU0603-C-NOSILK -> rcl_custom:C-EU0603-B-NOSILK
- C43, C60: value 1uF 10V -> 10n; device rcl_custom:C-EU0603-C-NOSILK -> rcl_custom:C-EU0402-B-NOSILK
Connections:
- net !RST: now also J1.!RESET; no longer JTAG1.10, TP2.TP
- net 2.85VA: now also C55.1
- net 3.3VD: now also C54.1, J1.VTREF; no longer JTAG1.1
- net GND: now also C25.2, C54.2, C55.2, J1.GND, J1.GND@2, J1.GNDDET; no longer JTAG1.3, JTAG1.5, JTAG1.9
- net OTG_FS_VBUS: now also D2.ANODE; no longer D1.A
- net TCK: now also J1.SWDCLK/TCK; no longer JTAG1.4
- net TDI: now also J1.NC/TDI; no longer JTAG1.8
- net TDO: now also J1.SWO/TDO; no longer JTAG1.6
- net TMS: now also J1.SWDIO/TMS; no longer JTAG1.2
- net VIN: now also C25.1, D2.CATHODE; no longer D1.C, TP18.TP
Other:
- note added: "0805"
- note added: "1206"
- note added: "Aux supply from USB debug"
- note added: "TODO: 0603 50V?"
- moved on the sheet: C1, C21, C26, C33, C38, C39, C40, C41, C42, C43, C59, C60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
