File: v2-rf-frontend-board.sch (EAGLE design)
At the start: 150 parts, among them J1 1.27MM-SWD-CONNECTOR, J2 CON_SMA-ENDFIRE_EMERSON_EMERS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, J3 ROCKETNET-CONNECTOR-16M, J4 ZX62D-B-5P8, J5 BREAKOUT, J7 CON_HIROSE_DM3D(MICROSD), Q1 NTR4101P, T1 ALT4532, T2 ALT4532, U1 MAX2769, U2 STM32F4V_100PIN_GPSBOARD, U3 KSZ8081, U4 7Q-16.368MBG-T, U5 XC2401A8167R-G, U6 MAX8510EXK29+T, U7 MAX8510EXK29+T, U8 LMZ12001, X1 25 MHz

Commit message: Silly clean up, ran ERC and DRC again.
Other:
- note removed: "MAX_INPUTS"
- note removed: "MAX_OUTPUTS"
Changed lines of the file:
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@@
 <text x="261.62" y="80.01" size="1.778" layer="95">3-wire faux-SPI serial config bus</text>
 <text x="64.77" y="179.07" size="1.778" layer="97">NC</text>
-<text x="345.44" y="93.98" size="1.778" layer="97">MAX_INPUTS</text>
-<text x="345.44" y="63.5" size="1.778" layer="97">MAX_OUTPUTS</text>
 <text x="314.452" y="30.226" size="1.778" layer="95">2mm digital int.
 to MAX2769</text>
@@
 <text x="297.18" y="135.89" size="1.778" layer="97" rot="R90">To COTS GPS
 (and FTDI)</text>
+<text x="372.11" y="95.25" size="2.54" layer="97" rot="R180">MAX INPUTS</text>
+<text x="375.92" y="67.31" size="2.54" layer="97" rot="R180">MAX OUTPUTS</text>
 </plain>
 <instances>
@@
 <bus name="MAX_!IDLE,MAX_!SHDN,MAX_CFG_SCLK,MAX_CFG_MOSI,MAX_CFG_!CS">
 <segment>
-<wire x1="342.9" y1="96.266" x2="342.9" y2="73.66" width="0.762" layer="92"/>
+<wire x1="347.98" y1="93.98" x2="342.9" y2="93.98" width="0.762" layer="92"/>
+<wire x1="342.9" y1="93.98" x2="342.9" y2="73.66" width="0.762" layer="92"/>
 </segment>
 </bus>
 <bus name="ANTFLAG,LD,I0-DATA_OUT,I1-CLK_SER,Q0-DATASYNC,Q1-TIMESYNC">
 <segment>
+<wire x1="347.98" y1="66.04" x2="342.9" y2="66.04" width="0.762" layer="92"/>
 <wire x1="342.9" y1="66.04" x2="342.9" y2="43.18" width="0.762" layer="92"/>
 </segment>
+<segment>
+<wire x1="347.98" y1="93.98" x2="350.52" y2="96.52" width="0.1524" layer="92"/>
+<wire x1="350.52" y1="96.52" x2="373.38" y2="96.52" width="0.1524" layer="92"/>
+<wire x1="373.38" y1="96.52" x2="373.38" y2="91.44" width="0.1524" layer="92"/>
+<wire x1="373.38" y1="91.44" x2="350.52" y2="91.44" width="0.1524" layer="92"/>
+<wire x1="350.52" y1="91.44" x2="347.98" y2="93.98" width="0.1524" layer="92"/>
+</segment>
+<segment>
+<wire x1="347.98" y1="66.04" x2="350.52" y2="68.58" width="0.1524" layer="92"/>
+<wire x1="350.52" y1="68.58" x2="377.19" y2="68.58" width="0.1524" layer="92"/>
+<wire x1="377.19" y1="68.58" x2="377.19" y2="63.5" width="0.1524" layer="92"/>
+<wire x1="377.19" y1="63.5" x2="350.52" y2="63.5" width="0.1524" layer="92"/>
+<wire x1="350.52" y1="63.5" x2="347.98" y2="66.04" width="0.1524" layer="92"/>
+</segment>
 </bus>

Commit message: Added modwire proposals for SPI 3-wire fix. See Issue 4 in gps-rf-board github repository.
Connections:
- net MAX_CFG_!CS: now also U2.PB9
- net MAX_CFG_MOSI: now also U2.PB15
- net MAX_CFG_SCLK: now also U2.PB10
Other:
- note added: "SPI2_MOSI AF=5 (MODWIRE)"
- note added: "SPI2_NSS AF=5 (MODWIRE)"
- note added: "SPI2_SCK AF=5 (MODWIRE)"
Changed lines of the file:
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@@
 <setting verticaltext="up"/>
 </settings>
-<grid distance="0.05" unitdist="inch" unit="inch" style="lines" multiple="2" display="yes" altdistance="0.01" altunitdist="inch" altunit="inch"/>
+<grid distance="0.1" unitdist="inch" unit="mm" style="lines" multiple="1" display="yes" altdistance="0.01" altunitdist="inch" altunit="mm"/>
 <layers>
 <layer number="1" name="Top" color="4" fill="1" visible="no" active="no"/>
@@
 <text x="372.11" y="95.25" size="2.54" layer="97" rot="R180">MAX INPUTS</text>
 <text x="375.92" y="67.31" size="2.54" layer="97" rot="R180">MAX OUTPUTS</text>
+<text x="155.194" y="17.272" size="1.9304" layer="97" ratio="14" rot="R90">SPI2_SCK AF=5 (MODWIRE)</text>
+<text x="165.354" y="24.892" size="1.9304" layer="97" ratio="14" rot="R90">SPI2_NSS AF=5 (MODWIRE)</text>
+<text x="360.934" y="123.952" size="1.9304" layer="97" ratio="13" rot="R90">SPI2_MOSI AF=5 (MODWIRE)</text>
 </plain>
 <instances>
@@
 <pinref part="J5" gate="G$1" pin="22"/>
 <wire x1="313.69" y1="88.9" x2="328.93" y2="88.9" width="0.1524" layer="91"/>
-<wire x1="328.93" y1="88.9" x2="342.9" y2="88.9" width="0.1524" layer="91"/>
+<wire x1="328.93" y1="88.9" x2="335.28" y2="88.9" width="0.1524" layer="91"/>
 <junction x="328.93" y="88.9"/>
 <junction x="313.69" y="88.9"/>
 <pinref part="U2" gate="U" pin="PE14"/>
+<pinref part="U2" gate="U" pin="PB15"/>
+<wire x1="335.28" y1="88.9" x2="342.9" y2="88.9" width="0.1524" layer="91"/>
+<wire x1="241.3" y1="187.96" x2="241.3" y2="193.04" width="0.8128" layer="91"/>
+<wire x1="241.3" y1="193.04" x2="355.6" y2="193.04" width="0.8128" layer="91"/>
+<wire x1="355.6" y1="193.04" x2="355.6" y2="106.68" width="0.8128" layer="91"/>
+<wire x1="355.6" y1="106.68" x2="335.28" y2="106.68" width="0.8128" layer="91"/>
+<wire x1="335.28" y1="106.68" x2="335.28" y2="88.9" width="0.8128" layer="91"/>
+<junction x="335.28" y="88.9"/>
 </segment>
 </net>
@@
 <segment>
 <pinref part="J5" gate="G$1" pin="21"/>
-<wire x1="328.93" y1="86.36" x2="342.9" y2="86.36" width="0.1524" layer="91"/>
+<wire x1="328.93" y1="86.36" x2="337.82" y2="86.36" width="0.1524" layer="91"/>
 <label x="261.62" y="86.36" size="1.778" layer="95"/>
+<wire x1="337.82" y1="86.36" x2="342.9" y2="86.36" width="0.1524" layer="91"/>
 <wire x1="313.69" y1="86.36" x2="254" y2="86.36" width="0.1524" layer="91"/>
 <pinref part="J5" gate="G$1" pin="2"/>
@@
 <junction x="328.93" y="86.36"/>
 <pinref part="U2" gate="U" pin="PE13"/>
+<pinref part="U2" gate="U" pin="PB10"/>
+<wire x1="170.18" y1="71.12" x2="157.48" y2="71.12" width="0.8128" layer="91"/>
+<wire x1="157.48" y1="71.12" x2="157.48" y2="15.24" width="0.8128" layer="91"/>
+<wire x1="157.48" y1="15.24" x2="337.82" y2="15.24" width="0.8128" layer="91"/>
+<wire x1="337.82" y1="15.24" x2="337.82" y2="86.36" width="0.8128" layer="91"/>
+<junction x="337.82" y="86.36"/>
 </segment>
 </net>
@@
 <pinref part="J5" gate="G$1" pin="20"/>
 <wire x1="313.69" y1="83.82" x2="328.93" y2="83.82" width="0.1524" layer="91"/>
-<wire x1="328.93" y1="83.82" x2="342.9" y2="83.82" width="0.1524" layer="91"/>
+<wire x1="328.93" y1="83.82" x2="332.74" y2="83.82" width="0.1524" layer="91"/>
 <junction x="328.93" y="83.82"/>
 <junction x="313.69" y="83.82"/>
 <pinref part="U2" gate="U" pin="PE12"/>
-</segment>
-</net>
+<pinref part="U2" gate="U" pin="PB9"/>
+<wire x1="332.74" y1="83.82" x2="342.9" y2="83.82" width="0.1524" layer="91"/>
+<wire x1="170.18" y1="68.58" x2="162.56" y2="68.58" width="0.8128" layer="91"/>
+<wire x1="162.56" y1="68.58" x2="162.56" y2="20.32" width="0.8128" layer="91"/>
+<wire x1="162.56" y1="20.32" x2="332.74" y2="20.32" width="0.8128" layer="91"/>
+<wire x1="332.74" y1="20.32" x2="332.74" y2="83.82" width="0.8128" layer="91"/>
+<junction x="332.74" y="83.82"/>
+</segment>
+</net>

Commit message: Removed SPI2_NSS modwire proposal from v2 schematic.
Connections:
- net MAX_CFG_!CS: no longer U2.PB9
Other:
- note removed: "SPI2_NSS AF=5 (MODWIRE)"
Changed lines of the file:
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@@
 <text x="375.92" y="67.31" size="2.54" layer="97" rot="R180">MAX OUTPUTS</text>
 <text x="155.194" y="17.272" size="1.9304" layer="97" ratio="14" rot="R90">SPI2_SCK AF=5 (MODWIRE)</text>
-<text x="165.354" y="24.892" size="1.9304" layer="97" ratio="14" rot="R90">SPI2_NSS AF=5 (MODWIRE)</text>
 <text x="360.934" y="123.952" size="1.9304" layer="97" ratio="13" rot="R90">SPI2_MOSI AF=5 (MODWIRE)</text>
 </plain>
@@
 <pinref part="J5" gate="G$1" pin="20"/>
 <wire x1="313.69" y1="83.82" x2="328.93" y2="83.82" width="0.1524" layer="91"/>
-<wire x1="328.93" y1="83.82" x2="332.74" y2="83.82" width="0.1524" layer="91"/>
 <junction x="328.93" y="83.82"/>
 <junction x="313.69" y="83.82"/>
 <pinref part="U2" gate="U" pin="PE12"/>
-<pinref part="U2" gate="U" pin="PB9"/>
-<wire x1="332.74" y1="83.82" x2="342.9" y2="83.82" width="0.1524" layer="91"/>
-<wire x1="170.18" y1="68.58" x2="162.56" y2="68.58" width="0.8128" layer="91"/>
-<wire x1="162.56" y1="68.58" x2="162.56" y2="20.32" width="0.8128" layer="91"/>
-<wire x1="162.56" y1="20.32" x2="332.74" y2="20.32" width="0.8128" layer="91"/>
-<wire x1="332.74" y1="20.32" x2="332.74" y2="83.82" width="0.8128" layer="91"/>
-<junction x="332.74" y="83.82"/>
-</segment>
-</net>
+<wire x1="328.93" y1="83.82" x2="342.9" y2="83.82" width="0.1524" layer="91"/>
+</segment>
+</net>

Commit message: Removed !SS line from patch, made it pretty, in schematic. Added older docs that should have been added. Updated BOM with digikey part numbers.
Other:
- note added: "MODWIRE"
- note added: "PA5: SPI1_SCK"
- note added: "PB10: SPI2_SCK / AF=5"
- note added: "PB15: SPI2_MOSI / AF=5"
- note added: "PB5: SPI1_MOSI"
- note added: "STM32F407VG (LQFP100)"
- note removed: "SPI2_MOSI AF=5 (MODWIRE)"
- note removed: "SPI2_SCK AF=5 (MODWIRE)"
- moved on the sheet: C10, C11, C20, C29, C30, C45, C46, C47, C48, C49, C50, C51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

Commit message: Added annotation for DEBUG-PHY-MODWIRE (currently on prototype)
Connections:
- removed net N$39: LED6.C, U3.LED0/ANEN_SPEED
- removed net N$57: TP1.1, U2.PE2
- new net DEBUG-PHY-MODWIRE: LED6.C, TP1.1, U2.PE2, U3.LED0/ANEN_SPEED
Changed lines of the file:
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@@
 <?xml version="1.0" encoding="utf-8"?>
 <!DOCTYPE eagle SYSTEM "eagle.dtd">
-<eagle version="6.6.0">
+<eagle version="6.5.0">
 <drawing>
 <settings>
@@
 <setting verticaltext="up"/>
 </settings>
-<grid distance="0.05" unitdist="inch" unit="inch" style="lines" multiple="2" display="no" altdistance="0.01" altunitdist="inch" altunit="inch"/>
+<grid distance="0.1" unitdist="inch" unit="mm" style="lines" multiple="1" display="yes" altdistance="0.01" altunitdist="inch" altunit="mm"/>
 <layers>
 <layer number="1" name="Top" color="4" fill="1" visible="no" active="no"/>
@@
 <text x="248.92" y="53.34" size="1.778" layer="97">PB5: SPI1_MOSI</text>
 <text x="326.39" y="36.83" size="1.778" layer="102" rot="R90">MODWIRE</text>
+<text x="110.49" y="92.71" size="1.778" layer="102" rot="R90">MODWIRE</text>
 </plain>
 <instances>
@@
 </segment>
 </net>
-<net name="N$57" class="0">
+<net name="DEBUG-PHY-MODWIRE" class="0">
 <segment>
 <pinref part="TP1" gate="G$1" pin="1"/>
 <pinref part="U2" gate="U" pin="PE2"/>
-<wire x1="149.86" y1="99.06" x2="160.02" y2="99.06" width="0.1524" layer="91"/>
+<wire x1="149.86" y1="99.06" x2="157.48" y2="99.06" width="0.1524" layer="91"/>
+<label x="101.6" y="88.9" size="1.778" layer="102" font="vector" rot="R180" xref="yes"/>
+<wire x1="157.48" y1="99.06" x2="160.02" y2="99.06" width="0.1524" layer="91"/>
+<wire x1="157.48" y1="104.14" x2="157.48" y2="99.06" width="0.1524" layer="91" style="shortdash"/>
+<junction x="157.48" y="99.06"/>
+<wire x1="101.6" y1="88.9" x2="111.76" y2="88.9" width="0.1524" layer="91" style="shortdash"/>
+<wire x1="111.76" y1="88.9" x2="111.76" y2="104.14" width="0.1524" layer="91" style="shortdash"/>
+<wire x1="111.76" y1="104.14" x2="157.48" y2="104.14" width="0.1524" layer="91" style="shortdash"/>
 </segment>
 </net>
@@
 <text x="273.05" y="110.49" size="1.778" layer="97">25 MHz from STM32</text>
 <text x="278.13" y="115.57" size="1.778" layer="97">50 MHz to STM32 ETH</text>
+<text x="238.76" y="83.82" size="1.778" layer="102">MODWIRE</text>
 </plain>
 <instances>
@@
 </segment>
 </net>
-<net name="N$39" class="0">
+<net name="DEBUG-PHY-MODWIRE" class="0">
 <segment>
 <pinref part="U3" gate="G$1" pin="LED0/ANEN_SPEED"/>
 <wire x1="220.98" y1="124.46" x2="236.22" y2="124.46" width="0.1524" layer="91"/>
-<wire x1="236.22" y1="124.46" x2="236.22" y2="71.12" width="0.1524" layer="91"/>
+<wire x1="236.22" y1="124.46" x2="236.22" y2="86.36" width="0.1524" layer="91"/>
+<wire x1="236.22" y1="86.36" x2="236.22" y2="71.12" width="0.1524" layer="91"/>
 <wire x1="236.22" y1="71.12" x2="223.52" y2="71.12" width="0.1524" layer="91"/>
 <wire x1="223.52" y1="71.12" x2="223.52" y2="78.74" width="0.1524" layer="91"/>
 <pinref part="LED6" gate="G$1" pin="C"/>
+<label x="256.54" y="86.36" size="1.778" layer="102" font="vector" xref="yes"/>
+<wire x1="256.54" y1="86.36" x2="236.22" y2="86.36" width="0.1524" layer="91" style="shortdash"/>
+<junction x="236.22" y="86.36"/>
 </segment>
 </net>

Commit message: Added modwire for SPI1-NSS. This should enable the use of STM32 SPI1 in slave mode to read data output.
Connections:
- new net N$3: U2.PB0
- new net SPI1-NSS: U2.PA4, U2.PA6
Changed lines of the file:
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@@
 <text x="257.81" y="90.17" size="1.778" layer="95">3-wire faux-SPI serial config bus</text>
 <text x="54.61" y="189.23" size="1.778" layer="97">NC</text>
-<text x="304.292" y="40.386" size="1.778" layer="95">2mm digital int.
+<text x="301.752" y="35.306" size="1.778" layer="95">2mm digital int.
 to MAX2769</text>
 <wire x1="250.19" y1="102.616" x2="250.19" y2="88.646" width="0.1524" layer="97" style="longdash"/>
@@
 <wire x1="299.212" y1="88.646" x2="299.212" y2="102.616" width="0.1524" layer="97" style="longdash"/>
 <wire x1="299.212" y1="102.616" x2="250.19" y2="102.616" width="0.1524" layer="97" style="longdash"/>
-<text x="261.874" y="45.466" size="1.778" layer="95">actual-SPI I/Q data in</text>
-<wire x1="245.872" y1="58.928" x2="245.872" y2="43.942" width="0.1524" layer="97" style="longdash"/>
-<wire x1="298.958" y1="58.928" x2="245.872" y2="58.928" width="0.1524" layer="97" style="longdash"/>
-<wire x1="298.958" y1="43.942" x2="298.958" y2="58.928" width="0.1524" layer="97" style="longdash"/>
-<wire x1="245.872" y1="43.942" x2="298.958" y2="43.942" width="0.1524" layer="97" style="longdash"/>
+<text x="256.794" y="49.276" size="1.778" layer="95">actual-SPI I/Q data in</text>
+<wire x1="248.412" y1="58.928" x2="248.412" y2="46.482" width="0.1524" layer="97" style="longdash"/>
+<wire x1="298.958" y1="58.928" x2="248.412" y2="58.928" width="0.1524" layer="97" style="longdash"/>
+<wire x1="298.958" y1="46.482" x2="298.958" y2="58.928" width="0.1524" layer="97" style="longdash"/>
+<wire x1="248.412" y1="46.482" x2="298.958" y2="46.482" width="0.1524" layer="97" style="longdash"/>
 <wire x1="35.56" y1="149.352" x2="35.56" y2="148.59" width="0.1524" layer="94"/>
 <wire x1="35.56" y1="148.59" x2="35.56" y2="102.616" width="0.4064" layer="94"/>
@@
 <text x="153.67" y="25.4" size="1.778" layer="102">MODWIRE</text>
 <text x="151.13" y="50.8" size="1.778" layer="102" rot="R90">MODWIRE</text>
-<text x="248.92" y="55.88" size="1.778" layer="97">PA5: SPI1_SCK</text>
-<text x="248.92" y="53.34" size="1.778" layer="97">PB5: SPI1_MOSI</text>
-<text x="326.39" y="36.83" size="1.778" layer="102" rot="R90">MODWIRE</text>
+<text x="251.46" y="55.88" size="1.778" layer="97">PA5: SPI1_SCK</text>
+<text x="251.46" y="53.34" size="1.778" layer="97">PB5: SPI1_MOSI</text>
+<text x="326.39" y="41.91" size="1.778" layer="102" rot="R90">MODWIRE</text>
 <text x="110.49" y="92.71" size="1.778" layer="102" rot="R90">MODWIRE</text>
+<text x="244.094" y="40.894" size="1.778" layer="102" rot="R180">MODWIRE</text>
 </plain>
 <instances>
@@
 </segment>
 </net>
+<net name="N$3" class="0">
+<segment>
+<pinref part="U2" gate="U" pin="PB0"/>
+<wire x1="243.84" y1="175.26" x2="251.46" y2="175.26" width="0.1524" layer="91"/>
+</segment>
+</net>
+<net name="SPI1-NSS" class="0">
+<segment>
+<pinref part="U2" gate="U" pin="PA4"/>
+<wire x1="243.84" y1="50.8" x2="246.38" y2="50.8" width="0.1524" layer="91" style="shortdash"/>
+<wire x1="246.38" y1="50.8" x2="246.38" y2="58.42" width="0.1524" layer="91" style="shortdash"/>
+<pinref part="U2" gate="U" pin="PA6"/>
+<wire x1="246.38" y1="58.42" x2="243.84" y2="58.42" width="0.1524" layer="91" style="shortdash"/>
+<label x="228.6" y="38.1" size="1.778" layer="102" rot="R180" xref="yes"/>
+<wire x1="228.6" y1="38.1" x2="246.38" y2="38.1" width="0.1524" layer="91" style="shortdash"/>
+<wire x1="246.38" y1="38.1" x2="246.38" y2="50.8" width="0.1524" layer="91" style="shortdash"/>
+<junction x="246.38" y="50.8"/>
+</segment>
+</net>

Commit message: Cleaned up modwire patches a bit. Added cuts in 0.1" double header.
Connections:
- new net N$4: J5.1, U2.PE14
- net MAX_CFG_MOSI: no longer J5.1, U2.PE14
- net MAX_CFG_SCLK: no longer J5.2, U2.PE13
- net SPI1-NSS: now also J5.2
Other:
- note added: "High speed serial 2 bit I/Q data in"
- note removed: "actual-SPI I/Q data in"
Changed lines of the file:
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@@
 <?xml version="1.0" encoding="utf-8"?>
 <!DOCTYPE eagle SYSTEM "eagle.dtd">
-<eagle version="6.5.0">
+<eagle version="6.6.0">
 <drawing>
 <settings>
@@
 <setting verticaltext="up"/>
 </settings>
-<grid distance="0.1" unitdist="inch" unit="mm" style="lines" multiple="1" display="yes" altdistance="0.01" altunitdist="inch" altunit="mm"/>
+<grid distance="0.05" unitdist="inch" unit="inch" style="lines" multiple="2" display="yes" altdistance="0.01" altunitdist="inch" altunit="inch"/>
 <layers>
 <layer number="1" name="Top" color="4" fill="1" visible="no" active="no"/>
@@
 <description>STM</description>
 <plain>
-<text x="257.81" y="90.17" size="1.778" layer="95">3-wire faux-SPI serial config bus</text>
+<text x="255.27" y="90.17" size="1.778" layer="95">3-wire faux-SPI serial config bus</text>
 <text x="54.61" y="189.23" size="1.778" layer="97">NC</text>
 <text x="301.752" y="35.306" size="1.778" layer="95">2mm digital int.
 to MAX2769</text>
 <wire x1="250.19" y1="102.616" x2="250.19" y2="88.646" width="0.1524" layer="97" style="longdash"/>
-<wire x1="250.19" y1="88.646" x2="299.212" y2="88.646" width="0.1524" layer="97" style="longdash"/>
-<wire x1="299.212" y1="88.646" x2="299.212" y2="102.616" width="0.1524" layer="97" style="longdash"/>
-<wire x1="299.212" y1="102.616" x2="250.19" y2="102.616" width="0.1524" layer="97" style="longdash"/>
-<text x="256.794" y="49.276" size="1.778" layer="95">actual-SPI I/Q data in</text>
-<wire x1="248.412" y1="58.928" x2="248.412" y2="46.482" width="0.1524" layer="97" style="longdash"/>
-<wire x1="298.958" y1="58.928" x2="248.412" y2="58.928" width="0.1524" layer="97" style="longdash"/>
-<wire x1="298.958" y1="46.482" x2="298.958" y2="58.928" width="0.1524" layer="97" style="longdash"/>
-<wire x1="248.412" y1="46.482" x2="298.958" y2="46.482" width="0.1524" layer="97" style="longdash"/>
+<wire x1="250.19" y1="88.646" x2="294.132" y2="88.646" width="0.1524" layer="97" style="longdash"/>
+<wire x1="294.132" y1="88.646" x2="294.132" y2="102.616" width="0.1524" layer="97" style="longdash"/>
+<wire x1="294.132" y1="102.616" x2="250.19" y2="102.616" width="0.1524" layer="97" style="longdash"/>
+<text x="274.32" y="38.1" size="1.778" layer="95">High speed serial
+2 bit I/Q data in</text>
+<wire x1="248.92" y1="35.56" x2="294.64" y2="35.56" width="0.1524" layer="97" style="longdash"/>
+<wire x1="294.64" y1="35.56" x2="294.64" y2="80.01" width="0.1524" layer="97" style="longdash"/>
+<wire x1="294.64" y1="80.01" x2="273.05" y2="80.01" width="0.1524" layer="97" style="longdash"/>
+<wire x1="273.05" y1="80.01" x2="273.05" y2="59.69" width="0.1524" layer="97" style="longdash"/>
+<wire x1="273.05" y1="59.69" x2="248.92" y2="59.69" width="0.1524" layer="97" style="longdash"/>
+<wire x1="248.92" y1="59.69" x2="248.92" y2="35.56" width="0.1524" layer="97" style="longdash"/>
 <wire x1="35.56" y1="149.352" x2="35.56" y2="148.59" width="0.1524" layer="94"/>
 <wire x1="35.56" y1="148.59" x2="35.56" y2="102.616" width="0.4064" layer="94"/>
@@
 <text x="326.39" y="41.91" size="1.778" layer="102" rot="R90">MODWIRE</text>
 <text x="110.49" y="92.71" size="1.778" layer="102" rot="R90">MODWIRE</text>
-<text x="244.094" y="40.894" size="1.778" layer="102" rot="R180">MODWIRE</text>
+<text x="243.586" y="49.784" size="1.778" layer="102" rot="R270">MODWIRE</text>
 </plain>
 <instances>
@@
 <net name="MAX_CFG_MOSI" class="0">
 <segment>
-<label x="251.46" y="99.06" size="1.778" layer="95"/>
-<wire x1="303.53" y1="99.06" x2="243.84" y2="99.06" width="0.1524" layer="91"/>
-<pinref part="J5" gate="G$1" pin="1"/>
 <pinref part="J5" gate="G$1" pin="22"/>
-<wire x1="303.53" y1="99.06" x2="318.77" y2="99.06" width="0.1524" layer="91"/>
 <wire x1="318.77" y1="99.06" x2="325.12" y2="99.06" width="0.1524" layer="91"/>
-<junction x="318.77" y="99.06"/>
-<junction x="303.53" y="99.06"/>
-<pinref part="U2" gate="U" pin="PE14"/>
 <pinref part="U2" gate="U" pin="PB15"/>
 <wire x1="325.12" y1="99.06" x2="332.74" y2="99.06" width="0.1524" layer="91"/>
@@
 <pinref part="J5" gate="G$1" pin="21"/>
 <wire x1="318.77" y1="96.52" x2="327.66" y2="96.52" width="0.1524" layer="91"/>
-<label x="251.46" y="96.52" size="1.778" layer="95"/>
 <wire x1="327.66" y1="96.52" x2="332.74" y2="96.52" width="0.1524" layer="91"/>
-<wire x1="303.53" y1="96.52" x2="243.84" y2="96.52" width="0.1524" layer="91"/>
-<pinref part="J5" gate="G$1" pin="2"/>
-<wire x1="318.77" y1="96.52" x2="303.53" y2="96.52" width="0.1524" layer="91"/>
-<junction x="303.53" y="96.52"/>
-<junction x="318.77" y="96.52"/>
-<pinref part="U2" gate="U" pin="PE13"/>
 <pinref part="U2" gate="U" pin="PB10"/>
 <wire x1="160.02" y1="81.28" x2="147.32" y2="81.28" width="0.1524" layer="91" style="shortdash"/>
@@
 <net name="Q0-DATASYNC" class="0">
 <segment>
-<label x="251.46" y="71.12" size="1.778" layer="95"/>
+<label x="274.32" y="71.12" size="1.778" layer="95"/>
 <wire x1="303.53" y1="71.12" x2="243.84" y2="71.12" width="0.1524" layer="91"/>
 <pinref part="J5" gate="G$1" pin="7"/>
@@
 <net name="Q1-TIMESYNC" class="0">
 <segment>
-<label x="251.46" y="76.2" size="1.778" layer="95"/>
+<label x="274.32" y="76.2" size="1.778" layer="95"/>
 <wire x1="303.53" y1="76.2" x2="243.84" y2="76.2" width="0.1524" layer="91"/>
 <pinref part="J5" gate="G$1" pin="6"/>
@@
 <pinref part="U2" gate="U" pin="PA6"/>
 <wire x1="246.38" y1="58.42" x2="243.84" y2="58.42" width="0.1524" layer="91" style="shortdash"/>
-<label x="228.6" y="38.1" size="1.778" layer="102" rot="R180" xref="yes"/>
-<wire x1="228.6" y1="38.1" x2="246.38" y2="38.1" width="0.1524" layer="91" style="shortdash"/>
+<label x="251.46" y="38.1" size="1.778" layer="102" xref="yes"/>
+<wire x1="251.46" y1="38.1" x2="246.38" y2="38.1" width="0.1524" layer="91" style="shortdash"/>
 <wire x1="246.38" y1="38.1" x2="246.38" y2="50.8" width="0.1524" layer="91" style="shortdash"/>
 <junction x="246.38" y="50.8"/>
-</segment>
-</net>
+<wire x1="303.53" y1="96.52" x2="297.18" y2="96.52" width="0.1524" layer="91" style="shortdash"/>
+<wire x1="297.18" y1="96.52" x2="297.18" y2="62.23" width="0.1524" layer="91" style="shortdash"/>
+<wire x1="297.18" y1="62.23" x2="246.38" y2="62.23" width="0.1524" layer="91" style="shortdash"/>
+<wire x1="246.38" y1="62.23" x2="246.38" y2="58.42" width="0.1524" layer="91" style="shortdash"/>
+<junction x="246.38" y="58.42"/>
+<pinref part="J5" gate="G$1" pin="2"/>
+</segment>
+</net>
+<net name="N$4" class="0">
+<segment>
+<pinref part="J5" gate="G$1" pin="1"/>
+<wire x1="303.53" y1="99.06" x2="243.84" y2="99.06" width="0.1524" layer="91"/>
+<pinref part="U2" gate="U" pin="PE14"/>
+</segment>
+</net>
