File: v2-rf-frontend-board.sch (EAGLE design)
At the start: 150 parts, among them J1 1.27MM-SWD-CONNECTOR, J2 CON_SMA-ENDFIRE_EMERSON_EMERS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, J3 ROCKETNET-CONNECTOR-16M, J4 ZX62D-B-5P8, J5 BREAKOUT, J7 CON_HIROSE_DM3D(MICROSD), Q1 NTR4101P, T1 ALT4532, T2 ALT4532, U1 MAX2769, U2 STM32F4V_100PIN_GPSBOARD, U3 KSZ8081, U4 7Q-16.368MBG-T, U5 XC2401A8167R-G, U6 MAX8510EXK29+T, U7 MAX8510EXK29+T, U8 LMZ12001, X1 25 MHz

Commit message: Whoops, fixed CLK and DATA mixup from MAX using even MORE modwires.
Connections:
- net Q0-DATASYNC renamed Q0-TIME_SYNC
- net Q1-TIMESYNC renamed Q1-DATA_SYNC
- removed net I0-DATA_OUT: J5.11, J5.12, U1.I0, U2.PB5
- removed net I1-CLK_SER: J5.10, J5.13, U1.I1, U2.PA5
- new net I0-CLK_SER: J5.10, J5.12, U1.I0, U2.PA5
- new net I1-DATA_OUT: J5.11, J5.13, U1.I1, U2.PB5
Changed lines of the file:
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@@
 <text x="110.49" y="92.71" size="1.778" layer="102" rot="R90">MODWIRE</text>
 <text x="243.586" y="49.784" size="1.778" layer="102" rot="R270">MODWIRE</text>
+<text x="304.8" y="59.69" size="1.778" layer="102">MODWIRE</text>
 </plain>
 <instances>
@@
 </segment>
 </net>
-<net name="Q0-DATASYNC" class="0">
+<net name="Q0-TIME_SYNC" class="0">
 <segment>
 <label x="274.32" y="71.12" size="1.778" layer="95"/>
@@
 </segment>
 </net>
-<net name="I0-DATA_OUT" class="0">
-<segment>
+<net name="I0-CLK_SER" class="0">
+<segment>
+<pinref part="J5" gate="G$1" pin="12"/>
+<wire x1="318.77" y1="53.34" x2="332.74" y2="53.34" width="0.1524" layer="91"/>
+<label x="274.32" y="55.88" size="1.778" layer="95"/>
+<wire x1="303.53" y1="55.88" x2="243.84" y2="55.88" width="0.1524" layer="91"/>
+<pinref part="J5" gate="G$1" pin="10"/>
+<pinref part="U2" gate="U" pin="PA5"/>
+<wire x1="303.53" y1="55.88" x2="303.53" y2="58.42" width="0.1524" layer="91" style="shortdash"/>
+<junction x="303.53" y="55.88"/>
+<wire x1="303.53" y1="58.42" x2="312.42" y2="58.42" width="0.1524" layer="91" style="shortdash"/>
+<wire x1="312.42" y1="58.42" x2="312.42" y2="54.61" width="0.1524" layer="91" style="shortdash"/>
+<wire x1="312.42" y1="54.61" x2="318.77" y2="54.61" width="0.1524" layer="91" style="shortdash"/>
+<wire x1="318.77" y1="54.61" x2="318.77" y2="53.34" width="0.1524" layer="91" style="shortdash"/>
+<junction x="318.77" y="53.34"/>
+</segment>
+</net>
+<net name="I1-DATA_OUT" class="0">
+<segment>
+<pinref part="J5" gate="G$1" pin="13"/>
+<wire x1="318.77" y1="55.88" x2="332.74" y2="55.88" width="0.1524" layer="91"/>
+<wire x1="318.77" y1="55.88" x2="318.77" y2="57.15" width="0.1524" layer="91" style="shortdash"/>
+<junction x="318.77" y="55.88"/>
+<wire x1="318.77" y1="57.15" x2="309.88" y2="57.15" width="0.1524" layer="91" style="shortdash"/>
+<wire x1="309.88" y1="57.15" x2="309.88" y2="54.61" width="0.1524" layer="91" style="shortdash"/>
 <label x="274.32" y="53.34" size="1.778" layer="95"/>
 <wire x1="303.53" y1="53.34" x2="243.84" y2="53.34" width="0.1524" layer="91"/>
 <pinref part="J5" gate="G$1" pin="11"/>
-<pinref part="J5" gate="G$1" pin="12"/>
-<wire x1="303.53" y1="53.34" x2="318.77" y2="53.34" width="0.1524" layer="91"/>
-<wire x1="318.77" y1="53.34" x2="332.74" y2="53.34" width="0.1524" layer="91"/>
-<junction x="318.77" y="53.34"/>
+<pinref part="U2" gate="U" pin="PB5"/>
+<wire x1="309.88" y1="54.61" x2="303.53" y2="54.61" width="0.1524" layer="91" style="shortdash"/>
+<wire x1="303.53" y1="54.61" x2="303.53" y2="53.34" width="0.1524" layer="91" style="shortdash"/>
 <junction x="303.53" y="53.34"/>
-<pinref part="U2" gate="U" pin="PB5"/>
-</segment>
-</net>
-<net name="I1-CLK_SER" class="0">
-<segment>
-<label x="274.32" y="55.88" size="1.778" layer="95"/>
-<wire x1="303.53" y1="55.88" x2="243.84" y2="55.88" width="0.1524" layer="91"/>
-<pinref part="J5" gate="G$1" pin="10"/>
-<pinref part="J5" gate="G$1" pin="13"/>
-<wire x1="303.53" y1="55.88" x2="318.77" y2="55.88" width="0.1524" layer="91"/>
-<wire x1="318.77" y1="55.88" x2="332.74" y2="55.88" width="0.1524" layer="91"/>
-<junction x="318.77" y="55.88"/>
-<junction x="303.53" y="55.88"/>
-<pinref part="U2" gate="U" pin="PA5"/>
 </segment>
 </net>
@@
 </segment>
 </net>
-<net name="Q1-TIMESYNC" class="0">
+<net name="Q1-DATA_SYNC" class="0">
 <segment>
 <label x="274.32" y="76.2" size="1.778" layer="95"/>
@@
 </segment>
 </net>
-<net name="Q0-DATASYNC" class="0">
+<net name="Q0-TIME_SYNC" class="0">
 <segment>
 <pinref part="U1" gate="G$1" pin="Q0"/>
@@
 </segment>
 </net>
-<net name="Q1-TIMESYNC" class="0">
+<net name="Q1-DATA_SYNC" class="0">
 <segment>
 <pinref part="U1" gate="G$1" pin="Q1"/>
@@
 </segment>
 </net>
-<net name="I1-CLK_SER" class="0">
+<net name="I1-DATA_OUT" class="0">
 <segment>
 <pinref part="U1" gate="G$1" pin="I1"/>
@@
 </segment>
 </net>
-<net name="I0-DATA_OUT" class="0">
+<net name="I0-CLK_SER" class="0">
 <segment>
 <pinref part="U1" gate="G$1" pin="I0"/>
