File: v2-rf-frontend-board.brd (EAGLE design)
At the start: 160 x 100 mm, 156 parts, among them J1 USB_MICROB, J2 MICROSD, J3 ROCKETNET-CONNECTOR-16M, Q1 NTR4101P, T1 ALT4532, T2 ALT4532, U1 MAX2769, U2 SAW, U3 LAN8710A-EZC, U4 7Q-16.368MBG-T, U5 XC2401, U7 LT4619_REDUCED, U8 STM32F4V, U9 LM3480IM4, X1 25 MHz, X2 BU-SMA-H

Commit message: Took a first try at Ethernet section. Tight but a little worried about trace widths.
Parts:
- R20: value 0R(board_mounted) -> 0R
- moved JP1 88.1 mm to (10.5, 13.3), turned to 90 degrees
- moved J3 81.0 mm to (16.8, 17.1), turned to 90 degrees
- moved U7 79.0 mm to (10.5, 62.5)
- moved D1 71.7 mm to (7.87, 26.4), turned to 180 degrees
- moved U3 51.6 mm to (31.4, 16.8)
- moved C21 44.2 mm to (7.05, 33.4)
- moved C1 41.4 mm to (6.99, 42.5)
- moved C28 35.0 mm to (44.6, 8.00), turned to 180 degrees
- moved R46 30.0 mm to (36.7, 17.7)
- moved R10 29.8 mm to (26.7, 14.6), turned to 270 degrees
- moved R11 29.0 mm to (25.4, 20.0), turned to 90 degrees
- moved C35 28.8 mm to (36.6, 16.5)
- moved R48 27.7 mm to (35.7, 11.7), turned to 270 degrees
- moved C34 27.2 mm to (33.3, 11.7), turned to 90 degrees
- moved C27 27.2 mm to (41.8, 11.0), turned to 180 degrees
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Connections:
- net N$59 renamed VDDA
Routing:
- net VDDA: track 0.00 -> 32.6 mm, vias 0 -> 5
- net PHY_CLK_25MHZ: track 29.9 -> 61.5 mm, vias 1 -> 3
- net 3.3VD: track 33.1 -> 58.1 mm, vias 13 -> 21
- net N$41: track 0.00 -> 22.8 mm
- net N$56: track 0.00 -> 21.9 mm, vias 0 -> 3
- net GND: track 48.3 -> 69.2 mm, vias 63 -> 53
- net N$42: track 0.00 -> 18.9 mm
- net N$44: track 0.00 -> 17.2 mm
- net OTG_FS_DP: track 0.00 -> 13.3 mm
- net ETH_RXD0: track 0.00 -> 10.7 mm, vias 0 -> 1
- net OTG_FS_VBUS: track 0.00 -> 10.5 mm
- net N$40: track 0.00 -> 10.3 mm
- net MAX_!IDLE: track 70.4 -> 60.2 mm
- net EPHY_NRST: track 0.00 -> 9.39 mm, vias 0 -> 2
- net OTG_FS_DM: track 0.00 -> 9.20 mm
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
Commit message: Ethernet basically done.
Parts:
- moved U7 32.1 mm to (8.89, 30.5)
- moved C11 27.5 mm to (92.7, 9.21)
- moved C15 27.5 mm to (95.6, 20.6)
- moved C18 27.5 mm to (87.6, 12.7)
- moved C3 27.5 mm to (81.6, 14.6)
- moved C4 27.5 mm to (81.6, 17.1)
- moved L2 27.5 mm to (104.5, 18.1)
- moved TP11 27.5 mm to (75.6, 16.2)
- moved TP15 27.5 mm to (75.6, 20.6)
- moved TP23 27.5 mm to (93.7, 10.2)
- moved TP24 27.5 mm to (75.6, 25.1)
- moved TP29 27.5 mm to (75.6, 9.21)
- moved C12 27.5 mm to (87.6, 14.0)
- moved C13 27.5 mm to (99.4, 12.4)
- moved C19 27.5 mm to (99.7, 17.8)
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Connections:
- net N$34 renamed PE0
Routing:
- net GND: track 69.2 -> 99.8 mm, vias 53 -> 61
- net MAX_CFG_SCLK: track 35.0 -> 28.2 mm
- net MAX_CFG_MOSI: track 36.1 -> 30.2 mm
- net MAX_CFG_!CS: track 34.1 -> 28.2 mm
- net N$46: track 6.63 -> 11.4 mm
- net Q1-TIMESYNC: track 40.0 -> 35.3 mm
- net ETH_MDINT: track 7.37 -> 2.75 mm
- net PE0: track 0.00 -> 4.41 mm
- net N$56: track 21.9 -> 17.7 mm
- net N$47: track 5.85 -> 9.18 mm
- net Q0-DATASYNC: track 39.3 -> 36.8 mm
- net ETH_TX_EN: track 7.23 -> 4.75 mm
- net VDDA: track 32.6 -> 30.3 mm
- net 3.3VD: track 58.1 -> 56.0 mm, vias 21 -> 22
- net ETH_TXD1: track 4.03 -> 5.96 mm
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- added copper zone on layer 1, net +5V
- added copper zone on layer 1, net 3.3VD
- added copper zone on layer 1, net VIN

Commit message: Finished board layout. Removed some test pads. Needs review.
Parts:
- removed TP26: (no value), testpad:TP06R
- removed TP36, TP37, TP38, TP42: TPTP06R, testpad:TP06R
- TP16, TP17, TP18, TP27, TP34, TP35: value TPTP06R -> (none)
- moved TP17 84.0 mm to (3.81, 28.6), flipped to the bottom
- moved TP16 80.5 mm to (14.0, 28.6), flipped to the bottom
- moved TP34 76.3 mm to (1.27, 39.4)
- moved TP18 72.3 mm to (17.1, 25.1)
- moved TP27 64.5 mm to (10.2, 28.3), flipped to the bottom
- moved TP35 64.2 mm to (18.4, 37.1)
- moved R1 61.9 mm to (3.49, 39.4)
- moved C26 57.0 mm to (3.49, 38.1)
- moved C33 56.8 mm to (9.21, 39.1)
- moved C39 53.7 mm to (18.7, 29.5)
- moved LED1 53.5 mm to (18.4, 35.9), turned to 270 degrees
- moved R6 51.0 mm to (20.0, 34.6), turned to 180 degrees
- moved C60 45.0 mm to (64.5, 37.8), turned to 270 degrees
- moved C59 43.6 mm to (70.2, 37.8), turned to 270 degrees
- moved C41 43.2 mm to (19.1, 33.0)
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Connections:
- net N$17 renamed VFB2
- net +5V: no longer TP37.TP
- net 3.3VA: no longer TP42.TP
- net 3.3VD: no longer TP38.TP
- net ANTBIAS: no longer TP26.TP
- net GND: no longer TP36.TP
Routing:
- net ETH_MDINT: track 2.75 -> 48.4 mm, vias 0 -> 4
- net GND: track 99.8 -> 141.4 mm, vias 61 -> 175
- net ETH_TXD1: track 5.96 -> 47.0 mm, vias 1 -> 2
- net EPHY_NRST: track 9.67 -> 47.6 mm, vias 2 -> 3
- net ETH_TXD0: track 5.22 -> 43.0 mm, vias 1 -> 2
- net ETH_TX_EN: track 4.75 -> 39.6 mm, vias 1 -> 2
- net !RST: track 3.22 -> 37.9 mm, vias 0 -> 2
- net ETH_MDIO: track 5.96 -> 40.4 mm, vias 0 -> 4
- net TDO: track 0.00 -> 32.5 mm, vias 0 -> 2
- net ETH_RXD1: track 9.45 -> 39.4 mm, vias 1 -> 2
- net ETH_RXD0: track 9.18 -> 37.0 mm, vias 1 -> 2
- net TDI: track 0.00 -> 27.4 mm, vias 0 -> 2
- net N$5: track 0.00 -> 25.1 mm, vias 0 -> 2
- net TCK: track 0.00 -> 24.0 mm, vias 0 -> 2
- net ETH_MDC: track 5.98 -> 29.5 mm, vias 0 -> 4
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- added copper zone on layer 2, net +5V
- added copper zone on layer 1, net ANTBIAS
- added copper zone on layer 1, net GND
- added copper zone on layer 1, net LNA2
- added copper zone on layer 1, net OTG_FS_VBUS
- added copper zone on layer 2, net OTG_FS_VBUS
- removed copper zone on layer 2, net VIN
Other:
- board size 160 x 100 mm -> 85.7 x 40.9 mm

Commit message: BOM done. Board done. All parts reviewed. Ready for review & ship.
Parts:
- R38, R39, R6: value 750 -> 68
- R40: value 300 -> 27
Changed lines of the file:
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@@
 <attribute name="VALUE" x="47.371" y="8.8265" size="0.6096" layer="27"/>
 </element>
-<element name="R38" library="rcl" package="R0402" value="750" x="49.2125" y="32.7025" smashed="yes" rot="R270">
+<element name="R38" library="rcl" package="R0402" value="68" x="49.2125" y="32.7025" smashed="yes" rot="R270">
 <attribute name="NAME" x="48.5775" y="36.0045" size="0.6096" layer="25" rot="R270"/>
 <attribute name="VALUE" x="49.2125" y="35.8775" size="0.6096" layer="27" rot="R270"/>
 </element>
-<element name="R39" library="rcl" package="R0402" value="750" x="47.9425" y="32.7025" smashed="yes" rot="R270">
+<element name="R39" library="rcl" package="R0402" value="68" x="47.9425" y="32.7025" smashed="yes" rot="R270">
 <attribute name="NAME" x="47.3075" y="36.0045" size="0.6096" layer="25" rot="R270"/>
 <attribute name="VALUE" x="47.9425" y="35.8775" size="0.6096" layer="27" rot="R270"/>
 </element>
-<element name="R40" library="rcl" package="R0402" value="300" x="50.4825" y="32.7025" smashed="yes" rot="R270">
+<element name="R40" library="rcl" package="R0402" value="27" x="50.4825" y="32.7025" smashed="yes" rot="R270">
 <attribute name="NAME" x="49.8475" y="36.0045" size="0.6096" layer="25" rot="R270"/>
 <attribute name="VALUE" x="50.4825" y="35.8775" size="0.6096" layer="27" rot="R270"/>
@@
 <attribute name="VALUE" x="17.4625" y="37.1475" size="0.6096" layer="27"/>
 </element>
-<element name="R6" library="rcl" package="R0402" value="750" x="20.0025" y="34.6075" smashed="yes" rot="R180">
+<element name="R6" library="rcl" package="R0402" value="68" x="20.0025" y="34.6075" smashed="yes" rot="R180">
 <attribute name="NAME" x="18.7325" y="35.2425" size="0.6096" layer="25"/>
 <attribute name="VALUE" x="20.0025" y="35.2425" size="0.6096" layer="27"/>

Commit message: Fixes as per design review. microUSB footprint needs help but symbol and signals OK. RF side placement adjusted but impedance 50 ohms wants 14mm wide trace. help.
Parts:
- removed J2: MICROSD, adafruit:MICROSD
- removed JP1: AUX HDR, SparkFun-Connectors:1X04_LOCK
- added R7: 100k, rcl:R0402
- added SD: CON_HIROSE_DM3D(MICROSD), con-usd-hirose-dm3-gpsboard:HIROSE_DM3D(MICRO-SD)
- added TP22, TP26, TP32, TP33: TEST-POINT, Tova:2MM-TEST-POINT
- C33, C40: device rcl:C1206 -> SparkFun-Passives:EIA6032
- J1: device SparkFun:MICRO-B-RA-TH -> con-hirose-microusb:ZX62D-B-5P8
- JTAG1: value (none) -> M05X2PTH; device microbuilder:2X05_1.27MM_SMT -> SparkFun-Connectors:AVR_ICSP
- U9: value LM3480IM4 -> LM3480IM3
- moved L6 11.0 mm to (78.8, 30.6)
- moved U5 9.68 mm to (78.8, 28.6), turned to 180 degrees
- moved C25 8.70 mm to (72.0, 27.6), turned to 90 degrees
- moved C56 7.44 mm to (81.7, 29.6), turned to 0 degrees
- moved JTAG1 7.38 mm to (62.9, 31.4)
- moved C24 7.37 mm to (73.3, 27.6), turned to 90 degrees
- moved C55 6.68 mm to (72.0, 24.3), turned to 270 degrees
- moved C57 6.10 mm to (81.7, 28.3), turned to 0 degrees
- moved J1 5.14 mm to (43.7, 40.1)
- moved C54 4.89 mm to (73.3, 24.3), turned to 270 degrees
- moved R3 2.03 mm to (21.4, 39.1)
- moved C40 1.61 mm to (16.4, 39.6)
- moved TP35 1.27 mm to (19.7, 37.1)
- moved L2 1.02 mm to (80.6, 26.4)
- moved D1 0.95 mm to (19.6, 24.9)
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Connections:
- removed net N$4: TP27.TP, U7.H5
- removed net N$46: J3.A1, JP1.1
- removed net N$47: J3.A2, JP1.2
- removed net N$48: J3.A3, JP1.3
- removed net N$50: J3.A4, JP1.4
- new net AUX1: J3.A1, TP22.1
- new net AUX2: J3.A2, TP26.1
- new net AUX3: J3.A3, TP32.1
- new net AUX4: J3.A4, TP33.1
- new net PGOOD: R7.1, TP27.TP, U7.H5
- net +5V: now also C33.P$1; no longer C33.1
- net 3.3VD: now also C40.P$1; no longer C40.1
- net GND: now also C33.P$2, C40.P$2, J1.G1, J1.G2, J1.G3, J1.G4, J1.G5, J1.G6, J1.P5, SD.G1, SD.G2, SD.G3, SD.G4, SD.P6, SD.S0, SD.S1, U3.GND, U8.PA4; no longer C33.2, C40.2, J1.5, J2.6, J2.CD1, J2.CD2, J2.MT1, J2.MT2, U3.EP1, U3.EP2, U3.EP3, U3.EP4, U3.EP5, U3.EP6, U3.EP7, U3.EP8, U3.EP9
- net N$6: now also R7.2
- net OTG_FS_DM: now also J1.P2; no longer J1.2
- net OTG_FS_DP: now also J1.P3; no longer J1.3
- net OTG_FS_VBUS: now also J1.P1; no longer J1.1
- net SDIO_CLK: now also SD.P5; no longer J2.5
- net SDIO_CMD: now also SD.P3; no longer J2.3
- net SDIO_D0: now also SD.P7; no longer J2.7
- net SDIO_D1: now also SD.P8; no longer J2.8
- net SDIO_D2: now also SD.P1; no longer J2.1
- net SDIO_D3: now also SD.P2; no longer J2.2
- net VDD: now also SD.P4; no longer J2.4
Routing:
- net GND: track 141.4 -> 101.4 mm, vias 175 -> 187
- net !RST: track 37.9 -> 53.0 mm
- net TDI: track 27.4 -> 40.2 mm
- net LNA1: track 1.46 -> 13.7 mm, vias 0 -> 2
- net PGOOD: track 0.00 -> 11.6 mm, vias 0 -> 2
- net N$46: track 11.4 -> 0.00 mm
- net LNA2: track 13.8 -> 25.2 mm
- net AUX1: track 0.00 -> 11.2 mm
- net TDO: track 32.5 -> 41.8 mm
- net AUX2: track 0.00 -> 9.23 mm
- net N$47: track 9.18 -> 0.00 mm
- net VIN: track 0.00 -> 8.76 mm
- net N$6: track 7.77 -> 16.5 mm
- net N$48: track 7.98 -> 0.00 mm
- net AUX3: track 0.00 -> 7.78 mm
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- added copper zone on layer 15, net +5V
- added copper zone on layer 15, net 3.3VA
- added copper zone on layer 15, net 3.3VD
- added copper zone on layer 16, net GND
- added copper zone on layer 2, net GND
- added copper zone on layer 15, net OTG_FS_VBUS
- removed copper zone on layer 2, net +5V
- removed copper zone on layer 2, net 3.3VA
- removed copper zone on layer 2, net 3.3VD
- removed copper zone on layer 1, net LNA2
- removed copper zone on layer 2, net OTG_FS_VBUS
Other:
- board size 85.7 x 40.9 mm -> 89.8 x 43.7 mm

Commit message: Updated microUSB symbol and library. Package not finalized.
Parts:
- removed J1: USB_MICROB, con-hirose-microusb:ZX62D-B-5P8
- added C62: 100n, rcl:C0402
- added U$1: ZX62D-B-5P8, con-hirose-microusb:ZX62D-B-5P8
- moved C57 5.08 mm to (81.7, 23.2)
- moved C56 3.59 mm to (82.2, 26.0)
- moved L2 3.06 mm to (78.4, 24.4)
- moved U5 2.96 mm to (78.3, 25.7), turned to 270 degrees
- moved L6 2.90 mm to (78.0, 27.8)
- moved X2 2.50 mm to (77.7, 33.9)
Connections:
- new net SHLD: C62.2, U$1.P$1, U$1.P$2, U$1.P$3, U$1.P$4
- net GND: now also C62.1, U$1.P5; no longer J1.G1, J1.G2, J1.G3, J1.G4, J1.G5, J1.G6, J1.P5
- net OTG_FS_DM: now also U$1.P2; no longer J1.P2
- net OTG_FS_DP: now also U$1.P3; no longer J1.P3
- net OTG_FS_VBUS: now also U$1.P1; no longer J1.P1
Routing:
- net OTG_FS_DM: track 12.4 -> 7.70 mm
- net LNA1: track 13.7 -> 8.95 mm, vias 2 -> 0
- net N$3: track 5.29 -> 1.45 mm, vias 2 -> 0
- net OTG_FS_DP: track 12.4 -> 9.09 mm
- net OTG_FS_VBUS: track 13.2 -> 10.4 mm
- net GND: track 101.4 -> 99.5 mm, vias 187 -> 185
- net ANTBIAS: track 10.3 -> 9.02 mm
- net 3.3VD: track 67.5 -> 66.3 mm
- net LNA2: track 25.2 -> 24.2 mm
- net 3.3VA: track 28.2 -> 28.0 mm, vias 6 -> 8

Commit message: Major changes to to PWR and GPS sheets. No change to board layout yet, waiting on feedback.
Parts:
- removed C57: 0.047uF, rcl:C0402
- removed TP16, TP17, TP27, TP34, TP35: (no value), testpad:TP06R
- removed U9: LM3480IM3, SparkFun-PowerIC:SOT23-3
- added L5: 9.1nH, SparkFun-Passives:C0402
- added R13: 470, rcl:R0402
- added U10: LMZ12001, SparkFun-PowerIC:TO-PMOD-7
- added U6: MAX8510EXK29+T, SparkFun-PowerIC:SC70
- C1: value 10u -> 1uF; device rcl:C1206 -> rcl:C0603
- C21: value 10u -> 220nF; device rcl:C1206 -> rcl:C0402
- C24, C54: value 0.47uF -> 100pF
- C26: value 22p -> 220nF
- C33: value 100u -> 10uF; device SparkFun-Passives:EIA6032 -> rcl:C0805
- C38: value 100n -> 100u; device rcl:C0402 -> SparkFun-Passives:EIA6032
- C39: value 22p -> 1uF; device rcl:C0402 -> rcl:C0603
- C40: value 100u -> 1uF; device SparkFun-Passives:EIA6032 -> rcl:C0603
- C41: value 100n -> 1uF; device rcl:C0402 -> rcl:C0603
- C42, C43: value 10n -> 1uF; device rcl:C0402 -> rcl:C0603
- C56: value 100pF -> 10nF
- C59, C60: value 1u -> 1uF
- L2: value 3.3nH -> 6.2nH
- R1: value 11.5k -> 10k
- R3: value 19.1k -> 3.3k
- R7: value 100k -> 240k
- U7: value LT4619_REDUCED -> MAX8510EXK29+T; device LT4619:LT4619 -> SparkFun-PowerIC:SC70
- moved C56 189.8 mm to (-21.3, -133.1)
- moved L2 181.1 mm to (-21.3, -126.7), turned to 0 degrees
- moved C55 174.3 mm to (-21.3, -122.9), turned to 0 degrees
- moved C54 171.0 mm to (-21.3, -118.1), turned to 0 degrees
- moved C25 169.0 mm to (-21.3, -113.3), turned to 0 degrees
- moved C24 165.7 mm to (-21.3, -108.5), turned to 0 degrees
- moved C60 161.3 mm to (-21.3, -98.8), turned to 0 degrees
- moved C59 160.4 mm to (-21.3, -94.0), turned to 0 degrees
- moved C19 158.3 mm to (-21.3, -103.6), turned to 0 degrees
- moved C43 157.6 mm to (-21.3, -89.2), turned to 0 degrees
- moved C42 148.1 mm to (-21.3, -84.3), turned to 0 degrees
- moved C40 120.3 mm to (-21.3, -74.7)
- moved C41 119.6 mm to (-21.3, -79.5)
- moved C33 106.5 mm to (-14.7, -64.3)
- moved U7 105.2 mm to (-21.6, -70.9), turned to 0 degrees
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Connections:
- net LNA2CHIP renamed N$1
- removed net +5V: C26.2, C33.P$1, C42.1, C60.1, U7.A10, U7.A11, U7.A12, U7.B10, U7.B11, U7.B12, U7.C10, U7.C11, U7.C12, U7.D10, U7.D11, U7.D12, U9.2
- removed net 3.3VA: C12.1, C13.1, C15.1, C16.1, C18.1, C43.1, C5.1, C56.1, C57.1, C59.1, C6.1, C8.1, U1.11, U1.13, U1.23, U1.4, U5.1, U9.1
- removed net ANTBIAS: C24.1, C25.1, C54.1, C55.1, L2.2, U1.3
- removed net LNA1: C19.2, U5.2
- removed net LNA1CHIP: C19.1, U1.27
- removed net PGOOD: R7.1, TP27.TP, U7.H5
- removed net VFB2: C39.1, R3.1, TP35.TP, U7.K6
- new net 2.85VA: C12.1, C13.1, C15.1, C16.1, C18.1, C42.1, C43.2, C5.1, C6.1, C8.1, U1.11, U1.13, U1.23, U1.4, U7.5
- new net 2.85VD: C14.1, C17.1, C58.1, C59.1, C60.2, C7.1, C9.1, R5.2, U1.14, U1.19, U4.4, U6.5
- new net N$10: R7.2, U10.2
- new net N$13: C43.1, U7.4
- new net N$17: C19.1, C22.1, C24.2, C25.2
- new net N$21: C54.1, C55.1, L6.4
- new net N$22: C55.2, L2.1, L5.2
- new net N$23: R13.1, U1.3
- new net N$4: C56.1, R13.2, U5.1
- net 3.3VD: now also C26.1, C38.P$1, C39.1, C40.1, C41.1, R1.2, U10.7, U6.1, U6.3, U7.1, U7.3; no longer C14.1, C17.1, C39.2, C40.P$1, C58.1, C7.1, C9.1, R5.2, U1.14, U1.19, U4.4, U7.A1, U7.A2, U7.A3, U7.B1, U7.B2, U7.B3, U7.C1, U7.C2, U7.C3, U7.D1, U7.D2, U7.D3
- net GND: now also C33.2, C38.P$2, C39.2, C40.2, L5.1, R3.1, U10.4, U10.EP, U6.2, U7.2; no longer C24.2, C25.2, C33.P$2, C38.2, C40.P$2, C43.2, C54.2, C55.2, C57.2, C60.2, R1.2, R3.2, U7.A4, U7.A5, U7.A6, U7.A7, U7.A8, U7.A9, U7.B4, U7.B5, U7.B6, U7.B7, U7.B8, U7.B9, U7.C4, U7.C5, U7.C6, U7.C7, U7.C8, U7.C9, U7.D4, U7.D5, U7.D6, U7.D7, U7.D8, U7.D9, U7.E1, U7.E10, U7.E11, U7.E12, U7.E2, U7.E3, U7.E4, U7.E5, U7.E6, U7.E7, U7.E8, U7.E9, U7.F1, U7.F10, U7.F11, U7.F12, U7.F2, U7.F3, U7.F4, U7.F5, U7.F7, U7.F8, U7.F9, U7.G1, U7.G10, U7.G11, U7.G12, U7.G2, U7.G3, U7.G4, U7.G5, U7.G6, U7.G7, U7.G8, U7.G9, U7.H1, U7.H11, U7.H12, U7.H2, U7.H4, U7.H6, U7.H7, U7.H8, U7.H9, U7.J6, U7.J7, U9.3
- net LNA2: no longer C22.1, L2.1
- net N$14: now also L2.2, U5.4; no longer C41.1, U7.K5
- net N$16: now also C60.1, U6.4; no longer C38.1, U7.K8
- net N$2: now also C19.2, U1.27; no longer TP17.TP, U7.H10
- net N$3: now also C25.1, U5.2; no longer L6.4, U5.4
- net N$5: now also C24.1, C54.2; no longer C26.1, R1.1, TP34.TP, U7.K7
- net N$6: now also C21.1, U10.5; no longer R7.2, U7.F6, U7.J8
- net N$7: now also C26.2, R1.1, R3.2, U10.6; no longer TP16.TP, U7.H3
- net VIN: now also C33.1, R7.1, U10.1; no longer C21.1, U7.J1, U7.J10, U7.J11, U7.J12, U7.J2, U7.J3, U7.J4, U7.K1, U7.K10, U7.K11, U7.K12, U7.K2, U7.K3, U7.K4, U7.K9, U7.L1, U7.L10, U7.L11, U7.L12, U7.L2, U7.L3, U7.L4, U7.L5, U7.L8, U7.L9, U7.M1, U7.M10, U7.M11, U7.M12, U7.M2, U7.M3, U7.M4, U7.M5, U7.M6, U7.M7, U7.M8, U7.M9
Routing:
- net GND: track 99.5 -> 71.2 mm, vias 185 -> 180
- net 3.3VA: track 28.0 -> 0.00 mm, vias 8 -> 0
- net N$5: track 25.1 -> 0.00 mm, vias 2 -> 0
- net VFB2: track 24.1 -> 0.00 mm, vias 3 -> 0
- net 3.3VD: track 66.3 -> 48.2 mm, vias 25 -> 19
- net 2.85VA: track 0.00 -> 17.4 mm, vias 0 -> 4
- net N$14: track 17.2 -> 0.00 mm, vias 2 -> 0
- net N$16: track 17.1 -> 0.00 mm, vias 2 -> 0
- net N$6: track 16.5 -> 0.00 mm, vias 2 -> 0
- net LNA2: track 24.2 -> 11.2 mm
- net PGOOD: track 11.6 -> 0.00 mm, vias 2 -> 0
- net +5V: track 10.3 -> 0.00 mm, vias 9 -> 5
- net ANTBIAS: track 9.02 -> 0.00 mm, vias 2 -> 0
- net LNA1: track 8.95 -> 0.00 mm
- net 2.85VD: track 0.00 -> 8.78 mm, vias 0 -> 3
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- added copper zone on layer 15, net 2.85VA
- removed copper zone on layer 15, net 3.3VA
