File: v2-rf-frontend-board.brd (EAGLE design)
At the start: 89.8 x 43.7 mm, 153 parts, among them J3 ROCKETNET-CONNECTOR-16M, Q1 NTR4101P, T1 ALT4532, T2 ALT4532, U1 MAX2769, U10 LMZ12001, U2 SAW, U3 LAN8710A-EZC, U4 7Q-16.368MBG-T, U5 XC2401, U6 MAX8510EXK29+T, U7 MAX8510EXK29+T, U8 STM32F4V, X1 25 MHz, X2 BU-SMA-H

Commit message: Made a capacitor options footprint and symbol for the 'do not populate' choice capacitor hack.
Parts:
- removed C25, C54, C55: 100pF, rcl:C0402
- C19, C22, C24: device rcl:C0402 -> wicker:CAP-OPTION
- moved C22 190.6 mm to (-31.0, -138.4), turned to 0 degrees
- moved C19 35.2 mm to (-26.4, -138.4)
- moved C24 33.2 mm to (-35.6, -138.4)
Connections:
- removed net N$1: C22.2, U1.25
- new net N$25: C19.2, C22.2
- net N$17: now also C19.3, U1.25; no longer C19.1, C22.1, C24.2, C25.2
- net N$2: now also C19.1; no longer C19.2
- net N$21: now also C24.2; no longer C54.1, C55.1
- net N$22: now also C24.3; no longer C55.2
- net N$3: now also C22.1; no longer C25.1
- net N$5: now also C22.3; no longer C54.2
Changed lines of the file:
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@@
 <attribute name="VALUE" x="73.5965" y="33.274" size="0.6096" layer="27" rot="R90"/>
-</element>
-<element name="C22" library="rcl" package="C0402" value="100pF" x="82.55" y="14.605" smashed="yes" rot="R180">
-<attribute name="NAME" x="81.915" y="14.9225" size="0.6096" layer="25" rot="R180"/>
-<attribute name="VALUE" x="83.185" y="14.2875" size="0.6096" layer="27"/>
 </element>
 <element name="X1" library="crystal" package="CTS406" value="25 MHz" x="46.6725" y="3.175" smashed="yes" rot="R180">
@@
 <element name="C59" library="rcl" package="C0603" value="1uF" x="-21.336" y="-93.98"/>
 <element name="C60" library="rcl" package="C0603" value="1uF" x="-21.336" y="-98.806"/>
-<element name="C19" library="rcl" package="C0402" value="100pF" x="-21.336" y="-103.632"/>
-<element name="C24" library="rcl" package="C0402" value="100pF" x="-21.336" y="-108.458"/>
-<element name="C25" library="rcl" package="C0402" value="100pF" x="-21.336" y="-113.284"/>
-<element name="C54" library="rcl" package="C0402" value="100pF" x="-21.336" y="-118.11"/>
-<element name="C55" library="rcl" package="C0402" value="100pF" x="-21.336" y="-122.936"/>
 <element name="L2" library="SparkFun-Passives" package="C0402" value="6.2nH" x="-21.336" y="-126.746"/>
 <element name="L5" library="SparkFun-Passives" package="C0402" value="9.1nH" x="-21.336" y="-129.032"/>
 <element name="C56" library="rcl" package="C0402" value="10nF" x="-21.336" y="-133.096"/>
 <element name="R13" library="rcl" package="R0402" value="470" x="-21.336" y="-137.922"/>
+<element name="C19" library="wicker" package="CAP-OPTION" value="100pF" x="-26.416" y="-138.43"/>
+<element name="C22" library="wicker" package="CAP-OPTION" value="100pF" x="-30.988" y="-138.43"/>
+<element name="C24" library="wicker" package="CAP-OPTION" value="100pF" x="-35.56" y="-138.43"/>
 </elements>
 <signals>
@@
 <wire x1="80.375" y1="13.605" x2="79.6025" y2="13.605" width="0" layer="19" extent="1-1"/>
 </signal>
-<signal name="N$1">
-<contactref element="C22" pad="2"/>
-<contactref element="U1" pad="25"/>
-<wire x1="79.6025" y1="14.605" x2="81.9" y2="14.605" width="0" layer="19" extent="1-1"/>
-</signal>
 <signal name="N$2">
-<contactref element="C19" pad="2"/>
 <contactref element="U1" pad="27"/>
-<wire x1="79.6025" y1="15.605" x2="-20.686" y2="-103.632" width="0" layer="19" extent="1-1"/>
+<contactref element="C19" pad="1"/>
+<wire x1="79.6025" y1="15.605" x2="-26.416" y2="-136.764" width="0" layer="19" extent="1-1"/>
 </signal>
 <signal name="N$4">
@@
 <wire x1="77.9399" y1="25.9461" x2="-21.986" y2="-133.096" width="0" layer="19" extent="1-1"/>
 </signal>
-<signal name="N$17">
+<signal name="N$3">
+<contactref element="U5" pad="2"/>
 <contactref element="C22" pad="1"/>
-<contactref element="C19" pad="1"/>
-<contactref element="C25" pad="2"/>
+<wire x1="77.9399" y1="25.4889" x2="-30.988" y2="-136.764" width="0" layer="19" extent="1-1"/>
+</signal>
+<signal name="N$5">
+<contactref element="C22" pad="3"/>
+<contactref element="C24" pad="1"/>
+<wire x1="-30.988" y1="-139.3594" x2="-35.56" y2="-136.764" width="0" layer="19" extent="1-1"/>
+</signal>
+<signal name="N$21">
+<contactref element="L6" pad="4"/>
 <contactref element="C24" pad="2"/>
-<wire x1="-20.686" y1="-108.458" x2="-20.686" y2="-113.284" width="0" layer="19" extent="1-1"/>
-<wire x1="-21.986" y1="-103.632" x2="-20.686" y2="-108.458" width="0" layer="19" extent="1-1"/>
-<wire x1="83.2" y1="14.605" x2="-21.986" y2="-103.632" width="0" layer="19" extent="1-1"/>
-</signal>
-<signal name="N$3">
-<contactref element="C25" pad="1"/>
-<contactref element="U5" pad="2"/>
-<wire x1="77.9399" y1="25.4889" x2="-21.986" y2="-113.284" width="0" layer="19" extent="1-1"/>
-</signal>
-<signal name="N$5">
-<contactref element="C24" pad="1"/>
-<contactref element="C54" pad="2"/>
-<wire x1="-21.986" y1="-108.458" x2="-20.686" y2="-118.11" width="0" layer="19" extent="1-1"/>
-</signal>
-<signal name="N$21">
-<contactref element="C55" pad="1"/>
-<contactref element="C54" pad="1"/>
-<contactref element="L6" pad="4"/>
-<wire x1="-21.986" y1="-118.11" x2="-21.986" y2="-122.936" width="0" layer="19" extent="1-1"/>
-<wire x1="78.329" y1="27.313" x2="-21.986" y2="-118.11" width="0" layer="19" extent="1-1"/>
+<wire x1="78.329" y1="27.313" x2="-35.56" y2="-138.064" width="0" layer="19" extent="1-1"/>
 </signal>
 <signal name="N$14">
@@
 </signal>
 <signal name="N$22">
-<contactref element="C55" pad="2"/>
 <contactref element="L2" pad="1"/>
 <contactref element="L5" pad="2"/>
+<contactref element="C24" pad="3"/>
+<wire x1="-20.686" y1="-129.032" x2="-35.56" y2="-139.3594" width="0" layer="19" extent="1-1"/>
 <wire x1="-21.986" y1="-126.746" x2="-20.686" y2="-129.032" width="0" layer="19" extent="1-1"/>
-<wire x1="-20.686" y1="-122.936" x2="-21.986" y2="-126.746" width="0" layer="19" extent="1-1"/>
 </signal>
 <signal name="N$23">
@@
 <wire x1="77.6525" y1="17.055" x2="-21.986" y2="-137.922" width="0" layer="19" extent="1-1"/>
 </signal>
+<signal name="N$17">
+<contactref element="U1" pad="25"/>
+<contactref element="C19" pad="3"/>
+<wire x1="79.6025" y1="14.605" x2="-26.416" y2="-139.3594" width="0" layer="19" extent="1-1"/>
+</signal>
+<signal name="N$25">
+<contactref element="C19" pad="2"/>
+<contactref element="C22" pad="2"/>
+<wire x1="-26.416" y1="-138.064" x2="-30.988" y2="-138.064" width="0" layer="19" extent="1-1"/>
+</signal>
 </signals>
