File: v2-rf-frontend-board.brd (EAGLE design)
At the start: 89.8 x 43.7 mm, 129 parts, among them J3 ROCKETNET-CONNECTOR-16M, Q1 NTR4101P, T1 ALT4532, T2 ALT4532, U1 MAX2769, U10 LMZ12001, U3 LAN8710A-EZC, U4 7Q-16.368MBG-T, U5 XC2401, U6 MAX8510EXK29+T, U7 MAX8510EXK29+T, U8 STM32F4V, X1 25 MHz, X2 BU-SMA-H

Commit message: Cleanup on Jenner's fine work. Mostly adding polygons to power signals, some additional caps, moving parts around for optimal placement, added mounting holes, made polygon lines consistent. NOT DONE YET, still have RF cleanup and Ethernet cleanup to do.
Parts:
- removed D1: 25V 1A, SparkFun-DiscreteSemi:SMA-DIODE_ALT
- removed JTAG1: M05X2PTH, SparkFun-Connectors:AVR_ICSP
- removed TP18, TP2: (no value), testpad:TP06R
- added C25, C54, C55: 100n, rcl_custom:0402-B-NOSILK
- added D2: DIODE-0603, diode-0603:0603-B-NOSILK-DIODE
- added J1: 1.27MM-SWD-CONNECTOR, con-swd:1.27MM_2X5
- added U$1, U$12, U$14, U$18: #4-BARE_MOUNTING_HOLE/.300, mount:#4/.300-BARE+STD_NUT_OR_STAR_WASHER
- C1: device rcl_custom:0603-C-NOSILK -> rcl_custom:0805-B-NOSILK
- C26: value 220nF 10V -> 220nF
- C38: value 100u 10V -> 100u
- C39: value 1uF 10V -> 1uF; device rcl_custom:0603-C-NOSILK -> rcl_custom:0603-B-NOSILK
- C40, C41, C42, C59: value 1uF 10V -> 1u; device rcl_custom:0603-C-NOSILK -> rcl_custom:0603-B-NOSILK
- C43, C60: value 1uF 10V -> 10n; device rcl_custom:0603-C-NOSILK -> rcl_custom:0402-B-NOSILK
- moved R6 18.0 mm to (25.1, 41.1)
- moved LED1 17.8 mm to (22.9, 41.1)
- moved C38 14.6 mm to (22.9, 32.3), turned to 90 degrees
- moved TP22 12.8 mm to (1.78, 16.0)
- moved C1 12.8 mm to (6.86, 32.3), turned to 90 degrees
- moved C33 12.7 mm to (4.83, 32.3)
- moved U10 12.3 mm to (13.7, 38.1), turned to 0 degrees
- moved TP26 12.0 mm to (1.78, 17.8)
- moved TP32 11.5 mm to (1.78, 19.8)
- moved TP33 10.8 mm to (1.78, 21.6)
- moved J3 8.47 mm to (5.33, 18.8)
- moved R3 8.16 mm to (16.3, 25.7), turned to 90 degrees
- moved C26 7.12 mm to (16.8, 27.2)
- moved C39 6.84 mm to (20.3, 32.3), turned to 90 degrees
- moved R7 5.57 mm to (11.2, 27.9)
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Connections:
- net !RST: now also J1.!RESET; no longer JTAG1.10, TP2.TP
- net 2.85VA: now also C55.1
- net 3.3VD: now also C54.1, J1.VTREF; no longer JTAG1.1
- net GND: now also C25.2, C54.2, C55.2, J1.GND, J1.GND@2, J1.GNDDET; no longer JTAG1.3, JTAG1.5, JTAG1.9
- net OTG_FS_VBUS: now also D2.ANODE; no longer D1.A
- net TCK: now also J1.SWDCLK; no longer JTAG1.4
- net TDI: now also J1.NC; no longer JTAG1.8
- net TDO: now also J1.SWO; no longer JTAG1.6
- net TMS: now also J1.SWDIO; no longer JTAG1.2
- net VIN: now also C25.1, D2.CATHODE; no longer D1.C, TP18.TP
Routing:
- net 3.3VD: track 80.0 -> 51.1 mm, vias 37 -> 41
- net VIN: track 16.7 -> 1.48 mm, vias 4 -> 8
- net N$26: track 5.94 -> 14.5 mm
- net N$27: track 5.79 -> 14.3 mm
- net OTG_FS_VBUS: track 43.7 -> 52.1 mm, vias 3 -> 7
- net N$20: track 5.59 -> 14.0 mm
- net N$8: track 5.52 -> 13.9 mm
- net AUX1: track 11.2 -> 3.23 mm
- net GND: track 42.3 -> 35.7 mm, vias 415 -> 257
- net N$7: track 11.1 -> 4.44 mm
- net AUX2: track 9.23 -> 3.03 mm
- net AUX3: track 7.78 -> 3.03 mm
- net !RST: track 34.8 -> 30.8 mm, vias 2 -> 1
- net 2.85VA: track 25.7 -> 21.8 mm, vias 5 -> 9
- net ETH_MDIO: track 40.6 -> 36.7 mm, vias 4 -> 2
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- added copper zone on layer 1, net 2.85VA
- added copper zone on layer 1, net 2.85VD
- added copper zone on layer 1, net 3.3VD
- added copper zone on layer 1, net OTG_FS_VBUS
- added copper zone on layer 16, net OTG_FS_VBUS
- added copper zone on layer 1, net VIN
- added copper zone on layer 16, net VIN
Other:
- board size 89.8 x 43.7 mm -> 89.7 x 43.9 mm

Commit message: Beeeeg changes to GPS board. Caught many small mistakes in STM and LAN wiring and footprints, fixed. Better layout of magnetics, replumbed the lines between STM32 and LAN, and more. Passes ERC and DRC, although still not quite done: want to double check SAW filters, find a smaller 50 MHz clock, and add other GPS interface.
Parts:
- removed C27: 22uF/6.3V, rcl_custom:1206-C
- removed C58: 470nF 10V, rcl_custom:0603-C-NOSILK
- removed LED2: BLUE, led:CHIP-LED0603
- removed LED4: RED, led:CHIP-LED0603
- removed TP1: (no value), testpad:TP06R
- added C57: 470n, rcl_custom:0402-C-NOSILK
- added C61: 100n, rcl_custom:0402-C-NOSILK
- added CD1: 6NC2_CLOCK_DRIVER, gogo:7X5MM_CLOCK_DRIVER
- added LED6: (no value), led:CHIPLED_0603
- added R14, R19: 10k, rcl_custom:0402-C-NOSILK
- added R17: 1k, rcl_custom:0402-C-NOSILK
- added TP2, TP4, TP5: (no value), testpad:TP06R
- C1: value 1uF 50V -> 1u 50V
- C11: value DNP -> 100n
- C12, C14, C16, C17, C19, C22, C24, C6, C8: value 100pF 10V -> 100p
- C13, C15, C18, C45, C46, C47, C48, C49, C5, C50, C7, C9: value 100nF 10V -> 100n
- C21: value 220nF 10V -> 220n
- C23, C28: value 22uF/6.3V -> 22u
- C25: value 100n -> 100n 50V
- C29, C30: value 18pF 10V -> 10p
- C3: value 27pF 10V -> 27p
- C31, C32, C35: value 100nF 10V -> 10n
- C33: value 10uF 50V -> 10u 50V
- C34: value 100nF 10V -> 470p
- C36: value 10uF/6.3V -> 100n; device rcl_custom:1206-C -> rcl_custom:0402-C-NOSILK
- C37: value 100nF 10V -> 22n
- C4: value 470pF 10V -> 470p
- C44: value 1nF 10V -> 100n
- C51, C52: value 2.2uF 10V -> 2.2u
- C53: value 100nF 10V -> 2.2u
- C56: value 10nF 10V -> 10n
- C62: value 100n 10V -> 100n 50V
- LED3: value GREEN -> (none); device led:CHIP-LED0603 -> apdm:PLCC-6
- R10, R11: value 75 -> 50
- R15: value 150 -> 47k
- R20: value 0R -> NP
- R22, R23, R24, R25: value 49.9R/1% -> 49.9 1%
- R27, R42, R43, R44, R45, R46, R47, R48: value 4.7k -> 10k
- R29: value 12.1k/1% -> 12.1k
- U2: value STM32F4V -> STM32F4V_100PIN_GPSBOARD
- moved R20 37.2 mm to (56.9, 8.38), turned to 180 degrees
- moved C28 28.5 mm to (23.0, 26.2), turned to 90 degrees
- moved L3 27.4 mm to (20.6, 26.4), turned to 90 degrees
- moved Q1 25.1 mm to (23.0, 40.3), turned to 270 degrees
- moved C23 24.5 mm to (18.5, 24.3), turned to 90 degrees
- moved R12 24.4 mm to (20.8, 40.3), turned to 270 degrees
- moved C11 22.2 mm to (54.7, 9.53), turned to 180 degrees
- moved C20 21.4 mm to (25.4, 39.5), turned to 90 degrees
- moved R9 20.0 mm to (68.3, 20.1)
- moved C10 18.8 mm to (26.5, 39.5), turned to 90 degrees
- moved R15 18.7 mm to (13.6, 4.06), turned to 90 degrees
- moved C36 15.2 mm to (18.8, 7.37), turned to 180 degrees
- moved C51 14.9 mm to (44.3, 29.3)
- moved C52 14.9 mm to (58.7, 25.4)
- moved LED1 13.0 mm to (25.8, 28.4), turned to 0 degrees
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- renumbered U8 to U2
Connections:
- net VDD renamed SD-VDD
- removed net ETH_CRX_DV: R45.2, U2.PA7, U3.15
- removed net LED3: LED3.A, U2.PD13
- removed net LED4: LED4.A, U2.PD14
- removed net N$56: C37.2, R20.1, T1.3, T2.3
- removed net N$63: R15.2, U3.18
- removed net PHY_CLK_25MHZ: C11.1, U2.PA8, U3.5
- new net ETH_CRS_DV: R45.2, U2.32, U3.15
- new net ETH_RMII_REF_CLK: CD1.3, R20.2, U2.24, U3.5
- new net MCO1-ETH-CLK: R20.1, U2.67
- new net N$1: R14.1, U3.2
- new net N$23: LED6.A, R17.1
- new net N$24: R17.2, U3.3
- new net N$34: LED3.5, U2.60
- new net N$37: LED3.1, R40.2
- new net N$38: SD1.S1, TP2.TP
- new net N$39: CD1.1, R15.1
- new net N$43: C52.2, U2.49
- new net N$45: C51.2, U2.73
- net !RST: now also U2.14; no longer U2.NRST
- net 2.85VD: now also C57.1; no longer C58.1
- net 3.3VD: now also C11.2, C36.2, C61.2, CD1.4, R15.2, TP4.TP, TP5.TP, U2.100, U2.11, U2.19, U2.21, U2.22, U2.28, U2.50, U2.6, U2.75; no longer C27.2, C51.2, C52.2, U2.VCAP1, U2.VCAP2, U2.VDD1, U2.VDD2, U2.VDD3, U2.VDD4, U2.VDD5, U2.VDD6
- net ANTFLAG: now also U2.36; no longer U2.PB1
- net EPHY_NRST: now also U2.84; no longer C36.2, U2.PA1
- net ETH_MDC: now also U2.16; no longer U2.PC1
- net ETH_MDINT: now also U2.26, U3.18; no longer R15.1, U2.PA3
- net ETH_MDIO: now also U2.25; no longer U2.PA2
- net ETH_RXD0: now also U2.33; no longer U2.PC4
- net ETH_RXD1: now also U2.34; no longer U2.PC5
- net ETH_TXD0: now also U2.51; no longer U2.PB12
- net ETH_TXD1: now also U2.52; no longer U2.PB13
- net ETH_TX_EN: now also U2.48; no longer U2.PB11
- net GND: now also C11.1, C57.2, C61.1, CD1.2, L6.B, L6.C, L6.E, L7.B, L7.C, L7.E, LED6.C, R19.2, U2.10, U2.20, U2.27, U2.74, U2.99; no longer C27.1, C58.2, L6.2, L6.3, L6.5, L7.2, L7.3, L7.5, SD1.S1, U2.PA4, U2.PDR_ON, U2.VSS1, U2.VSS2, U2.VSS3
- net I0-DATA_OUT: now also U2.91; no longer U2.PB5
- net I1-CLK_SER: now also U2.30; no longer U2.PA5
- net LD: now also U2.37; no longer U2.PB2
- net LED2: now also LED3.2, U2.61; no longer LED2.A, U2.PD11
- net LNA2: now also L6.A; no longer L6.1
- net LNAOUT: now also L7.A; no longer L7.1
- net MAX_!IDLE: now also U2.42; no longer U2.PE11
- net MAX_!SHDN: now also U2.41; no longer U2.PE10
- net MAX_CFG_!CS: now also U2.43; no longer U2.PE12
- net MAX_CFG_MOSI: now also U2.45; no longer U2.PE14
- net MAX_CFG_SCLK: now also U2.44; no longer U2.PE13
- net MIXIN: now also L7.D; no longer L7.4
- net N$11: now also LED3.6, U2.58; no longer LED2.C, R40.2
- net N$12: now also LED3.4, R39.2; no longer LED3.C, R38.2
- net N$18: now also LED3.3, R38.2; no longer LED4.C, R39.2
- net N$21: now also L6.D; no longer L6.4
- net N$9: now also R19.1, U2.94; no longer TP1.TP, U2.BOOT0
- net OSC_IN: now also U2.12; no longer U2.PH0
- net OSC_OUT: now also U2.13; no longer U2.PH1
- net OTG_FS_DM: now also U2.70; no longer U2.PA11
- net OTG_FS_DP: now also U2.71; no longer U2.PA12
- net OTG_FS_VBUS: now also U2.68; no longer U2.PA9
- net PE0: now also U2.81; no longer U2.PE0
- net Q0-DATASYNC: now also U2.38; no longer U2.PE7
- net Q1-TIMESYNC: now also U2.40; no longer U2.PE9
- net SDIO_CLK: now also U2.80; no longer U2.PC12
- net SDIO_CMD: now also U2.83; no longer U2.PD2
- net SDIO_D0: now also U2.65; no longer U2.PC8
- net SDIO_D1: now also U2.66; no longer U2.PC9
- net SDIO_D2: now also U2.78; no longer U2.PC10
- net SDIO_D3: now also U2.79; no longer U2.PC11
- net TCK: now also U2.76; no longer U2.PA14
- net TDI: now also U2.77; no longer U2.PA15
- net TDO: now also U2.89; no longer U2.PB3
- net TMS: now also U2.72; no longer U2.PA13
- net VDDA: now also C37.2, R14.2, T1.3, T2.3; no longer R20.2
- net XTAL: no longer C11.2
Routing:
- net PHY_CLK_25MHZ: track 77.7 -> 0.00 mm, vias 5 -> 0
- net ETH_RMII_REF_CLK: track 0.00 -> 47.6 mm, vias 0 -> 2
- net ETH_CRS_DV: track 0.00 -> 32.6 mm, vias 0 -> 2
- net ETH_CRX_DV: track 31.0 -> 0.00 mm, vias 3 -> 0
- net EPHY_NRST: track 47.6 -> 18.9 mm, vias 3 -> 0
- net MCO1-ETH-CLK: track 0.00 -> 25.9 mm, vias 0 -> 4
- net SD-VDD: track 24.8 -> 0.00 mm, vias 2 -> 0
- net PE0: track 10.7 -> 33.6 mm
- net GND: track 35.7 -> 15.0 mm, vias 257 -> 156
- net N$56: track 17.9 -> 0.00 mm, vias 3 -> 0
- net N$24: track 0.00 -> 16.0 mm, vias 0 -> 2
- net 2.85VA: track 21.8 -> 6.06 mm, vias 9 -> 12
- net ETH_MDINT: track 48.4 -> 36.3 mm, vias 4 -> 2
- net MAX_!IDLE: track 57.3 -> 46.1 mm, vias 3 -> 1
- net 2.85VD: track 13.5 -> 2.92 mm, vias 9 -> 13
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- added copper zone on layer 1, net SD-VDD
- added copper zone on layer 1, net VDDA
- added copper zone on layer 16, net VDDA
Other:
- board size 89.7 x 43.9 mm -> 86.6 x 43.9 mm

Commit message: Switched to the KSZ8081RNA PHY layer IC, the best PHY layer IC ever. I'm sure we'll hate it later, but for now, it's great. New library and datasheet and schematic, still need to wire it up.
Parts:
- removed C36: 100n, rcl_custom:0402-C-NOSILK
- removed C53: 2.2u, rcl_custom:0402-C-NOSILK
- removed CD1: 6NC2_CLOCK_DRIVER, gogo:7X5MM_CLOCK_DRIVER
- removed R14, R27, R28, R44, R45, R46, R47, R48: 10k, rcl_custom:0402-C-NOSILK
- removed R16: 2.2k, rcl_custom:0402-C-NOSILK
- removed R20: NP, rcl_custom:0402-C-NOSILK
- removed R22, R23, R24, R25: 49.9 1%, rcl_custom:0402-C-NOSILK
- removed R29: 12.1k, rcl_custom:0402-C-NOSILK
- added C27: 100n, rcl_custom:0402-C-NOSILK
- C23: value 22u -> 100n; device rcl_custom:1206-C -> rcl_custom:0402-C-NOSILK
- C31: value 10n -> 2.2u
- C32: value 10n -> 22u; device rcl_custom:0402-C-NOSILK -> rcl_custom:1206-C
- C34: value 470p -> 100n
- C35: value 10n -> 100n
- C37: value 22n -> 100n
- C44: value 100n -> 1n 2kv
- LED6: value (none) -> GRN
- R10, R11: value 50 -> 75
- R15: value 47k -> 6.49k
- R42, R43: value 10k -> 1k
- U3: value LAN8710A-EZC -> KSZ8081; device OLIMEX_IC:QFN-32(DRILLS) -> ksz8081:QFN-24
- moved C23 16.1 mm to (22.9, 8.76), turned to 0 degrees
- moved C35 12.3 mm to (19.7, 8.89)
- moved R15 12.0 mm to (24.6, 8.64), turned to 0 degrees
- moved C32 5.85 mm to (22.6, 7.24), turned to 0 degrees
- moved U3 5.18 mm to (21.3, 12.8), turned to 270 degrees
- moved C34 2.05 mm to (25.5, 6.35), turned to 0 degrees
- moved C31 1.45 mm to (26.0, 7.37), turned to 0 degrees
Connections:
- removed net N$55: R29.2, U3.32
- removed net N$58: C34.2, C53.2, U3.6
- removed net PHYAD0: R46.1, U3.13
- removed net PHYAD1: R47.1, U3.7
- removed net PHYAD2: R48.1, U3.8
- removed net RMIISEL: R27.2, U3.9
- new net N$46: R15.2, U3.9
- new net VDDA_3.3: C32.2, C34.2, L3.1, U3.2
- net 3.3VD: now also C27.2, R17.2, U3.14; no longer C35.1, C36.2, CD1.4, R15.2, R16.1, R27.1, R28.1, R44.1, R45.1, U3.12
- net EPHY_NRST: now also U3.24; no longer R28.2, U3.19
- net ETH_CRS_DV: no longer R45.2
- net ETH_MDC: now also U3.11; no longer U3.17
- net ETH_MDINT: now also R43.2; no longer R16.2
- net ETH_MDIO: now also R42.2, U3.10; no longer R44.2, U3.16
- net ETH_RMII_REF_CLK: now also U3.16; no longer CD1.3, R20.2, U3.5
- net ETH_RXD0: now also U3.13; no longer R42.2, U3.11
- net ETH_RXD1: now also U3.12; no longer R43.2, U3.10
- net ETH_TXD0: now also U3.20; no longer U3.22
- net ETH_TXD1: now also U3.21; no longer U3.23
- net ETH_TX_EN: now also U3.19; no longer U3.21
- net GND: now also C23.2, C27.1, C31.2, C35.1, R15.1, U3.22, U3.PAD; no longer C23.1, C31.1, C35.2, C36.1, C53.1, CD1.2, LED6.C, R29.1, R46.2, R47.2, R48.2, U3.24, U3.25, U3.GND
- net MCO1-ETH-CLK: now also U3.8; no longer R20.1
- net N$1: now also C23.1, C31.1, U3.1; no longer R14.1, U3.2
- net N$24: now also C35.2, T1.3; no longer R17.2, U3.3
- net N$39: now also LED6.C, U3.23; no longer CD1.1, R15.1
- net N$40: now also U3.3; no longer R22.1, U3.30
- net N$41: now also U3.6; no longer R25.1, U3.29
- net N$42: now also U3.5; no longer R24.1, U3.28
- net N$44: now also U3.4; no longer R23.1, U3.31
- net VDDA: no longer C23.2, C31.2, C32.2, L3.1, R14.2, R22.2, R23.2, R24.2, R25.2, T1.3, U3.1, U3.27
Routing:
- net VDDA: track 48.6 -> 1.08 mm, vias 8 -> 2
- net ETH_RMII_REF_CLK: track 47.6 -> 4.16 mm, vias 2 -> 0
- net N$41: track 17.2 -> 0.00 mm
- net N$42: track 15.5 -> 0.00 mm
- net 3.3VD: track 49.7 -> 35.1 mm, vias 48 -> 41
- net N$24: track 16.0 -> 3.24 mm, vias 2 -> 0
- net N$44: track 12.1 -> 0.00 mm
- net N$40: track 11.3 -> 0.00 mm
- net N$1: track 6.53 -> 0.00 mm, vias 2 -> 0
- net ETH_RXD0: track 37.2 -> 30.9 mm
- net ETH_RXD1: track 37.1 -> 31.6 mm
- net GND: track 15.0 -> 10.8 mm, vias 156 -> 154
- net RMIISEL: track 4.10 -> 0.00 mm
- net N$39: track 3.73 -> 0.00 mm
- net PHYAD2: track 3.37 -> 0.00 mm
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
Commit message: PHY layout, plus connection to COTS GPS board via a 0.1" header that could also be (shock!) an FTDI cable. Last thing left: SAW filters!
Parts:
- removed C31: 2.2u, rcl_custom:0402-C-NOSILK
- added C36: 2.2u, rcl_custom:0603-B-NOSILK
- added JP3: (no value), pinhead:1X06
- added LED2, LED4, LED5: YLW, led:CHIP-LED0603
- added R14, R16, R20: 1k, rcl_custom:0402-C-NOSILK
- added TP1, TP3, TP6, TP7, TP8: TEST-POINT, Tova:2MM-TEST-POINT
- LED3: device apdm:PLCC-6 -> Tova:PLCC-6
- R6: value 68 -> 1k
- moved C35 15.0 mm to (15.9, 23.4), turned to 90 degrees
- moved C34 10.9 mm to (24.8, 17.3), turned to 270 degrees
- moved C23 10.8 mm to (25.8, 19.2), turned to 90 degrees
- moved C32 10.0 mm to (21.1, 17.1)
- moved R43 8.27 mm to (32.0, 18.0), turned to 0 degrees
- moved C27 7.78 mm to (31.0, 15.2), turned to 180 degrees
- moved U3 7.10 mm to (27.7, 16.0)
- moved L3 7.08 mm to (22.4, 19.6)
- moved C28 4.71 mm to (20.8, 22.0), turned to 0 degrees
- moved R15 4.42 mm to (27.4, 12.1), turned to 90 degrees
- moved R42 4.36 mm to (29.8, 11.3), turned to 90 degrees
- moved R17 2.79 mm to (25.8, 25.5), turned to 90 degrees
- moved LED6 1.52 mm to (25.8, 23.4), turned to 180 degrees
- moved C29 0.92 mm to (52.3, 7.37)
- moved C30 0.92 mm to (44.2, 5.84)
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Connections:
- net VDDA renamed N$47
- new net 3.3VD1: LED2.C, U2.55
- new net N$48: T1.4, U3.3
- new net N$49: LED4.C, U2.56
- new net N$50: LED5.C, U2.57
- new net N$51: LED4.A, R16.1
- new net N$52: LED5.A, R20.1
- new net N$53: JP3.3, TP8.1
- new net N$54: TP7.1, U2.4
- new net N$55: TP6.1, U2.3
- new net N$56: TP3.1, U2.2
- new net N$57: TP1.1, U2.1
- new net USART6_RX: JP3.4, U2.64
- new net USART6_TX: JP3.5, U2.63
- net 3.3VD: now also JP3.2, R14.2, R16.2, R20.2
- net GND: now also C36.2, JP3.1; no longer C31.2
- net N$1: now also C36.1; no longer C31.1
- net N$40: now also U3.5; no longer U3.3
- net N$41: now also U3.4; no longer U3.6
- net N$42: now also LED2.A, R14.1; no longer T1.4, U3.5
- net N$44: now also U3.6; no longer U3.4
Routing:
- net USART6_TX: track 0.00 -> 39.7 mm, vias 0 -> 1
- net USART6_RX: track 0.00 -> 39.3 mm, vias 0 -> 1
- net ETH_RMII_REF_CLK: track 4.16 -> 42.1 mm
- net N$41: track 0.00 -> 15.5 mm
- net N$48: track 0.00 -> 14.4 mm
- net N$44: track 0.00 -> 14.4 mm
- net N$40: track 0.00 -> 13.7 mm
- net 3.3VD: track 35.1 -> 46.0 mm, vias 41 -> 47
- net 3.3VD1: track 0.00 -> 6.58 mm
- net N$39: track 0.00 -> 5.92 mm, vias 0 -> 2
- net N$49: track 0.00 -> 5.67 mm
- net MCO1-ETH-CLK: track 24.3 -> 29.2 mm, vias 4 -> 2
- net ETH_MDIO: track 30.1 -> 35.0 mm
- net N$50: track 0.00 -> 4.60 mm
- net N$57: track 0.00 -> 4.49 mm
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- added copper zone on layer 1, net VDDA_3.3
- removed copper zone on layer 1, net N$47
- removed copper zone on layer 16, net N$47

Commit message: Checked SAW and LNA, moved to endfire SMA, still need to cleanup RF and also, see README for the beginning of a component writeup and a todo list.
Parts:
- removed L7: SAW_1.4X1.1, swift-nav:SAW_1.4X1.1
- removed X2: BU-SMA-H, con-coax:BU-SMA-H
- added J2: CON_SMA-ENDFIRE_EMERSON_EMERSON-142-0701-801, emerson-sma-endfire:SMA-CON-EMERSON
- added L8: SF14-1575F5UU19, saw_1.4x1.1:SAW_1.4X1.1
- L6: value SAW_1.4X1.1 -> SF14-1575F5UU19; device swift-nav:SAW_1.4X1.1 -> saw_1.4x1.1:SAW_1.4X1.1
- U5: value XC2401 -> XC2401A8167R-G; device swift-nav:XC2401 -> xc2401:USPN-4B02
- moved L2 6.45 mm to (88.5, 21.1)
- moved L5 6.45 mm to (88.5, 22.7)
- moved L6 3.59 mm to (79.1, 30.1), turned to 180 degrees
- moved C24 2.12 mm to (79.9, 23.1), turned to 90 degrees
- moved C19 0.25 mm to (82.2, 19.2)
- moved C22 0.13 mm to (82.2, 20.4)
- moved R4 0.13 mm to (82.2, 17.0)
Connections:
- net GND: now also J2.GND, J2.GND@1, J2.GND@2, J2.GND@3, L6.2, L6.3, L6.5, L8.2, L8.3, L8.5; no longer L6.B, L6.C, L6.E, L7.B, L7.C, L7.E, X2.2, X2.3, X2.4, X2.5
- net LNA2: now also J2.SIG, L6.1; no longer L6.A, X2.1
- net LNAOUT: now also L8.1; no longer L7.A
- net MIXIN: now also L8.4; no longer L7.D
- net N$21: now also L6.4; no longer L6.D
Routing:
- net N$21: track 1.19 -> 10.6 mm
- net N$5: track 5.34 -> 2.49 mm
- net N$14: track 2.35 -> 0.00 mm
- net N$22: track 2.14 -> 0.00 mm
- net GND: track 13.6 -> 13.0 mm
- net LNA2: track 3.98 -> 4.54 mm

Commit message: Better RF layout. Now doing tented vias for a tighter layout, also changed design rules to get same signal vias closer in to pads. Is 1x width enough clearance to ground for RF signals? And then the real question: done?
Parts:
- moved L2 4.24 mm to (84.3, 21.7)
- moved R4 3.60 mm to (84.8, 14.6), turned to 270 degrees
- moved L5 3.33 mm to (85.3, 21.7), turned to 90 degrees
- moved C56 2.73 mm to (82.3, 20.1), turned to 180 degrees
- moved C22 2.09 mm to (82.7, 18.4)
- moved C19 1.97 mm to (82.7, 17.3)
- moved U5 1.97 mm to (83.9, 19.9)
- moved L8 1.83 mm to (74.4, 21.7), turned to 270 degrees
- moved R13 1.57 mm to (82.3, 21.0), turned to 0 degrees
- moved C24 1.53 mm to (81.0, 22.1), turned to 0 degrees
- moved L6 1.02 mm to (80.1, 30.1)
Routing:
- net ANTFLAG: track 43.3 -> 37.9 mm
- net N$22: track 0.00 -> 3.38 mm
- net MAX_!IDLE: track 46.1 -> 43.0 mm
- net PGM: track 3.12 -> 6.10 mm, vias 0 -> 2
- net N$5: track 2.49 -> 4.62 mm
- net GND: track 13.0 -> 11.2 mm, vias 194 -> 233
- net ANTBIAS: track 8.31 -> 6.71 mm
- net N$2: track 4.22 -> 2.82 mm
- net N$17: track 7.18 -> 5.78 mm
- net LNAOUT: track 6.93 -> 8.08 mm
- net 2.85VA: track 6.06 -> 4.91 mm, vias 12 -> 15
- net N$14: track 0.00 -> 1.14 mm
- net LNA2: track 4.54 -> 3.52 mm
- net MIXIN: track 5.11 -> 4.19 mm

Commit message: New, better, small, yellow, different crystal, and more notes on components.
Parts:
- X1: device crystal:CTS406 -> 8Y_25MHzCrystal:8Y
- moved C30 5.62 mm to (49.8, 5.21), turned to 180 degrees
- moved X1 1.80 mm to (50.0, 6.86), turned to 0 degrees
- moved C29 0.64 mm to (51.9, 6.86)
- renumbered U10 to U8, USB to J4
Connections:
- net GND: now also X1.2, X1.4
- net OSC_IN: now also X1.1; no longer X1.3
- net OSC_OUT: now also X1.3; no longer X1.1
Routing:
- net OSC_IN: track 9.75 -> 7.66 mm
- net OSC_OUT: track 6.66 -> 6.10 mm
