File: v2-rf-frontend-board.brd (EAGLE design)
At the start: 86.6 x 43.9 mm, 134 parts, among them J1 1.27MM-SWD-CONNECTOR, J2 CON_SMA-ENDFIRE_EMERSON_EMERS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, J3 ROCKETNET-CONNECTOR-16M, J4 ZX62D-B-5P8, Q1 NTR4101P, T1 ALT4532, T2 ALT4532, U1 MAX2769, U2 STM32F4V_100PIN_GPSBOARD, U3 KSZ8081, U4 7Q-16.368MBG-T, U5 XC2401A8167R-G, U6 MAX8510EXK29+T, U7 MAX8510EXK29+T, U8 LMZ12001, X1 25 MHz

Commit message: DONE.
Parts:
- removed C1: 1u 50V, rcl_custom:0805-B-NOSILK
- removed TP23: (no value), testpad:TP06R
- added C31, C64: 100n, rcl_custom:0402-C-NOSILK
- added C53, C58: 2.2u, rcl_custom:0603-B-NOSILK
- added C63: 100p, rcl_custom:0402-C-NOSILK
- added C65: 1u 50V, rcl_custom:0603-B-NOSILK
- added TP10, TP9: TEST-POINT, Tova:2MM-TEST-POINT
- C10: value 100n 10V -> 100n
- C2: value 100n 10V -> 10n
- C20: value 2.2u 10V -> 2.2u; device rcl_custom:0603-C-NOSILK -> rcl_custom:0603-B-NOSILK
- C21: value 220n -> 100n
- C25, C43, C54, C55, C60: device rcl_custom:0402-B-NOSILK -> rcl_custom:0402-C-NOSILK
- C26: value 220nF -> 22n
- C39: value 1uF -> 1u
- C51, C52: device rcl_custom:0603-C-NOSILK -> rcl_custom:0603-B-NOSILK
- C57: value 470n -> 100p
- L2, L5, R10, R11, R12, R13, R14, R15, R16, R17, R18, R19, R2, R20, R38, R39, R40, R42, R43, R5, R6, R8, R9: device rcl_custom:0402-C-NOSILK -> rcl_custom:0402-C-NOSILK@1
- L3: value FB0805/600R/200mA(201209-601) -> HF70ACC201209-T; device rcl_custom:0805-C-NOSILK -> rcl_custom:0805-C-NOSILK@1
- LED1, LED2, LED4, LED5: device led:CHIP-LED0603 -> led:CHIPLED_0603
- LED3: value (none) -> RGB
- LED6: value GRN -> YLW
- R1: value 10k -> 3.32k; device rcl_custom:0402-C-NOSILK -> rcl_custom:0402-C-NOSILK@1
- R3: value 3.3k -> 1.07k; device rcl_custom:0402-C-NOSILK -> rcl_custom:0402-C-NOSILK@1
- R4: value 0 -> 1k; device rcl_custom:0402-C-NOSILK -> rcl_custom:0402-C-NOSILK@1
- R7: value 249k -> 61.9k; device rcl_custom:0402-C-NOSILK -> rcl_custom:0402-C-NOSILK@1
- moved C48 0.38 mm to (57.0, 26.7)
- moved C60 0.25 mm to (65.0, 31.2)
- moved C21 0.25 mm to (15.0, 27.9)
- moved C33 0.25 mm to (5.08, 32.3)
- moved C38 0.13 mm to (23.0, 32.3)
- moved C39 0.13 mm to (20.4, 32.3)
- moved C51 0.13 mm to (44.3, 29.2)
- moved C8 0.13 mm to (81.8, 13.1)
- moved R4 0.13 mm to (85.0, 14.6)
- renumbered JP1 to J5, JP3 to J6, SD1 to J7
Connections:
- net N$1 renamed VDD_1.2_ETH_SUPP
- net N$14 renamed EXT-LNA-IN
- net N$2 renamed LNA1
- net N$21 renamed SMA-FILTERED
- net N$3 renamed EXTLNA-OUT
- net N$35 renamed TCXO-OUT
- net N$4 renamed LNA-POWER-FILTERED
- net N$5 renamed STRAIGHT-THROUGH
- removed net N$17: C19.3, U1.25
- new net SMA-RAW: J2.SIG, L6.1
- net 2.85VA: now also C58.1, R13.1
- net 2.85VD: now also C31.1, C53.1
- net ANTBIAS: now also C63.1, C64.1, TP10.1; no longer R13.1
- net CLKOUT: now also TP9.1; no longer TP23.TP
- net GND: now also C31.2, C53.2, C58.2, C63.2, C64.2, C65.2; no longer C1.2
- net LNA2: now also C19.3, U1.25; no longer J2.SIG, L6.1
- net VIN: now also C65.1; no longer C1.1
Routing:
- net 3.3VD: track 46.0 -> 40.0 mm, vias 47 -> 50
- net N$17: track 5.78 -> 0.00 mm
- net SMA-RAW: track 0.00 -> 3.52 mm
- net ANTBIAS: track 6.71 -> 10.2 mm, vias 2 -> 1
- net LNA2: track 3.52 -> 5.78 mm
- net OTG_FS_VBUS: track 52.2 -> 53.7 mm, vias 5 -> 8
- net CLKOUT: track 3.76 -> 5.14 mm
- net MAX_!IDLE: track 43.0 -> 41.9 mm
- net 2.85VA: track 4.91 -> 5.96 mm, vias 15 -> 19
- net GND: track 11.2 -> 10.3 mm, vias 233 -> 323
- net CPOUT: track 6.28 -> 5.76 mm
- net 2.85VD: track 2.92 -> 3.09 mm, vias 13 -> 16
- net VIN: vias 8 -> 10
Other:
- board text added: "GPS Raw Data Capture Board V2 Portland State Aerospace - http://psas.pdx.edu/ - Jenner Hanni and Andrew Greenberg"
- board text removed: "GPS RF FRONT-END BOARD V2 FEB 2014, Portland State Aerospace JENNER HANNI and ANDREW GREENBERG"
