File: v2-rf-frontend-board.brd (EAGLE design)
At the start: 86.6 x 43.9 mm, 140 parts, among them J1 1.27MM-SWD-CONNECTOR, J2 CON_SMA-ENDFIRE_EMERSON_EMERS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, J3 ROCKETNET-CONNECTOR-16M, J4 ZX62D-B-5P8, J5 BREAKOUT, J7 CON_HIROSE_DM3D(MICROSD), Q1 NTR4101P, T1 ALT4532, T2 ALT4532, U1 MAX2769, U2 STM32F4V_100PIN_GPSBOARD, U3 KSZ8081, U4 7Q-16.368MBG-T, U5 XC2401A8167R-G, U6 MAX8510EXK29+T, U7 MAX8510EXK29+T, U8 LMZ12001, X1 25 MHz

Commit message: OMG TEST POINTS!!!!11!!
Parts:
- added TP11, TP12, TP13, TP14, TP15, TP16, TP17, TP18, TP19, TP20: TEST-POINT, Tova:2MM-TEST-POINT
- R38: value 68 -> 400
- R39: value 68 -> 110
- R40: value 27 -> 900
- moved C60 0.28 mm to (64.8, 31.4)
- moved C43 0.13 mm to (64.8, 37.0)
Connections:
- new net N$1: TP11.1, U8.3
- new net N$2: TP16.1, U3.17
- net 2.85VA: now also TP15.1
- net 2.85VD: now also TP14.1
- net 3.3VD: now also TP13.1
- net GND: now also TP17.1, TP18.1, TP19.1, TP20.1
- net VIN: now also TP12.1
Routing:
- net N$1: track 0.00 -> 13.6 mm, vias 0 -> 1
- net N$2: track 0.00 -> 9.31 mm, vias 0 -> 1

Commit message: Silly clean up, ran ERC and DRC again.
Changed lines of the file:
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@@
 <layer number="23" name="tOrigins" color="15" fill="1" visible="yes" active="yes"/>
 <layer number="24" name="bOrigins" color="15" fill="1" visible="yes" active="yes"/>
-<layer number="25" name="tNames" color="7" fill="1" visible="yes" active="yes"/>
+<layer number="25" name="tNames" color="7" fill="1" visible="no" active="yes"/>
 <layer number="26" name="bNames" color="7" fill="1" visible="no" active="yes"/>
 <layer number="27" name="tValues" color="7" fill="1" visible="no" active="yes"/>
@@
 <via x="28.067" y="36.83" extent="1-16" drill="0.254"/>
 <via x="40.64" y="38.227" extent="1-16" drill="0.254"/>
-<via x="58.674" y="26.797" extent="1-16" drill="0.254"/>
+<via x="58.674" y="27.051" extent="1-16" drill="0.254"/>
 <via x="74.93" y="41.91" extent="1-16" drill="0.254"/>
 <via x="76.581" y="21.463" extent="1-16" drill="0.254"/>

Commit message: Added modwire proposals for SPI 3-wire fix. See Issue 4 in gps-rf-board github repository.
Connections:
- net MAX_CFG_!CS: now also U2.96
- net MAX_CFG_MOSI: now also U2.54
- net MAX_CFG_SCLK: now also U2.47
Changed lines of the file:
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@@
 <wire x1="69.977" y1="20.32" x2="69.977" y2="23.495" width="0.2032" layer="1"/>
 <wire x1="69.977" y1="23.495" x2="67.183" y2="26.289" width="0.2032" layer="1"/>
+<contactref element="U2" pad="47"/>
+<wire x1="57.026" y1="22.177" x2="57.026" y2="23.677" width="0" layer="19" extent="1-1"/>
 </signal>
 <signal name="MAX_CFG_MOSI">
@@
 <wire x1="70.358" y1="20.447" x2="70.358" y2="23.749" width="0.2032" layer="1"/>
 <wire x1="70.358" y1="23.749" x2="67.437" y2="26.67" width="0.2032" layer="1"/>
+<contactref element="U2" pad="54"/>
+<wire x1="57.026" y1="22.677" x2="53.776" y2="26.927" width="0" layer="19" extent="1-1"/>
 </signal>
 <signal name="MAX_CFG_!CS">
@@
 <wire x1="57.026" y1="21.677" x2="59.777" y2="21.677" width="0.2032" layer="1"/>
 <wire x1="59.777" y1="21.677" x2="61.849" y2="23.749" width="0.2032" layer="1"/>
+<contactref element="U2" pad="96"/>
+<wire x1="41.526" y1="15.177" x2="57.026" y2="21.677" width="0" layer="19" extent="1-1"/>
 </signal>
 <signal name="N$9">

Commit message: Removed SPI2_NSS modwire proposal from v2 schematic.
Connections:
- net MAX_CFG_!CS: no longer U2.96
Changed lines of the file:
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@@
 <wire x1="57.026" y1="21.677" x2="59.777" y2="21.677" width="0.2032" layer="1"/>
 <wire x1="59.777" y1="21.677" x2="61.849" y2="23.749" width="0.2032" layer="1"/>
-<contactref element="U2" pad="96"/>
-<wire x1="41.526" y1="15.177" x2="57.026" y2="21.677" width="0" layer="19" extent="1-1"/>
 </signal>
 <signal name="N$9">

Commit message: Added annotation for DEBUG-PHY-MODWIRE (currently on prototype)
Connections:
- removed net N$39: LED6.C, U3.23
- removed net N$57: TP1.1, U2.1
- new net DEBUG-PHY-MODWIRE: LED6.C, TP1.1, U2.1, U3.23
Routing:
- net DEBUG-PHY-MODWIRE: track 0.00 -> 10.4 mm, vias 0 -> 2
- net N$39: track 5.92 -> 0.00 mm, vias 2 -> 0
- net N$57: track 4.49 -> 0.00 mm
Changed lines of the file:
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@@
 <?xml version="1.0" encoding="utf-8"?>
 <!DOCTYPE eagle SYSTEM "eagle.dtd">
-<eagle version="6.6.0">
+<eagle version="6.5.0">
 <drawing>
 <settings>
@@
 </polygon>
 </signal>
-<signal name="N$39">
+<signal name="DEBUG-PHY-MODWIRE">
 <contactref element="U3" pad="23"/>
 <contactref element="LED6" pad="C"/>
@@
 <wire x1="26.936" y1="20.078" x2="26.936" y2="22.594" width="0.2286" layer="16"/>
 <wire x1="26.936" y1="22.594" x2="26.924" y2="22.606" width="0.2286" layer="16"/>
+<contactref element="TP1" pad="1"/>
+<contactref element="U2" pad="1"/>
+<wire x1="39.37" y1="10.795" x2="39.624" y2="10.795" width="0.2286" layer="1"/>
+<wire x1="39.624" y1="10.795" x2="40.64" y2="11.811" width="0.2286" layer="1"/>
+<wire x1="40.64" y1="11.811" x2="42.164" y2="11.811" width="0.2286" layer="1"/>
+<wire x1="42.164" y1="11.811" x2="42.545" y2="11.43" width="0.2286" layer="1"/>
+<wire x1="42.545" y1="11.43" x2="43.273" y2="11.43" width="0.2286" layer="1"/>
+<wire x1="43.273" y1="11.43" x2="43.276" y2="11.427" width="0.2286" layer="1"/>
+<wire x1="26.936" y1="17.862" x2="39.37" y2="10.795" width="0" layer="19" extent="1-1"/>
 </signal>
 <signal name="N$24">
@@
 <wire x1="42.164" y1="10.795" x2="41.148" y2="10.795" width="0.2286" layer="1"/>
 </signal>
-<signal name="N$57">
-<contactref element="TP1" pad="1"/>
-<contactref element="U2" pad="1"/>
-<wire x1="39.37" y1="10.795" x2="39.624" y2="10.795" width="0.2286" layer="1"/>
-<wire x1="39.624" y1="10.795" x2="40.64" y2="11.811" width="0.2286" layer="1"/>
-<wire x1="40.64" y1="11.811" x2="42.164" y2="11.811" width="0.2286" layer="1"/>
-<wire x1="42.164" y1="11.811" x2="42.545" y2="11.43" width="0.2286" layer="1"/>
-<wire x1="42.545" y1="11.43" x2="43.273" y2="11.43" width="0.2286" layer="1"/>
-<wire x1="43.273" y1="11.43" x2="43.276" y2="11.427" width="0.2286" layer="1"/>
-</signal>
 <signal name="USART6_TX">

Commit message: Added modwire for SPI1-NSS. This should enable the use of STM32 SPI1 in slave mode to read data output.
Connections:
- new net N$3: U2.35
- new net SPI1-NSS: U2.29, U2.31
Changed lines of the file:
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@@
 <wire x1="31.623" y1="10.668" x2="33.02" y2="10.668" width="0.2032" layer="16"/>
+</signal>
+<signal name="N$3">
+<contactref element="U2" pad="35"/>
+</signal>
+<signal name="SPI1-NSS">
+<contactref element="U2" pad="29"/>
+<contactref element="U2" pad="31"/>
+<wire x1="57.026" y1="14.677" x2="57.026" y2="15.677" width="0" layer="19" extent="1-1"/>
 </signal>
 </signals>

Commit message: Cleaned up modwire patches a bit. Added cuts in 0.1" double header.
Connections:
- new net N$4: J5.1, U2.45
- net MAX_CFG_MOSI: no longer J5.1, U2.45
- net MAX_CFG_SCLK: no longer J5.2, U2.44
- net SPI1-NSS: now also J5.2
Routing:
- net MAX_CFG_MOSI: track 29.0 -> 17.5 mm
- net MAX_CFG_SCLK: track 26.5 -> 16.1 mm
- net N$4: track 0.00 -> 8.93 mm
Changed lines of the file:
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@@
 <?xml version="1.0" encoding="utf-8"?>
 <!DOCTYPE eagle SYSTEM "eagle.dtd">
-<eagle version="6.5.0">
+<eagle version="6.6.0">
 <drawing>
 <settings>
@@
 <setting verticaltext="up"/>
 </settings>
-<grid distance="0.005" unitdist="inch" unit="inch" style="lines" multiple="1" display="yes" altdistance="0.001" altunitdist="inch" altunit="inch"/>
+<grid distance="0.005" unitdist="inch" unit="inch" style="lines" multiple="1" display="no" altdistance="0.001" altunitdist="inch" altunit="inch"/>
 <layers>
 <layer number="1" name="Top" color="4" fill="1" visible="yes" active="yes"/>
@@
 <layer number="14" name="Route14" color="1" fill="6" visible="no" active="no"/>
 <layer number="15" name="SUPPLY" color="14" fill="1" visible="no" active="yes"/>
-<layer number="16" name="Bottom" color="1" fill="1" visible="yes" active="yes"/>
+<layer number="16" name="Bottom" color="1" fill="1" visible="no" active="yes"/>
 <layer number="17" name="Pads" color="2" fill="1" visible="yes" active="yes"/>
 <layer number="18" name="Vias" color="2" fill="1" visible="yes" active="yes"/>
@@
 <layer number="20" name="Dimension" color="15" fill="1" visible="yes" active="yes"/>
 <layer number="21" name="tPlace" color="7" fill="1" visible="yes" active="yes"/>
-<layer number="22" name="bPlace" color="7" fill="1" visible="yes" active="yes"/>
+<layer number="22" name="bPlace" color="7" fill="1" visible="no" active="yes"/>
 <layer number="23" name="tOrigins" color="15" fill="1" visible="yes" active="yes"/>
-<layer number="24" name="bOrigins" color="15" fill="1" visible="yes" active="yes"/>
+<layer number="24" name="bOrigins" color="15" fill="1" visible="no" active="yes"/>
 <layer number="25" name="tNames" color="7" fill="1" visible="no" active="yes"/>
 <layer number="26" name="bNames" color="7" fill="1" visible="no" active="yes"/>
@@
 <layer number="50" name="dxf" color="7" fill="1" visible="no" active="no"/>
 <layer number="51" name="tDocu" color="7" fill="1" visible="yes" active="yes"/>
-<layer number="52" name="bDocu" color="7" fill="1" visible="yes" active="yes"/>
+<layer number="52" name="bDocu" color="7" fill="1" visible="no" active="yes"/>
 <layer number="53" name="tGND_GNDA" color="7" fill="9" visible="no" active="no"/>
 <layer number="54" name="bGND_GNDA" color="1" fill="9" visible="no" active="no"/>
@@
 <layer number="100" name="Hidden_Layer" color="7" fill="1" visible="no" active="no"/>
 <layer number="101" name="Flex-Kleb" color="7" fill="1" visible="no" active="no"/>
-<layer number="102" name="FIXME" color="12" fill="1" visible="yes" active="yes"/>
+<layer number="102" name="FIXME" color="12" fill="1" visible="no" active="yes"/>
 <layer number="103" name="tMap" color="7" fill="1" visible="no" active="yes"/>
 <layer number="104" name="Name" color="7" fill="1" visible="no" active="yes"/>
@@
 <contactref element="U1" pad="9"/>
 <contactref element="J5" pad="21"/>
-<contactref element="J5" pad="2"/>
-<wire x1="59.261" y1="22.177" x2="60.325" y2="23.241" width="0.2032" layer="1"/>
-<wire x1="60.325" y1="23.241" x2="60.325" y2="25.019" width="0.2032" layer="1"/>
-<wire x1="60.325" y1="25.019" x2="61.595" y2="26.289" width="0.2032" layer="1"/>
-<wire x1="61.595" y1="26.289" x2="64.643" y2="26.289" width="0.2032" layer="16"/>
 <wire x1="64.516" y1="26.289" x2="64.643" y2="26.289" width="0.2032" layer="1"/>
 <wire x1="74.639" y1="16.367" x2="73.93" y2="16.367" width="0.2032" layer="1"/>
 <wire x1="67.183" y1="26.289" x2="64.643" y2="26.289" width="0.2032" layer="1"/>
-<contactref element="U2" pad="44"/>
-<wire x1="57.026" y1="22.177" x2="59.261" y2="22.177" width="0.2032" layer="1"/>
 <wire x1="73.93" y1="16.367" x2="69.977" y2="20.32" width="0.2032" layer="1"/>
 <wire x1="69.977" y1="20.32" x2="69.977" y2="23.495" width="0.2032" layer="1"/>
 <wire x1="69.977" y1="23.495" x2="67.183" y2="26.289" width="0.2032" layer="1"/>
 <contactref element="U2" pad="47"/>
-<wire x1="57.026" y1="22.177" x2="57.026" y2="23.677" width="0" layer="19" extent="1-1"/>
+<wire x1="57.026" y1="23.677" x2="64.516" y2="26.289" width="0" layer="19" extent="1-1"/>
 </signal>
 <signal name="MAX_CFG_MOSI">
 <contactref element="U1" pad="8"/>
-<contactref element="J5" pad="1"/>
 <contactref element="J5" pad="22"/>
-<wire x1="64.389" y1="28.829" x2="61.849" y2="28.829" width="0.2032" layer="16"/>
-<wire x1="58.364" y1="22.677" x2="59.69" y2="24.003" width="0.2032" layer="1"/>
-<wire x1="59.69" y1="24.003" x2="59.69" y2="25.019" width="0.2032" layer="1"/>
-<wire x1="59.69" y1="25.019" x2="60.325" y2="25.654" width="0.2032" layer="1"/>
-<wire x1="60.325" y1="25.654" x2="60.325" y2="27.305" width="0.2032" layer="1"/>
-<wire x1="60.325" y1="27.305" x2="61.849" y2="28.829" width="0.2032" layer="1"/>
 <wire x1="67.437" y1="26.67" x2="67.437" y2="27.305" width="0.2032" layer="1"/>
 <wire x1="67.437" y1="27.305" x2="65.913" y2="28.829" width="0.2032" layer="1"/>
 <wire x1="65.913" y1="28.829" x2="64.389" y2="28.829" width="0.2032" layer="1"/>
-<contactref element="U2" pad="45"/>
-<wire x1="57.026" y1="22.677" x2="58.364" y2="22.677" width="0.2032" layer="1"/>
 <wire x1="74.639" y1="16.867" x2="73.938" y2="16.867" width="0.2032" layer="1"/>
 <wire x1="73.938" y1="16.867" x2="70.358" y2="20.447" width="0.2032" layer="1"/>
@@
 <wire x1="70.358" y1="23.749" x2="67.437" y2="26.67" width="0.2032" layer="1"/>
 <contactref element="U2" pad="54"/>
-<wire x1="57.026" y1="22.677" x2="53.776" y2="26.927" width="0" layer="19" extent="1-1"/>
+<wire x1="53.776" y1="26.927" x2="64.389" y2="28.829" width="0" layer="19" extent="1-1"/>
 </signal>
 <signal name="MAX_CFG_!CS">
@@
 <contactref element="U2" pad="29"/>
 <contactref element="U2" pad="31"/>
+<contactref element="J5" pad="2"/>
+<wire x1="57.026" y1="15.677" x2="61.595" y2="26.289" width="0" layer="19" extent="1-1"/>
 <wire x1="57.026" y1="14.677" x2="57.026" y2="15.677" width="0" layer="19" extent="1-1"/>
 </signal>
+<signal name="N$4">
+<contactref element="J5" pad="1"/>
+<contactref element="U2" pad="45"/>
+<wire x1="58.364" y1="22.677" x2="59.69" y2="24.003" width="0.2032" layer="1"/>
+<wire x1="59.69" y1="24.003" x2="59.69" y2="25.019" width="0.2032" layer="1"/>
+<wire x1="59.69" y1="25.019" x2="60.325" y2="25.654" width="0.2032" layer="1"/>
+<wire x1="60.325" y1="25.654" x2="60.325" y2="27.305" width="0.2032" layer="1"/>
+<wire x1="60.325" y1="27.305" x2="61.849" y2="28.829" width="0.2032" layer="1"/>
+<wire x1="57.026" y1="22.677" x2="58.364" y2="22.677" width="0.2032" layer="1"/>
+</signal>
 </signals>
