File: gps-to-spi.sch (EAGLE design)
At the start: 10 parts, among them IC1 74HC165D, IC2 74HC165D, IC3 74AC175D, IC4 74LS32D, IC5 74HC08D, IC6 74AHC1G14DBV, Q1 NTR4101P, U1 74HC40103D,652

Commit message: OK, I had to polish it: names, test points, header inputs/outputs, no ERC errors.
Parts:
- added C1, C2, C3, C4, C5, C6, C7: 100n, rcl_custom:C-EU0603-B-NOSILK
- added C8: 10u, rcl_custom:C-EU0603-B-NOSILK
- added JP1: (no value), pinhead:PINHD-1X5
- added JP2, JP3: (no value), pinhead:PINHD-1X4
- added TP1, TP10, TP11, TP12, TP13, TP14, TP15, TP16, TP17, TP18, TP19, TP2, TP20, TP21, TP3, TP4, TP5, TP6, TP7, TP8, TP9: TEST-POINT, Tova:TEST-POINT
- R2: value (none) -> 10k
Connections:
- removed net N$1: IC3A.D2, IC3A.Q1, IC4A.I0, IC5B.I1, U1.CP
- removed net N$10: IC2A.SH/!LD, IC3A.!Q3
- removed net N$11: IC1A.INH, IC2A.QH
- removed net N$7: IC4D.O, Q1.G, R2.2, U1.~PL
- removed net N$9: IC1A.SH/!LD, IC3A.!Q2
- new net !SEND_SPI: IC2A.SH/!LD, IC3A.!Q3, TP15.1
- new net !SS-START: IC3A.D2, IC3A.Q1, IC4A.I0, IC5B.I1, TP13.1, U1.CP
- new net INIT: IC4D.O, Q1.G, R2.2, TP12.1, U1.~PL
- new net LATCH-NIBBLE: IC1A.SH/!LD, IC3A.!Q2, TP14.1
- new net N$15: IC1A.D, TP1.1
- new net N$16: IC1A.C, TP2.1
- new net N$17: IC1A.B, TP3.1
- new net N$18: IC1A.A, TP4.1
- new net SCLK-PAUSE: IC1A.INH, IC2A.QH, TP10.1
- net !SS: now also JP2.3, TP17.1
- net 16.384MHZ: now also JP1.5, TP5.1
- net 25MHZ: now also JP2.4, TP11.1
- net GND: now also C1.2, C2.2, C3.2, C4.2, C5.2, C6.2, C7.2, C8.2, IC1A.SER, JP3.1, JP3.2
- net I0: now also JP1.4, TP6.1
- net I1: now also JP1.3, TP7.1
- net MOSI: now also JP2.1, TP18.1
- net N$13: now also TP20.1
- net N$14: now also TP21.1
- net N$5: now also TP16.1
- net Q0: now also JP1.2, TP8.1
- net Q1: now also JP1.1, TP9.1
- net SCLK: now also JP2.2, TP19.1
- net VCC: now also C1.1, C2.1, C3.1, C4.1, C5.1, C6.1, C7.1, C8.1, IC3A.CLR, JP3.3, JP3.4
Other:
- note added: "Power In"
- moved on the sheet: IC1P, IC2P, IC3P, IC4P, IC5C, IC5D, IC5P, IC6, IC6P
