File: v3-gps.brd (EAGLE design)
At the start: 86.6 x 43.9 mm, 168 parts, among them J1 1.27MM-SWD-CONNECTOR, J2 CON_SMA-ENDFIRE_EMERSON_EMERS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, J3 ROCKETNET-CONNECTOR-16M, J4 ZX62D-B-5P8, J7 CON_HIROSE_DM3D(MICROSD), Q1 NTR4101P, T1 ALT4532, T2 ALT4532, U1 MAX2769, U10 MINICIRCUITS-BP2G, U11 MAX8510EXK29+T, U2 STM32F4V_100PIN_GPSBOARD, U3 KSZ8081, U4 7Q-16.368MBG-T, U5 XC2401A8167R-G, U6 MAX8510EXK29+T, U7 MAX8510EXK29+T, U8 LMZ12001, U9 VENUS638FLPX-L, X1 25 MHz

Commit message: First commit of the GPS v3 board, which includes the CPLD and SkyTraq ICs.
Parts:
- U10: value MINICIRCUITS-BP2G -> BP2G+
Changed lines of the file:
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@@
 <element name="C1" library="rcl_custom" package="0402-C-NOSILK" value="100p" x="1.016" y="-2.413"/>
 <element name="U9" library="SparkFun-RF" package="VENUS638FLPX" value="VENUS638FLPX-L" x="16.891" y="-8.001"/>
-<element name="U10" library="minicircuits-splitter" package="MINICIRCUITS" value="MINICIRCUITS-BP2G" x="3.683" y="-19.685"/>
+<element name="U10" library="minicircuits-splitter" package="MINICIRCUITS" value="BP2G+" x="3.683" y="-19.685"/>
 <element name="LED7" library="led" package="CHIPLED_0603" value="YLW" x="-2.921" y="-21.717"/>
 <element name="C19" library="rcl_custom" package="0402-C-NOSILK" value="1u" x="-3.937" y="-25.654"/>

Commit message: More rough drafting on the CPLD. Added 1.8V supply (kind of), added some cleanup notes on clock, etc. TODO: everything still, including cleanup up 1.8V supply and probably splitting the power domains on the CPLD.
Parts:
- added C71, C72, C73, C74: 100p, rcl_custom:0402-C-NOSILK
- added C75, C76: 1u, rcl_custom:0603-B-NOSILK
- added C77: 10n, rcl_custom:0402-C-NOSILK
- added C78: 100n, rcl_custom:0402-C-NOSILK
- added IC1: XC2C32A_VQ44_2, dp_devices:VQ44
- added JP1: (no value), pinhead:1X06
- added TP21: TEST-POINT, Tova:2MM-TEST-POINT
- added VR1: MIC5025-1.8V, dp_devices:SOT-23-5
Connections:
- new net N$3: IC1.10, JP1.6
- new net N$35: IC1.9, JP1.5
- new net N$53: IC1.24, JP1.4
- new net N$57: IC1.11, JP1.3
- new net N$58: C77.2, VR1.4
- new net N$59: U1.17
- new net N$60: U1.18
- new net N$61: U1.21
- new net N$62: U1.20
- new net V18: C74.1, C76.1, C77.1, C78.1, IC1.15, TP21.1, VR1.5
- net 3.3VD: now also C71.1, C72.1, C73.1, C75.1, IC1.26, IC1.35, IC1.7, JP1.1, VR1.1, VR1.3
- net GND: now also C71.2, C72.2, C73.2, C74.2, C75.2, C76.2, C78.2, IC1.17, IC1.25, IC1.4, JP1.2, VR1.2

Commit message: using the GPS Carrier from AV4, expanded the size of the board to fit in the AV4 C channel and give more room. Moved everything onto that larger board, with preliminary placement. About to rip up and flip  STM because of OCD (just can't stand it), so checking in before I do something as stupid as that.
Parts:
- added C79: 1u, rcl_custom:0402-C-NOSILK
- added C80: 100p, rcl_custom:0402-C-NOSILK
- moved TP21 214.6 mm to (73.8, 45.3), turned to 180 degrees
- moved C77 213.5 mm to (80.1, 46.1), turned to 180 degrees
- moved C78 211.0 mm to (73.5, 50.8), turned to 270 degrees
- moved C76 207.6 mm to (75.6, 50.9), turned to 270 degrees
- moved C75 204.0 mm to (77.3, 51.1), turned to 270 degrees
- moved VR1 200.8 mm to (81.7, 50.2), turned to 270 degrees
- moved C74 193.5 mm to (80.6, 47.8), turned to 180 degrees
- moved C73 191.7 mm to (73.0, 54.1), turned to 270 degrees
- moved C72 188.9 mm to (74.8, 54.5), turned to 270 degrees
- moved C71 185.6 mm to (76.1, 54.6), turned to 270 degrees
- moved U11 137.4 mm to (23.7, 28.3), turned to 180 degrees
- moved TP9 136.4 mm to (18.9, 27.2), turned to 90 degrees
- moved C70 134.0 mm to (22.0, 28.8), turned to 180 degrees
- moved C69 132.0 mm to (22.0, 27.8), turned to 180 degrees
- moved C67 129.7 mm to (26.0, 28.1), turned to 270 degrees
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Connections:
- removed net BAR_GND: C24.1, C66.-, R22.1, U10.1, U10.3, U10.4, U10.6, U10.7
- net 2.85V-S: now also C79.1, C80.1
- net AGND: now also C56.2, J2.GND, J2.GND@1, J2.GND@2, J2.GND@3, L5.1, L6.2, L6.3, L6.5, U10.1, U10.3, U10.4, U10.6, U10.7, U5.3
- net GND: now also C24.1, C66.-, C79.2, C80.2, R22.1; no longer C56.2, J2.GND, J2.GND@1, J2.GND@2, J2.GND@3, L5.1, L6.2, L6.3, L6.5, U5.3
- net MAX-RF: now also U10.5; no longer U10.8
- net STQ-RF: now also U10.8; no longer U10.5
Routing:
- net STM_USART6_TX: track 39.5 -> 0.00 mm, vias 1 -> 0
- net STM_USART6_RX: track 37.3 -> 0.00 mm, vias 1 -> 0
- net MAX-RF: track 0.00 -> 33.4 mm
- net MAX_!IDLE: track 32.8 -> 0.00 mm, vias 1 -> 0
- net ANTFLAG: track 30.3 -> 0.00 mm, vias 1 -> 0
- net LD: track 23.8 -> 0.00 mm, vias 1 -> 0
- net MAX_CFG_MOSI: track 16.0 -> 0.00 mm
- net MAX_CFG_!CS: track 14.1 -> 0.00 mm
- net MAX_CFG_SCLK: track 13.4 -> 0.00 mm
- net MAX_!SHDN: track 10.5 -> 0.00 mm, vias 2 -> 0
- net SMA-FILTERED: track 9.53 -> 0.91 mm
- net PGM: track 6.22 -> 0.00 mm, vias 2 -> 0
- net DEBUG-PHY-MODWIRE: track 10.2 -> 5.92 mm
- net GND: track 8.55 -> 4.65 mm, vias 323 -> 291
- net LNA-POWER-FILTERED: track 2.55 -> 0.00 mm
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Other:
- board size 86.6 x 43.9 mm -> 86.6 x 62.2 mm

Commit message: New LNA+SAW filter, plus starting to lay stuff out.
Parts:
- removed L6: SF14-1575F5UU19, saw_1.4x1.1:SAW_1.4X1.1
- removed LED3: RGB, Tova:PLCC-6
- removed U5: XC2401A8167R-G, xc2401:USPN-4B02
- added C81: 47p, rcl_custom:0402-C-NOSILK
- added LED8: (no value), led-rgb-rohm:KINGBRITE_RGBLED_1.6X1.26
- added R25: 4.7k, rcl_custom:0402-C-NOSILK@1
- added U12: AVAGO-ALM-GPXX, ic-lna-ALM-GPxx-Avago:AVAGO+SAW+LNA
- C1: value 100p -> 330p
- C28, C32, C33: device rcl_custom:1206-C -> rcl_custom:1206-C@1
- C56: value 10n -> 100n
- L2: value 6.2nH -> 22n; device rcl_custom:0402-C-NOSILK@1 -> rcl_custom:.0402-B-NOSILK
- L3: device rcl_custom:0805-C-NOSILK@1 -> rcl_custom:.0805-C-NOSILK
- L5: value 9.1nH -> 1.8n; device rcl_custom:0402-C-NOSILK@1 -> rcl_custom:.0402-B-NOSILK
- R13: value 470 -> 10
- moved C66 46.1 mm to (62.1, 8.64), turned to 180 degrees
- moved TP18 44.8 mm to (56.9, 7.37), turned to 90 degrees
- moved TP9 42.0 mm to (57.0, 9.53), turned to 180 degrees
- moved R24 41.2 mm to (63.2, 13.3), turned to 180 degrees
- moved D1 39.4 mm to (60.8, 13.3), turned to 0 degrees
- moved C70 36.6 mm to (55.1, 13.3), turned to 0 degrees
- moved C30 36.5 mm to (26.5, 51.7), turned to 45 degrees
- moved C69 35.8 mm to (55.1, 14.4), turned to 0 degrees
- moved C29 35.1 mm to (26.2, 49.0), turned to 315 degrees
- moved TP6 33.8 mm to (25.9, 57.0), turned to 270 degrees
- moved X1 33.8 mm to (27.5, 50.3), turned to 225 degrees
- moved TP7 33.2 mm to (25.9, 55.4), turned to 270 degrees
- moved C68 33.1 mm to (54.2, 15.9), turned to 0 degrees
- moved U11 32.9 mm to (53.3, 13.8), turned to 0 degrees
- moved C61 31.8 mm to (28.4, 46.2), turned to 0 degrees
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Connections:
- removed net EXT-LNA-IN: L2.2, U5.4
- removed net SMA-FILTERED: L2.1, L5.2, L6.4
- removed net SMA-RAW: J2.SIG, L6.1
- new net N$63: IC1.20
- new net N$64: IC1.21, U1.16
- new net N$65: R25.2, U12.8
- new net N$66: L5.2, U12.7
- new net STM_SPI1_MISO: IC1.38, U2.31
- new net STM_SPI1_MOSI: IC1.36, U2.91
- new net STM_SPI1_NSS: IC1.34, U2.29
- new net STM_SPI1_SCK: IC1.37, U2.30
- net 2.85VA: now also C1.1, L2.2, R25.1
- net 3.3VD: now also LED8.2; no longer R38.1, R39.1, R40.1
- net AGND: now also C1.2, C81.2; no longer L5.1, L6.2, L6.3, L6.5, U5.3
- net GND: now also U12.2, U12.3, U12.4, U12.9, U12.P$1, U12.P$2
- net LED2: now also R39.2; no longer LED3.2
- net LNA-POWER-FILTERED: now also C81.1, L2.1, L5.1; no longer U5.1
- net N$11: now also R40.2; no longer LED3.6
- net N$12: now also LED8.4, R38.1; no longer LED3.4, R39.2
- net N$14: now also U12.6; no longer C1.1
- net N$18: now also LED8.1, R39.1; no longer LED3.3, R38.2
- net N$34: now also R38.2; no longer LED3.5
- net N$37: now also LED8.3, R40.1; no longer LED3.1, R40.2
- net N$5: now also J2.SIG, U12.1; no longer C1.2, U5.2
- net N$59: now also IC1.22
- net N$60: now also IC1.23
- net N$61: now also IC1.28
- net N$62: now also IC1.29
Routing:
- net OTG_FS_VBUS: track 53.7 -> 0.01 mm
- net MAX-RF: track 33.4 -> 0.00 mm
- net TDO: track 32.3 -> 0.00 mm, vias 1 -> 0
- net PE0: track 33.6 -> 1.50 mm
- net ETH_RXD1: track 31.9 -> 0.00 mm, vias 2 -> 0
- net ETH_MDINT: track 31.0 -> 0.00 mm, vias 2 -> 0
- net ETH_CRS_DV: track 29.9 -> 0.00 mm, vias 2 -> 0
- net ETH_TXD0: track 32.3 -> 2.42 mm, vias 2 -> 0
- net ETH_TX_EN: track 31.2 -> 1.43 mm, vias 2 -> 0
- net ETH_RMII_REF_CLK: track 42.1 -> 12.6 mm
- net ETH_RXD0: track 30.4 -> 0.91 mm, vias 2 -> 0
- net ETH_TXD1: track 32.5 -> 3.16 mm, vias 2 -> 0
- net !RST: track 30.6 -> 1.56 mm, vias 1 -> 0
- net TCK: track 26.8 -> 0.00 mm, vias 2 -> 0
- net SDIO_D3: track 25.8 -> 0.00 mm
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
Commit message: Digital portion of v3 basically laid out, RF sections laid out. To do: verify CPLD power supply, think more about ground/power separation for RF section.
Parts:
- removed LED8: (no value), led-rgb-rohm:KINGBRITE_RGBLED_1.6X1.26
- removed TP3, TP6, TP7: TEST-POINT, Tova:2MM-TEST-POINT
- added LED3: (no value), apdm:LED-3528
- C1, C10, C11, C12, C13, C14, C15, C16, C17, C18, C19, C2, C21, C22, C23, C24, C25, C26, C27, C29, C3, C30, C31, C34, C35, C37, C4, C43, C44, C45, C46, C47, C48, C49, C5, C50, C54, C55, C56, C57, C6, C60, C61, C62, C63, C64, C69, C7, C70, C71, C72, C73, C74, C77, C78, C79, C8, C80, C81, C9: device rcl_custom:0402-C-NOSILK -> rcl_custom:.0402-C-NOSILK
- C20, C36, C39, C40, C41, C42, C51, C52, C53, C58, C59, C65, C67, C68, C75, C76: device rcl_custom:0603-B-NOSILK -> rcl_custom:.0603-B-NOSILK
- C28, C32, C33: device rcl_custom:1206-C@1 -> rcl_custom:1206-C
- TP16: value TEST-POINT -> (none); device Tova:2MM-TEST-POINT -> apdm:PAD-ROUND-0.7+CREAM-NOSILK
- moved J1 60.5 mm to (23.6, 56.6), turned to 0 degrees
- moved C60 51.0 mm to (52.7, 20.7)
- moved TP14 51.0 mm to (55.8, 24.0)
- moved C40 51.0 mm to (49.1, 22.9)
- moved C59 51.0 mm to (53.7, 22.9)
- moved U6 51.0 mm to (51.4, 22.6)
- moved C72 43.6 mm to (68.3, 30.5), turned to 0 degrees
- moved C73 42.3 mm to (63.8, 39.8), turned to 90 degrees
- moved C74 39.9 mm to (71.9, 45.0)
- moved C77 38.7 mm to (72.8, 48.0), turned to 90 degrees
- moved VR1 37.3 mm to (75.6, 46.2), turned to 90 degrees
- moved C76 34.9 mm to (71.9, 46.2), turned to 180 degrees
- moved TP20 34.4 mm to (85.2, 27.4)
- moved TP21 34.3 mm to (71.1, 49.4)
- moved C78 33.2 mm to (71.5, 47.5), turned to 180 degrees
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Connections:
- removed net N$54: TP7.1, U2.4
- removed net N$55: TP6.1, U2.3
- removed net N$56: TP3.1, U2.2
- removed net STM_SPI1_MISO: IC1.38, U2.31
- net 3.3VD: now also LED3.1, LED3.2, LED3.3; no longer LED8.2
- net N$12: now also LED3.5; no longer LED8.4
- net N$18: now also LED3.4; no longer LED8.1
- net N$2: now also TP16.PAD; no longer TP16.1
- net N$37: now also LED3.6; no longer LED8.3
Routing:
- net OTG_FS_VBUS: track 0.01 -> 120.6 mm
- net OTG_FS_DM: track 0.00 -> 37.6 mm
- net OTG_FS_DP: track 0.00 -> 37.4 mm
- net STM_SPI1_MOSI: track 0.00 -> 35.0 mm, vias 0 -> 1
- net STM_SPI1_NSS: track 0.00 -> 32.0 mm, vias 0 -> 1
- net STM_SPI1_SCK: track 0.00 -> 31.0 mm, vias 0 -> 1
- net TDI: track 0.00 -> 26.7 mm
- net TCK: track 0.00 -> 25.7 mm
- net ETH_TXD0: track 2.42 -> 27.5 mm, vias 0 -> 2
- net ETH_TXD1: track 3.16 -> 28.2 mm, vias 0 -> 2
- net TMS: track 0.00 -> 25.0 mm, vias 0 -> 1
- net SDIO_CLK: track 0.00 -> 24.7 mm, vias 0 -> 2
- net SDIO_CMD: track 0.00 -> 24.6 mm, vias 0 -> 2
- net ETH_TX_EN: track 1.43 -> 25.5 mm, vias 0 -> 2
- net SDIO_D0: track 0.00 -> 23.9 mm, vias 0 -> 2
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- added copper zone on layer 1, net AGND
- added copper zone on layer 2, net AGND
- added copper zone on layer 15, net OTG_FS_VBUS
- added copper zone on layer 1, net V18
- removed copper zone on layer 15, net 2.85VA
- removed copper zone on layer 15, net 2.85VD

Commit message: Added link to the MAX2769 google doc, as well as renamed things to be BOM, and committed some minor changes in the layout and notes in the schematic.
Parts:
- moved C19 8.47 mm to (42.3, 4.19)
- moved C69 8.47 mm to (46.9, 12.4)
- moved C70 8.47 mm to (46.9, 11.4)
- moved R21 8.47 mm to (42.4, 2.29)
- moved R24 8.47 mm to (55.0, 11.4)
- moved TP25 8.47 mm to (49.7, 3.05)
- moved TP28 8.47 mm to (44.6, 3.05)
- moved TP9 8.47 mm to (48.8, 7.62)
- moved C66 8.47 mm to (53.8, 6.73)
- moved C67 8.47 mm to (42.8, 12.2)
- moved C68 8.47 mm to (46.0, 14.0)
- moved R22 8.47 mm to (41.9, 9.14)
- moved R23 8.47 mm to (42.0, 7.49)
- moved TP18 8.47 mm to (48.6, 5.46)
- moved TP29 8.47 mm to (42.0, 6.10)
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Routing:
- net OTG_FS_VBUS: track 120.6 -> 122.6 mm

Commit message: 90% done! All analog routed, only 9 airwires left to the CPLD which is trivial (but should be rerouted for easy of routing and also for maybe power domains? In any case, it just needs: stiching, double checking, reduce size of board, tnames, and other pre-production checkouts.
Parts:
- added C82: 100n, rcl_custom:.0402-C-NOSILK
- added SH1: BMI-S-202-SHIELD, hw-laird-bmi-s-202:BMI-S-202
- moved TP10 19.1 mm to (32.9, 7.11), turned to 270 degrees
- moved R9 19.0 mm to (39.1, 10.0), turned to 90 degrees
- moved C41 18.6 mm to (26.8, 22.5), turned to 90 degrees
- moved R8 17.8 mm to (40.4, 41.0), turned to 0 degrees
- moved C67 17.7 mm to (60.3, 14.6), turned to 270 degrees
- moved TP8 16.6 mm to (51.2, 15.1)
- moved C64 16.6 mm to (34.8, 6.60), turned to 0 degrees
- moved C63 16.4 mm to (34.8, 7.62), turned to 0 degrees
- moved C66 15.7 mm to (59.8, 21.2), turned to 90 degrees
- moved C79 15.5 mm to (46.9, 1.40)
- moved U9 15.4 mm to (49.8, 7.87)
- moved TP30 15.4 mm to (50.5, 1.40)
- moved C80 14.9 mm to (47.8, 1.40)
- moved L8 14.8 mm to (33.1, 9.02), turned to 0 degrees
- moved R21 14.6 mm to (57.0, 3.43)
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Connections:
- net N$59 renamed Q1
- net N$60 renamed Q0
- net N$61 renamed I1
- net N$62 renamed I0
- net TCXO-OUT renamed N$54
- removed net N$63: IC1.20
- net AGND: now also SH1.P$1, SH1.P$10, SH1.P$11, SH1.P$12, SH1.P$2, SH1.P$3, SH1.P$4, SH1.P$5, SH1.P$6, SH1.P$7, SH1.P$8, SH1.P$9
- net GND: now also C82.1
- net MAX-RF: now also U10.8; no longer U10.5
- net STQ-RF: now also U10.5; no longer U10.8
- net STQ-VBAT: now also C82.2
Routing:
- net STM_USART6_RX: track 0.00 -> 61.7 mm, vias 0 -> 4
- net STM_USART6_TX: track 0.00 -> 60.6 mm, vias 0 -> 4
- net MAX_!IDLE: track 0.00 -> 56.4 mm, vias 0 -> 4
- net ANTFLAG: track 0.00 -> 54.2 mm, vias 0 -> 4
- net LD: track 0.00 -> 47.4 mm, vias 0 -> 2
- net MAX_CFG_MOSI: track 0.00 -> 44.3 mm, vias 0 -> 2
- net MAX_!SHDN: track 0.00 -> 42.7 mm, vias 0 -> 2
- net MAX_CFG_!CS: track 0.00 -> 38.4 mm, vias 0 -> 2
- net MAX_CFG_SCLK: track 0.00 -> 38.0 mm, vias 0 -> 2
- net I0: track 0.00 -> 35.5 mm
- net I1: track 0.00 -> 35.3 mm
- net Q0: track 0.00 -> 30.5 mm
- net Q1: track 0.00 -> 30.0 mm
- net N$64: track 0.00 -> 29.4 mm
- net STQ-VBAT: track 0.00 -> 28.3 mm, vias 0 -> 2
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- added copper zone on layer 1, net 2.85V-S
- added copper zone on layer 15, net 2.85V-S
- added copper zone on layer 15, net 2.85VA
- added copper zone on layer 15, net 2.85VD
- added copper zone on layer 16, net AGND

Commit message: Shrunk board to 3.0 inches (OoooooooCD!), added the beginnings of stitched vias, cleanup here and there. TODO: final conections to CPLD, then cleanup.
Parts:
- moved TP20 20.3 mm to (64.8, 26.9)
- moved C62 10.4 mm to (74.3, 43.4)
- moved J4 10.4 mm to (74.8, 49.1)
- moved U$14 10.4 mm to (72.1, 4.06)
- moved U$18 10.4 mm to (72.1, 58.2)
- moved TP19 6.99 mm to (12.1, 21.1)
- moved R24 6.36 mm to (62.2, 16.6), turned to 270 degrees
- moved D1 4.43 mm to (62.2, 14.2), turned to 90 degrees
- moved TP2 0.76 mm to (55.9, 45.1)
- moved J7 0.76 mm to (63.6, 47.2)
- moved C66 0.52 mm to (59.9, 20.7), turned to 270 degrees
Routing:
- net OTG_FS_VBUS: track 124.5 -> 109.1 mm
- net OTG_FS_DM: track 37.6 -> 28.2 mm
- net OTG_FS_DP: track 37.4 -> 28.0 mm
- net STQ-VBAT: track 28.3 -> 22.2 mm, vias 2 -> 0
- net N$57: track 14.8 -> 12.5 mm
- net TDO: track 19.8 -> 18.5 mm
- net TDI: track 26.7 -> 25.5 mm
- net TCK: track 25.7 -> 24.9 mm
- net SDIO_D2: track 18.5 -> 17.7 mm
- net SDIO_D1: track 23.6 -> 22.8 mm
- net SDIO_D0: track 23.9 -> 23.1 mm
- net SDIO_CMD: track 24.6 -> 23.9 mm
- net SDIO_CLK: track 24.7 -> 23.9 mm
- net SDIO_D3: track 21.4 -> 20.6 mm
- net GND: vias 206 -> 325
Other:
- board size 86.6 x 62.2 mm -> 76.2 x 62.2 mm
- board text added: "jGPS + COTS Board V3 Portland State Aerospace Society http://psas.pdx.edu/ Jenner Hanni and Andrew Greenberg"
- board text removed: "GPS Raw Data Capture Board V2 Portland State Aerospace - http://psas.pdx.edu/ - Jenner Hanni and Andrew Greenberg"
