File: v3-gps.brd (EAGLE design)
At the start: 76.2 x 62.2 mm, 182 parts, among them IC1 XC2C32A_VQ44_2, J1 1.27MM-SWD-CONNECTOR, J2 CON_SMA-ENDFIRE_EMERSON_EMERS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, J3 ROCKETNET-CONNECTOR-16M, J4 ZX62D-B-5P8, J7 CON_HIROSE_DM3D(MICROSD), Q1 NTR4101P, T1 ALT4532, T2 ALT4532, U1 MAX2769, U10 BP2G+, U11 MAX8510EXK29+T, U12 AVAGO-ALM-GPXX, U2 STM32F4V_100PIN_GPSBOARD, U3 KSZ8081, U4 7Q-16.368MBG-T, U6 MAX8510EXK29+T, U7 MAX8510EXK29+T, U8 LMZ12001, U9 VENUS638FLPX-L, X1 25 MHz

Commit message: Couldn't help myself; wired all the things. Left to do: clean-up, mostly. Verify CPLD pins, verify MAX connections and SkyTraq connections, design review, etc.
Parts:
- moved C52 1.53 mm to (44.2, 41.0), turned to 0 degrees
- moved R20 1.44 mm to (54.0, 45.6)
- moved R14 1.44 mm to (54.0, 43.1)
- moved R16 1.44 mm to (54.0, 44.3)
- moved C50 1.37 mm to (47.9, 57.0)
- moved LED5 1.35 mm to (51.7, 45.6)
- moved LED2 1.35 mm to (51.7, 43.1)
- moved LED4 1.35 mm to (51.7, 44.3)
- moved C51 1.17 mm to (49.9, 56.1), turned to 270 degrees
- moved TP2 0.65 mm to (56.5, 45.2)
- moved C48 0.38 mm to (46.6, 42.5)
- moved TP16 0.28 mm to (30.2, 35.7)
- moved R43 0.25 mm to (33.1, 39.2)
- moved C49 0.18 mm to (33.5, 59.4)
- moved R19 0.13 mm to (36.1, 59.4)
Connections:
- net N$43 renamed VCAP_1
- net N$45 renamed VCAP_2
- net N$9 renamed BOOT0
- new net N$9: IC1.1
- net N$64: now also IC1.32; no longer IC1.21
- net Q0: now also IC1.30; no longer IC1.23
- net Q1: now also IC1.31; no longer IC1.22
- net STM_SPI1_MOSI: now also IC1.21; no longer IC1.36
- net STM_SPI1_NSS: now also IC1.22; no longer IC1.34
- net STM_SPI1_SCK: now also IC1.23; no longer IC1.37
Routing:
- net STM_SPI1_MOSI: track 16.3 -> 29.4 mm, vias 1 -> 2
- net STM_SPI1_NSS: track 13.1 -> 25.5 mm, vias 1 -> 2
- net STM_SPI1_SCK: track 12.0 -> 22.5 mm, vias 1 -> 2
- net GND: track 8.94 -> 14.3 mm, vias 325 -> 324
- net 3.3VD: track 57.6 -> 53.7 mm
- net I1: track 35.3 -> 38.6 mm
- net I0: track 35.5 -> 38.5 mm
- net Q0: track 30.5 -> 33.3 mm
- net ANTFLAG: track 54.2 -> 51.6 mm
- net Q1: track 30.0 -> 32.5 mm
- net N$64: track 29.4 -> 32.0 mm
- net N$57: track 12.5 -> 14.9 mm
- net N$49: track 6.77 -> 5.31 mm
- net N$50: track 6.14 -> 4.84 mm
- net 3.3VD1: track 7.16 -> 6.30 mm
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Other:
- outline, holes or cut-outs redrawn

Commit message: More tweaks, notes, board now almost done. Still to do: 42 MHz clock, double check power plane routing, 16MHz clock cleanup.
Parts:
- added R26: 10k, rcl_custom:0402-C-NOSILK@1
- C71, C72, C73, C74: value 100p -> 100n
- moved TP19 65.9 mm to (77.9, 24.3)
- moved TP18 24.5 mm to (77.9, 21.7)
- moved TP20 13.1 mm to (77.9, 27.2)
- moved C72 0.80 mm to (54.2, 27.2), turned to 180 degrees
- moved C71 0.52 mm to (64.9, 34.4)
- moved TP16 0.25 mm to (30.2, 35.9)
- moved TP17 0.25 mm to (20.3, 43.7)
- moved C73 0.13 mm to (50.5, 36.3)
- moved J1 0.13 mm to (23.6, 56.5)
Connections:
- net N$64 renamed MAX-CLKOUT
- net AGND: now also U12.2, U12.3, U12.4, U12.9, U12.P$1, U12.P$2
- net GND: now also R26.1; no longer U12.2, U12.3, U12.4, U12.9, U12.P$1, U12.P$2
- net N$9: now also IC1.18, R26.2; no longer IC1.1
Routing:
- net 3.3VD: track 53.7 -> 46.4 mm, vias 64 -> 63
- net GND: track 14.3 -> 12.1 mm, vias 324 -> 335
- net N$9: track 0.00 -> 1.78 mm
- net AGND: track 4.49 -> 5.31 mm
- net SDIO_D2: track 17.7 -> 18.2 mm
- net OTG_FS_VBUS: track 109.1 -> 108.8 mm, vias 8 -> 7
Other:
- board text added: "3.3"
- board text added: "GND"
- board text added: "TMS"

Commit message: Done! Removed power split plane because that was stupid on further reflection, added clock comparator, cleaned up ERCs and DRCs.
Parts:
- added C83, C84: 100n, rcl_custom:.0402-C-NOSILK
- added R27: 10k, rcl_custom:0402-C-NOSILK@1
- added U5: LT1719S6, ic-comparator-linear-lt1719:SOT23-6
- U2: value STM32F4V_100PIN_GPSBOARD -> STM32F407VG
- moved TP19 61.3 mm to (16.5, 23.4)
- moved TP20 44.7 mm to (37.2, 8.64)
- moved TP18 30.5 mm to (47.4, 23.1)
- moved R26 0.40 mm to (56.8, 41.8), turned to 270 degrees
Connections:
- net ANTFLAG renamed MAX_ANTFLAG
- net DEBUG-PHY-MODWIRE renamed ETH_DEBUG
- net EPHY_NRST renamed ETH_PHY_NRST
- net LD renamed MAX_LD
- net MAX_CFG_MOSI renamed MAX_CFG_SPI2_MOSI
- net MAX_CFG_SCLK renamed MAX_CFG_SPI2_SCLK
- net MCO1-ETH-CLK renamed ETH_MCO1_CLK
- net N$11 renamed RGB-B
- net N$34 renamed RGB-R
- net N$49 renamed LED4
- net N$50 renamed LED5
- net N$9 renamed CPLD_IN_ONLY
- net OTG_FS_DM renamed USB_FS_DM
- net OTG_FS_DP renamed USB_FS_DP
- net OTG_FS_VBUS renamed USB_FS_VBUS
- net PE0 renamed SDIO_PWR
- net STM_SPI1_SCK renamed MAX_OUT_SPI1_SCK
- removed net 3.3VD1: LED2.C, U2.55
- removed net STM_SPI1_MOSI: IC1.21, U2.91
- removed net STM_SPI1_NSS: IC1.22, U2.29
- new net MAX_OUT_SPI1_MOSI: IC1.20, U2.91
- new net MAX_OUT_SPI1_NSS: IC1.21, U2.29
- new net MAX_OUT_SPI_CLK: IC1.22, U2.53
- new net N$43: C84.1, R27.1, U5.1
- new net N$45: R27.2, U1.16, U5.3
- new net RGB-G: R39.2, U2.61
- net 3.3VD: now also C83.1, U5.4
- net GND: now also C83.2, C84.2, U5.2, U5.6
- net LED2: now also LED2.C, U2.55; no longer R39.2, U2.61
- net MAX-CLKOUT: now also U5.5; no longer U1.16
Routing:
- net N$45: track 0.00 -> 34.9 mm
- net MAX_OUT_SPI1_MOSI: track 0.00 -> 29.7 mm, vias 0 -> 2
- net STM_SPI1_MOSI: track 29.4 -> 0.00 mm, vias 2 -> 0
- net MAX-CLKOUT: track 32.0 -> 5.33 mm
- net MAX_OUT_SPI1_NSS: track 0.00 -> 25.9 mm, vias 0 -> 2
- net STM_SPI1_NSS: track 25.5 -> 0.00 mm, vias 2 -> 0
- net MAX_OUT_SPI_CLK: track 0.00 -> 10.6 mm
- net 3.3VD1: track 6.30 -> 0.00 mm
- net ETH_MDIO: track 23.8 -> 28.6 mm
- net LED2: track 1.95 -> 6.30 mm
- net MAX_!IDLE: track 56.5 -> 52.8 mm
- net ETH_MDC: track 28.1 -> 31.8 mm
- net N$43: track 0.00 -> 2.72 mm
- net RGB-G: track 0.00 -> 1.95 mm
- net USB_FS_VBUS: track 108.8 -> 110.0 mm, vias 7 -> 8
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
Commit message: Forgot to add a few ground vias....
Routing:
- net GND: vias 334 -> 336
Changed lines of the file:
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@@
 <layer number="27" name="tValues" color="7" fill="1" visible="no" active="yes"/>
 <layer number="28" name="bValues" color="7" fill="1" visible="no" active="yes"/>
-<layer number="29" name="tStop" color="7" fill="3" visible="no" active="yes"/>
+<layer number="29" name="tStop" color="7" fill="3" visible="yes" active="yes"/>
 <layer number="30" name="bStop" color="7" fill="6" visible="no" active="yes"/>
 <layer number="31" name="tCream" color="7" fill="4" visible="no" active="yes"/>
@@
 <via x="57.785" y="26.035" extent="1-16" drill="0.254"/>
 <via x="53.213" y="27.178" extent="1-16" drill="0.254"/>
-<via x="50.165" y="26.035" extent="1-16" drill="0.254"/>
+<via x="50.165" y="26.162" extent="1-16" drill="0.254"/>
 <via x="47.625" y="26.035" extent="1-16" drill="0.254"/>
 <via x="60.325" y="25.019" extent="1-16" drill="0.254"/>
@@
 <contactref element="C84" pad="2"/>
 <contactref element="U5" pad="6"/>
+<via x="47.752" y="27.559" extent="1-16" drill="0.254"/>
+<via x="47.117" y="28.194" extent="1-16" drill="0.254"/>
 </signal>
 <signal name="SD-VDD">

Commit message: Forgot to add comparator library earlier. Added bzillions of test points, to CPLD and STM, for future mod wires :) Also left RF class isolate to 25 mils, forgot to reset that during the last commit. Nothing left as far as I can see.
Parts:
- added TP23, TP24, TP3, TP31, TP34, TP35, TP36, TP37, TP38, TP39, TP40, TP6, TP7: TEST-POINT15MIL-TEST-POINT, Tova:15MIL-TEST-POINT
- TP1, TP10, TP11, TP12, TP13, TP14, TP15, TP17, TP18, TP19, TP20, TP21, TP22, TP25, TP26, TP27, TP28, TP29, TP30, TP32, TP33, TP8, TP9: value TEST-POINT -> TEST-POINT15MIL-TEST-POINT; device Tova:2MM-TEST-POINT -> Tova:15MIL-TEST-POINT
Connections:
- net MAX_OUT_SPI1_MOSI renamed CPLD_OUT_SPI1_MOSI
- net MAX_OUT_SPI1_NSS renamed CPLD_OUT_SPI1_NSS
- net MAX_OUT_SPI1_SCK renamed CPLD_OUT_SPI1_SCK
- net MAX_OUT_SPI_CLK renamed CPLD_OUT_SPI_CLK
- new net CPLD_DEBUG: IC1.19, U2.59
- new net N$11: IC1.42, TP23.P$1
- new net N$34: IC1.40, TP31.P$1
- new net N$49: IC1.38, TP34.P$1
- new net N$50: TP35.P$1, U2.86
- new net N$55: TP36.P$1, U2.88
- new net N$56: TP37.P$1, U2.82
- new net N$59: TP38.P$1, U2.35
- new net N$60: TP39.P$1, U2.2
- new net N$61: TP40.P$1, U2.4
- new net N$9: IC1.44, TP24.P$1
- net 2.85V-S: now also TP9.P$1; no longer TP9.1
- net 2.85VA: now also TP15.P$1; no longer TP15.1
- net 2.85VD: now also TP14.P$1; no longer TP14.1
- net 3.3VD: now also TP13.P$1; no longer TP13.1
- net ANTBIAS: now also TP10.P$1; no longer TP10.1
- net AUX1: now also TP22.P$1; no longer TP22.1
- net AUX2: now also TP26.P$1; no longer TP26.1
- net AUX3: now also TP32.P$1; no longer TP32.1
- net AUX4: now also TP33.P$1; no longer TP33.1
- net GND: now also TP17.P$1, TP18.P$1, TP19.P$1, TP20.P$1, TP3.P$1, TP6.P$1, TP7.P$1; no longer TP17.1, TP18.1, TP19.1, TP20.1
- net N$1: now also TP11.P$1; no longer TP11.1
- net N$22: now also TP29.P$1; no longer TP29.1
- net N$25: now also TP8.P$1; no longer TP8.1
- net STM_USART6_RX: now also TP27.P$1; no longer TP27.1
- net STM_USART6_TX: now also TP25.P$1; no longer TP25.1
- net STQ-!RST: now also TP28.P$1; no longer TP28.1
- net STQ-PPS: now also TP30.P$1; no longer TP30.1
- net V18: now also TP21.P$1; no longer TP21.1
- net VIN: now also TP12.P$1; no longer TP12.1
- net XTAL: now also TP1.P$1; no longer TP1.1
Routing:
- net CPLD_DEBUG: track 0.00 -> 21.3 mm, vias 0 -> 2
- net N$61: track 0.00 -> 2.81 mm
- net N$59: track 0.00 -> 2.35 mm
- net N$50: track 0.00 -> 2.25 mm
- net N$55: track 0.00 -> 2.08 mm
- net N$56: track 0.00 -> 2.06 mm
- net N$49: track 0.00 -> 1.70 mm
- net N$9: track 0.00 -> 1.69 mm
- net N$34: track 0.00 -> 1.68 mm
- net N$11: track 0.00 -> 1.67 mm
- net N$60: track 0.00 -> 1.59 mm
- net MAX_ANTFLAG: track 51.6 -> 52.7 mm

Commit message: Added part numbers to some of the odder components. Found the supercap is no longer made, so switched it to an instock item. Also checked on other components, like the LNA and splitter. Cleaned up schematic notes, added comments, added stiching around RF lines (not necessary, but yay OCD) and ran ERC and DRCs again.
Parts:
- removed C66: (no value), SparkFun-Passives:EN_J2
- removed TP37: TEST-POINT15MIL-TEST-POINT, Tova:15MIL-TEST-POINT
- added C85: DSK-3R3H334T-HL, cap-elna-ds:CAP-ELNA-DS-SERIES
- LED3: value (none) -> SMLV56RGB1W1
- U12: value AVAGO-ALM-GPXX -> ALM-GP002
- U8: value LMZ12001 -> LMZ12001TZ-ADJ/NOPB
- moved TP35 0.90 mm to (40.9, 59.2)
- moved TP36 0.90 mm to (39.8, 59.2)
Connections:
- removed net N$56: TP37.P$1, U2.82
- net GND: now also C85.-; no longer C66.-
- net STQ-VBAT: now also C85.+; no longer C66.+
Routing:
- net N$56: track 2.06 -> 0.00 mm
- net N$50: track 2.25 -> 1.30 mm
- net N$55: track 2.08 -> 1.25 mm
- net GND: vias 336 -> 409

Commit message: So many little tweaks: updated ground planes, created BOM and then found out that everything doesn't exist anymore, so found new part numbers and in some cases (like the supercap) found new parts, arranged TNAMES, stitched RF lines, updated values for LED Rs, and more that I've forgotten already.
Parts:
- C19, C79: device rcl_custom:.0402-C-NOSILK -> rcl_custom:.0603-C-NOSILK
- C62: value 100n 50V -> 1n 2kv
- R12: value 1.5k -> 10k
- R14, R16, R20: value 1k -> 3.32k
- R38: value 400 -> 3.32k
- R39: value 110 -> 3.32k
- R40: value 900 -> 3.32k
- TP16: device apdm:PAD-ROUND-0.7+CREAM-NOSILK -> testpad:TP06R
- U1: value MAX2769 -> MAX2769ETI+
- U14: value MIC5025-1.8V -> MIC5319-1.8V
- moved TP29 4.50 mm to (60.6, 8.76)
- moved C80 2.44 mm to (49.7, 2.92), turned to 0 degrees
- moved C19 2.33 mm to (58.5, 6.86)
- moved C22 1.98 mm to (57.4, 6.60)
- moved U11 1.98 mm to (59.2, 16.3)
- moved C24 1.98 mm to (57.4, 4.83)
- moved C69 1.98 mm to (56.8, 16.5)
- moved U9 1.98 mm to (51.2, 9.27)
- moved C68 1.98 mm to (59.3, 13.5)
- moved C70 1.98 mm to (59.1, 14.6)
- moved LED7 1.98 mm to (59.8, 10.0)
- moved R23 1.98 mm to (57.8, 10.0)
- moved TP7 1.98 mm to (61.8, 13.3)
- moved TP30 1.98 mm to (51.9, 2.79)
- moved R21 1.98 mm to (58.4, 4.83)
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- renumbered IC1 to U13, VR1 to U14
Connections:
- net CPLD_OUT_SPI_CLK renamed CPLD_OUT_SPI_CLK_SRC
- net N$22 renamed LED/GPIO
- net N$25 renamed RTC
- net N$2: now also TP16.TP; no longer TP16.PAD
Routing:
- net 3.3VD: track 46.4 -> 42.2 mm
- net 2.85V-S: track 13.2 -> 10.3 mm, vias 14 -> 15
- net LED/GPIO: track 2.99 -> 5.61 mm
- net STQ-VBAT: track 22.4 -> 24.7 mm
- net STM_USART6_RX: track 61.7 -> 59.5 mm
- net AGND: track 5.31 -> 7.41 mm, vias 11 -> 13
- net STQ-RF: track 25.0 -> 26.9 mm
- net RTC: track 2.92 -> 1.66 mm
- net STM_USART6_TX: track 60.6 -> 59.8 mm
- net GND: vias 409 -> 414
- added copper zone on layer 15, net AGND

Commit message: OK now it's really done. tnames cleaned up more, ERC and DRC gone over, BOM updated and price calculated, found lack of stock on certain items, etc.
Parts:
- moved TP21 7.45 mm to (63.5, 40.4)
- moved C84 0.89 mm to (47.8, 29.5)
- moved R27 0.89 mm to (49.5, 31.4)
- moved U5 0.89 mm to (50.3, 29.0)
- moved R26 0.85 mm to (56.4, 42.5)
- moved C71 0.76 mm to (64.9, 35.2)
- moved C72 0.76 mm to (54.2, 27.9)
- moved C73 0.76 mm to (50.5, 37.1)
- moved C75 0.76 mm to (65.2, 42.8)
- moved C76 0.76 mm to (58.5, 43.6)
- moved C78 0.76 mm to (58.2, 44.8)
- moved JP1 0.76 mm to (67.8, 37.2)
- moved TP23 0.76 mm to (60.2, 27.7)
- moved TP24 0.76 mm to (61.8, 27.7)
- moved TP31 0.76 mm to (58.5, 27.7)
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Routing:
- net V18: track 1.71 -> 4.01 mm
- net CPLD_OUT_SPI1_NSS: track 25.9 -> 25.0 mm
- net 2.85VA: track 16.7 -> 15.9 mm
- net Q1: track 32.5 -> 33.3 mm
- net Q0: track 33.3 -> 34.1 mm
- net I1: track 38.6 -> 39.4 mm
- net I0: track 38.5 -> 39.2 mm
- net CPLD_OUT_SPI_CLK_SRC: track 10.6 -> 9.83 mm
- net CPLD_OUT_SPI1_SCK: track 22.8 -> 22.0 mm
- net CPLD_DEBUG: track 21.3 -> 20.6 mm
- net CPLD_OUT_SPI1_MOSI: track 29.7 -> 29.1 mm
- net GND: vias 414 -> 419
