File: v3-gps.brd (EAGLE design)
At the start: 76.2 x 62.2 mm, 199 parts, among them J1 1.27MM-SWD-CONNECTOR, J2 CON_SMA-ENDFIRE_EMERSON_EMERS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, J3 ROCKETNET-CONNECTOR-16M, J4 ZX62D-B-5P8, J7 CON_HIROSE_DM3D(MICROSD), Q1 NTR4101P, T1 ALT4532, T2 ALT4532, U1 MAX2769ETI+, U10 BP2G+, U11 MAX8510EXK29+T, U12 ALM-GP002, U13 XC2C32A_VQ44_2, U14 MIC5319-1.8V, U2 STM32F407VG, U3 KSZ8081, U4 7Q-16.368MBG-T, U5 LT1719S6, U6 MAX8510EXK29+T, U7 MAX8510EXK29+T, U8 LMZ12001TZ-ADJ/NOPB, U9 VENUS638FLPX-L, X1 25 MHz

Commit message: Added 1.8V library, cleaned up power layer after seeing gerbers, added more comments on schematic after viewing PDF, and commited both for those folks without EAGLE.
Parts:
- moved C54 0.13 mm to (18.9, 50.5)
Connections:
- net V18 renamed 1.8V
Changed lines of the file:
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@@
 <layers>
 <layer number="1" name="Top" color="4" fill="1" visible="yes" active="yes"/>
-<layer number="2" name="GND" color="7" fill="1" visible="no" active="yes"/>
+<layer number="2" name="GND" color="7" fill="1" visible="yes" active="yes"/>
 <layer number="3" name="Route3" color="4" fill="3" visible="no" active="no"/>
 <layer number="4" name="Route4" color="1" fill="4" visible="no" active="no"/>
@@
 <layer number="13" name="Route13" color="4" fill="5" visible="no" active="no"/>
 <layer number="14" name="Route14" color="1" fill="6" visible="no" active="no"/>
-<layer number="15" name="SUPPLY" color="14" fill="1" visible="no" active="yes"/>
+<layer number="15" name="SUPPLY" color="14" fill="1" visible="yes" active="yes"/>
 <layer number="16" name="Bottom" color="1" fill="1" visible="yes" active="yes"/>
 <layer number="17" name="Pads" color="2" fill="1" visible="yes" active="yes"/>
@@
 <layer number="37" name="tTest" color="7" fill="1" visible="no" active="yes"/>
 <layer number="38" name="bTest" color="7" fill="1" visible="no" active="yes"/>
-<layer number="39" name="tKeepout" color="4" fill="11" visible="yes" active="yes"/>
+<layer number="39" name="tKeepout" color="4" fill="11" visible="no" active="yes"/>
 <layer number="40" name="bKeepout" color="1" fill="11" visible="no" active="yes"/>
-<layer number="41" name="tRestrict" color="4" fill="10" visible="yes" active="yes"/>
+<layer number="41" name="tRestrict" color="4" fill="10" visible="no" active="yes"/>
 <layer number="42" name="bRestrict" color="1" fill="10" visible="no" active="yes"/>
 <layer number="43" name="vRestrict" color="2" fill="10" visible="no" active="yes"/>
@@
 <attribute name="VALUE" x="10.182" y="49.746" size="1" layer="27" ratio="10" rot="R90"/>
 </element>
-<element name="C54" library="rcl_custom" package=".0402-C-NOSILK" value="100n" x="19.05" y="50.546" smashed="yes" rot="R90">
-<attribute name="NAME" x="19.431" y="47.498" size="0.635" layer="25" font="vector" ratio="20" rot="R90"/>
-<attribute name="VALUE" x="20.85" y="49.746" size="1" layer="27" ratio="10" rot="R90"/>
+<element name="C54" library="rcl_custom" package=".0402-C-NOSILK" value="100n" x="18.923" y="50.546" smashed="yes" rot="R90">
+<attribute name="NAME" x="19.304" y="47.498" size="0.635" layer="25" font="vector" ratio="20" rot="R90"/>
+<attribute name="VALUE" x="20.723" y="49.746" size="1" layer="27" ratio="10" rot="R90"/>
 </element>
 <element name="J1" library="con-swd" package="1.27MM_2X5" value="1.27MM-SWD-CONNECTOR" x="23.622" y="56.515" smashed="yes">
@@
 </element>
 <element name="U13" library="dp_devices" package="VQ44" value="XC2C32A_VQ44_2" x="57.785" y="35.052" smashed="yes" rot="R180">
-<attribute name="NAME" x="64.389" y="30.734" size="0.635" layer="25" font="vector" ratio="20"/>
+<attribute name="NAME" x="62.992" y="29.845" size="0.635" layer="25" font="vector" ratio="20"/>
 <attribute name="VALUE" x="60.96" y="36.8046" size="1.397" layer="27" ratio="10" rot="R180"/>
 </element>
@@
 <vertex x="46.482" y="27.178"/>
 <vertex x="46.482" y="25.273"/>
-<vertex x="60.96" y="25.273"/>
-<vertex x="60.96" y="15.24"/>
+<vertex x="63.881" y="25.273"/>
+<vertex x="63.881" y="15.24"/>
 <vertex x="52.324" y="15.24"/>
 <vertex x="52.324" y="22.733"/>
 <vertex x="30.48" y="22.733"/>
-<vertex x="30.48" y="20.193"/>
-<vertex x="25.019" y="20.193"/>
+<vertex x="30.48" y="20.447"/>
+<vertex x="25.019" y="20.447"/>
 <vertex x="25.019" y="25.273"/>
 <vertex x="39.624" y="25.273"/>
@@
 <vertex x="24.638" y="50.292"/>
 </polygon>
-<via x="18.796" y="49.403" extent="1-16" drill="0.254"/>
-<via x="19.304" y="49.403" extent="1-16" drill="0.254"/>
+<via x="18.669" y="49.403" extent="1-16" drill="0.254"/>
+<via x="19.177" y="49.403" extent="1-16" drill="0.254"/>
 <via x="20.701" y="48.895" extent="1-16" drill="0.254"/>
 <via x="20.193" y="48.895" extent="1-16" drill="0.254"/>
-<via x="23.495" y="48.641" extent="1-16" drill="0.254"/>
+<via x="23.495" y="46.355" extent="1-16" drill="0.254"/>
 <via x="22.987" y="48.641" extent="1-16" drill="0.254"/>
-<via x="22.479" y="48.641" extent="1-16" drill="0.254"/>
+<via x="22.479" y="46.355" extent="1-16" drill="0.254"/>
 <via x="17.78" y="45.466" extent="1-16" drill="0.254"/>
 <contactref element="J1" pad="VTREF"/>
@@
 <via x="21.844" y="41.656" extent="1-16" drill="0.254"/>
 <via x="22.86" y="41.656" extent="1-16" drill="0.254"/>
-<via x="22.352" y="41.656" extent="1-16" drill="0.254"/>
+<via x="22.352" y="42.672" extent="1-16" drill="0.254"/>
 <via x="33.02" y="45.72" extent="1-16" drill="0.254"/>
 <wire x1="31.747" y1="45.792" x2="32.948" y2="45.792" width="0.254" layer="1"/>
@@
 <via x="73.279" y="40.767" extent="1-16" drill="0.254"/>
 <via x="72.898" y="40.513" extent="1-16" drill="0.254"/>
-<polygon width="0.127" layer="2" isolate="0.254" thermals="no" rank="6">
+<polygon width="0.127" layer="2" isolate="0.2032" thermals="no" rank="6">
 <vertex x="0" y="62.23"/>
 <vertex x="0" y="25.781"/>
@@
 <via x="21.971" y="50.927" extent="1-16" drill="0.254"/>
 <via x="20.701" y="52.197" extent="1-16" drill="0.254"/>
-<via x="18.288" y="50.927" extent="1-16" drill="0.254"/>
+<via x="17.907" y="50.927" extent="1-16" drill="0.254"/>
 <via x="63.5" y="56.134" extent="1-16" drill="0.254"/>
 <via x="63.5" y="58.674" extent="1-16" drill="0.254"/>
@@
 <contactref element="TP14" pad="P$1"/>
 <polygon width="0.127" layer="15">
-<vertex x="51.054" y="15.748"/>
-<vertex x="51.054" y="22.479"/>
-<vertex x="30.861" y="22.479"/>
+<vertex x="51.943" y="15.748"/>
+<vertex x="51.943" y="22.352"/>
+<vertex x="30.861" y="22.352"/>
 <vertex x="30.861" y="15.748"/>
 </polygon>
@@
 <contactref element="U9" pad="58"/>
 <polygon width="0.127" layer="15">
-<vertex x="45.847" y="14.859"/>
-<vertex x="45.847" y="1.778"/>
-<vertex x="66.167" y="1.778"/>
-<vertex x="66.167" y="14.859"/>
+<vertex x="48.006" y="14.859"/>
+<vertex x="48.006" y="1.778"/>
+<vertex x="63.881" y="1.778"/>
+<vertex x="63.881" y="14.859"/>
 </polygon>
 <via x="49.149" y="2.286" extent="1-16" drill="0.254"/>
@@
 <wire x1="59.563" y1="45.662" x2="60.51" y2="45.662" width="0.127" layer="1"/>
 </signal>
-<signal name="V18">
-<contactref element="C76" pad="1"/>
-<contactref element="U14" pad="5"/>
-<contactref element="TP21" pad="P$1"/>
-<contactref element="C78" pad="1"/>
-<contactref element="C77" pad="1"/>
-<contactref element="U13" pad="15"/>
-<contactref element="C74" pad="1"/>
-<polygon width="0.127" layer="1" isolate="0.2032" thermals="no">
-<vertex x="59.817" y="39.878"/>
-<vertex x="59.817" y="41.91"/>
-<vertex x="61.722" y="41.91"/>
-<vertex x="61.722" y="45.212"/>
-<vertex x="58.42" y="45.212"/>
-<vertex x="58.42" y="41.91"/>
-<vertex x="58.928" y="41.91"/>
-<vertex x="58.928" y="39.878"/>
-</polygon>
-<wire x1="63.5" y1="40.386" x2="62.865" y2="40.386" width="0.127" layer="1"/>
-<wire x1="62.865" y1="40.386" x2="62.357" y2="40.894" width="0.127" layer="1"/>
-<wire x1="62.357" y1="40.894" x2="62.357" y2="41.783" width="0.127" layer="1"/>
-<wire x1="62.357" y1="41.783" x2="61.595" y2="42.545" width="0.127" layer="1"/>
-<wire x1="61.595" y1="42.545" x2="60.996" y2="42.545" width="0.127" layer="1"/>
-<wire x1="60.996" y1="42.545" x2="60.93" y2="42.611" width="0.127" layer="1"/>
-</signal>
 <signal name="Q1">
 <contactref element="U1" pad="17"/>
@@
 <wire x1="29.972" y1="54.737" x2="28.956" y2="54.737" width="0.127" layer="1"/>
 </signal>
+<signal name="1.8V">
+<contactref element="C74" pad="1"/>
+<contactref element="U13" pad="15"/>
+<contactref element="TP21" pad="P$1"/>
+<contactref element="C77" pad="1"/>
+<contactref element="C76" pad="1"/>
+<contactref element="C78" pad="1"/>
+<contactref element="U14" pad="5"/>
+<polygon width="0.127" layer="1" isolate="0.2032" thermals="no">
+<vertex x="59.817" y="39.878"/>
+<vertex x="59.817" y="41.91"/>
+<vertex x="61.722" y="41.91"/>
+<vertex x="61.722" y="45.212"/>
+<vertex x="58.42" y="45.212"/>
+<vertex x="58.42" y="41.91"/>
+<vertex x="58.928" y="41.91"/>
+<vertex x="58.928" y="39.878"/>
+</polygon>
+<wire x1="60.93" y1="42.611" x2="62.037" y2="42.611" width="0.127" layer="1"/>
+<wire x1="62.037" y1="42.611" x2="62.357" y2="42.291" width="0.127" layer="1"/>
+<wire x1="62.357" y1="42.291" x2="62.357" y2="41.021" width="0.127" layer="1"/>
+<wire x1="62.357" y1="41.021" x2="62.992" y2="40.386" width="0.127" layer="1"/>
+<wire x1="62.992" y1="40.386" x2="63.5" y2="40.386" width="0.127" layer="1"/>
+</signal>
 </signals>

Commit message: Widended interface between digital and RF sections, added spacing to high speed MAX outputs, Added THads for scope ground clips and silk area for board #. Added GPS_RESET, and cleaned up STM scehamtic a bit.
Parts:
- moved TP3 17.2 mm to (42.9, 9.27)
- moved R27 1.33 mm to (48.3, 31.0)
- moved C13 0.13 mm to (29.3, 16.1)
Connections:
- net N$45 renamed MAX_CLK_OUT
- net VDD_1.2_ETH_SUPP renamed VDD_1.2
- new net CPLD_RESET: U13.14, U2.69
Routing:
- net CPLD_RESET: track 0.00 -> 26.1 mm, vias 0 -> 2
- net I0: track 39.2 -> 36.6 mm
- net I1: track 39.4 -> 37.2 mm
- net Q1: track 33.3 -> 31.7 mm
- net MAX_CLK_OUT: track 35.1 -> 33.5 mm
- net Q0: track 34.1 -> 32.6 mm
- net STM_USART6_RX: track 59.5 -> 58.9 mm
- net STM_USART6_TX: track 59.8 -> 59.2 mm
- net GND: vias 419 -> 440
Other:
- board text added: "jGPS + COTS Board v3.0 Portland State Aerospace Society http://psas.pdx.edu/ 2015/04/01 Jenner Hanni & Andrew Greenberg"
- board text removed: "jGPS + COTS Board V3 Portland State Aerospace Society http://psas.pdx.edu/ Jenner Hanni and Andrew Greenberg"
