File: v3-gps.sch (EAGLE design)
At the start: 168 parts, among them J1 1.27MM-SWD-CONNECTOR, J2 CON_SMA-ENDFIRE_EMERSON_EMERS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, J3 ROCKETNET-CONNECTOR-16M, J4 ZX62D-B-5P8, J7 CON_HIROSE_DM3D(MICROSD), Q1 NTR4101P, T1 ALT4532, T2 ALT4532, U1 MAX2769, U10 MINICIRCUITS-BP2G, U11 MAX8510EXK29+T, U2 STM32F4V_100PIN_GPSBOARD, U3 KSZ8081, U4 7Q-16.368MBG-T, U5 XC2401A8167R-G, U6 MAX8510EXK29+T, U7 MAX8510EXK29+T, U8 LMZ12001, U9 VENUS638FLPX-L, X1 25 MHz

Commit message: First commit of the GPS v3 board, which includes the CPLD and SkyTraq ICs.
Parts:
- U10: value MINICIRCUITS-BP2G -> BP2G+
Changed lines of the file:
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@@
 <setting verticaltext="up"/>
 </settings>
-<grid distance="0.05" unitdist="inch" unit="inch" style="lines" multiple="2" display="yes" altdistance="0.01" altunitdist="inch" altunit="inch"/>
+<grid distance="0.1" unitdist="inch" unit="inch" style="lines" multiple="1" display="no" altdistance="0.01" altunitdist="inch" altunit="inch"/>
 <layers>
 <layer number="1" name="Top" color="4" fill="1" visible="no" active="no"/>
@@
 <part name="C1" library="rcl_custom" deviceset="C-EU" device="0402-C-NOSILK" value="100p"/>
 <part name="U9" library="SparkFun-RF" deviceset="VENUS638FLPX-L" device=""/>
-<part name="U10" library="minicircuits-splitter" deviceset="MINICIRCUITS-BP2G" device=""/>
+<part name="U10" library="minicircuits-splitter" deviceset="MINICIRCUITS-BP2G" device="" value="BP2G+"/>
 <part name="DIG_GND36" library="supply" deviceset="GND_BAR" device="" value="GND"/>
 <part name="AGND1" library="supply1" deviceset="AGND" device=""/>

Commit message: More rough drafting on the CPLD. Added 1.8V supply (kind of), added some cleanup notes on clock, etc. TODO: everything still, including cleanup up 1.8V supply and probably splitting the power domains on the CPLD.
Parts:
- added C71, C72, C73, C74: 100p, rcl_custom:C-EU0402-C-NOSILK
- added C75, C76: 1u, rcl_custom:C-EU0603-B-NOSILK
- added C77: 10n, rcl_custom:C-EU0402-C-NOSILK
- added C78: 100n, rcl_custom:C-EU0402-C-NOSILK
- added IC1: XC2C32A_VQ44_2, dp_devices:XC2C32A_VQ44_2
- added JP1: (no value), pinhead:PINHD-1X6
- added TP21: TEST-POINT, Tova:TEST-POINT
- added VR1: MIC5025-1.8V, dp_devices:MIC5205
Connections:
- new net N$3: IC1.TMS, JP1.6
- new net N$35: IC1.TDI, JP1.5
- new net N$53: IC1.TDO, JP1.4
- new net N$57: IC1.TCK, JP1.3
- new net N$58: C77.2, VR1.BYP
- new net N$59: U1.Q1
- new net N$60: U1.Q0
- new net N$61: U1.I1
- new net N$62: U1.I0
- new net V18: C74.1, C76.1, C77.1, C78.1, IC1.VDDINT, TP21.1, VR1.OUT
- net 3.3VD: now also C71.1, C72.1, C73.1, C75.1, IC1.VDDAUX, IC1.VDDIO1, IC1.VDDIO2, JP1.1, VR1.EN, VR1.IN
- net GND: now also C71.2, C72.2, C73.2, C74.2, C75.2, C76.2, C78.2, IC1.GND@0, IC1.GND@1, IC1.GND@2, JP1.2, VR1.GND
Other:
- note added: "2.85V For SkyTraq supply"
- note added: "Splitter"
- note added: "SuperCap"
- note added: "TODO: WHAT DO WE DO WITH CLKOUT?"
- note added: "clock cleanup"
- moved on the sheet: C2, C21, C25, C26, C33, C38, C39, C40, C41, C42, C43, C54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

Commit message: using the GPS Carrier from AV4, expanded the size of the board to fit in the AV4 C channel and give more room. Moved everything onto that larger board, with preliminary placement. About to rip up and flip  STM because of OCD (just can't stand it), so checking in before I do something as stupid as that.
Parts:
- added C79: 1u, rcl_custom:C-EU0402-C-NOSILK
- added C80: 100p, rcl_custom:C-EU0402-C-NOSILK
Connections:
- removed net BAR_GND: C24.1, C66.-, R22.1, U10.GND
- net 2.85V-S: now also C79.1, C80.1
- net AGND: now also C56.2, J2.GND, L5.1, L6.GND@1, L6.GND@2, L6.GND@3, U10.GND, U5.VSS
- net GND: now also C24.1, C66.-, C79.2, C80.2, R22.1; no longer C56.2, J2.GND, L5.1, L6.GND@1, L6.GND@2, L6.GND@3, U5.VSS
- net MAX-RF: now also U10.PORT2; no longer U10.PORT1
- net STQ-RF: now also U10.PORT1; no longer U10.PORT2
Other:
- note added: "THIS SHOULD BE AGND?!?!"
- moved on the sheet: C22, J2

Commit message: New LNA+SAW filter, plus starting to lay stuff out.
Parts:
- removed L6: SF14-1575F5UU19, saw_1.4x1.1:SAW_1.4X1.1
- removed LED3: RGB, Tova:LED_RGB_PLCC-6
- removed U5: XC2401A8167R-G, xc2401:XC2401
- added C81: 47p, rcl_custom:C-EU0402-C-NOSILK
- added LED8: (no value), led-rgb-rohm:LED_RGB_COMMON_ANODE-1.6X1.26
- added R25: 4.7k, rcl_custom:R-US_0402-C-NOSILK
- added U12: AVAGO-ALM-GPXX, ic-lna-ALM-GPxx-Avago:AVAGO-ALM-GPXX
- C1: value 100p -> 330p
- C56: value 10n -> 100n
- L2: value 6.2nH -> 22n; device rcl_custom:L-US0402-C-NOSILK -> rcl_custom:L-US0402-B-NOSILK
- L5: value 9.1nH -> 1.8n; device rcl_custom:L-US0402-C-NOSILK -> rcl_custom:L-US0402-B-NOSILK
- R13: value 470 -> 10
Connections:
- removed net EXT-LNA-IN: L2.2, U5.RFIN
- removed net SMA-FILTERED: L2.1, L5.2, L6.OUT
- removed net SMA-RAW: J2.SIG, L6.IN
- new net N$63: IC1.IO_14
- new net N$64: IC1.IO_13, U1.CLKOUT
- new net N$65: R25.2, U12.SD
- new net N$66: L5.2, U12.VDD
- new net STM_SPI1_MISO: IC1.IO_0, U2.PA6
- new net STM_SPI1_MOSI: IC1.IO_2, U2.PB5
- new net STM_SPI1_NSS: IC1.IO_3, U2.PA4
- new net STM_SPI1_SCK: IC1.IO_1, U2.PA5
- net 2.85VA: now also C1.1, L2.2, R25.1
- net 3.3VD: now also LED8.COMMON_ANODE; no longer R38.1, R39.1, R40.1
- net AGND: now also C1.2, C81.2; no longer L5.1, L6.GND@1, L6.GND@2, L6.GND@3, U5.VSS
- net LED2: now also R39.2; no longer LED3G.K
- net LNA-POWER-FILTERED: now also C81.1, L2.1, L5.1; no longer U5.VDD
- net N$11: now also R40.2; no longer LED3R.K
- net N$12: now also LED8.GK, R38.1; no longer LED3B.A, R39.2
- net N$14: now also U12.RF-OUT; no longer C1.1
- net N$18: now also LED8.BK, R39.1; no longer LED3G.A, R38.2
- net N$34: now also R38.2; no longer LED3B.K
- net N$37: now also LED8.RK, R40.1; no longer LED3R.A, R40.2
- net N$5: now also J2.SIG, U12.RF-IN; no longer C1.2, U5.RFOUT
- net N$59: now also IC1.IO_12
- net N$60: now also IC1.IO_11
- net N$61: now also IC1.IO_9
- net N$62: now also IC1.IO_8
Other:
- note removed: "+15 dB LNA"
- note removed: "1.5 GHz SAW Filter"
- note removed: "As per datasheet, for 2.85V supply"
- moved on the sheet: C1, C56, R13, R38, R39, R40, U10

Commit message: Digital portion of v3 basically laid out, RF sections laid out. To do: verify CPLD power supply, think more about ground/power separation for RF section.
Parts:
- removed LED8: (no value), led-rgb-rohm:LED_RGB_COMMON_ANODE-1.6X1.26
- removed TP3, TP6, TP7: TEST-POINT, Tova:TEST-POINT
- added LED3: (no value), apdm:LED-RGB-SEPARATE-3528
- TP16: value TEST-POINT -> (none); device Tova:TEST-POINT -> apdm:PAD+X-0.7
Connections:
- removed net N$54: TP7.1, U2.PE5
- removed net N$55: TP6.1, U2.PE4
- removed net N$56: TP3.1, U2.PE3
- removed net STM_SPI1_MISO: IC1.IO_0, U2.PA6
- net 3.3VD: now also LED3B.A, LED3G.A, LED3R.A; no longer LED8.COMMON_ANODE
- net N$12: now also LED3R.K; no longer LED8.GK
- net N$18: now also LED3G.K; no longer LED8.BK
- net N$2: now also TP16.P; no longer TP16.1
- net N$37: now also LED3B.K; no longer LED8.RK
Other:
- note added: "Don't need MISO!"
- moved on the sheet: L3
Changed lines of the file:
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@@
 <setting verticaltext="up"/>
 </settings>
-<grid distance="0.05" unitdist="inch" unit="inch" style="lines" multiple="2" display="yes" altdistance="0.01" altunitdist="inch" altunit="inch"/>
+<grid distance="0.05" unitdist="inch" unit="inch" style="lines" multiple="2" display="no" altdistance="0.01" altunitdist="inch" altunit="inch"/>
 <layers>
 <layer number="1" name="Top" color="4" fill="1" visible="no" active="no"/>
@@
 <part name="R20" library="rcl_custom" deviceset="R-US_" device="0402-C-NOSILK" value="1k"/>
 <part name="3.3VD1" library="SparkFun-Aesthetics" deviceset="3.3VD" device=""/>
-<part name="TP3" library="Tova" deviceset="TEST-POINT" device=""/>
-<part name="TP6" library="Tova" deviceset="TEST-POINT" device=""/>
-<part name="TP7" library="Tova" deviceset="TEST-POINT" device=""/>
 <part name="L8" library="saw_1.4x1.1" deviceset="SAW_1.4X1.1" device="" value="SF14-1575F5UU19"/>
 <part name="J2" library="emerson-sma-endfire" deviceset="CON_SMA-ENDFIRE_EMERSON_EMERSON-142-0701-801" device=""/>
@@
 <part name="TP14" library="Tova" deviceset="TEST-POINT" device=""/>
 <part name="TP15" library="Tova" deviceset="TEST-POINT" device=""/>
-<part name="TP16" library="Tova" deviceset="TEST-POINT" device=""/>
 <part name="GND23" library="SparkFun-Aesthetics" deviceset="GND" device=""/>
 <part name="TP17" library="Tova" deviceset="TEST-POINT" device=""/>
@@
 <part name="L5" library="rcl_custom" deviceset="L-US" device="0402-B-NOSILK" value="1.8n"/>
 <part name="C81" library="rcl_custom" deviceset="C-EU" device="0402-C-NOSILK" value="47p"/>
-<part name="LED8" library="led-rgb-rohm" deviceset="LED_RGB_COMMON_ANODE-*" device="1.6X1.26"/>
+<part name="TP16" library="apdm" deviceset="PAD+X" device="-0.7"/>
+<part name="LED3" library="apdm" deviceset="LED-RGB-SEPARATE-*" device="3528"/>
 </parts>
 <sheets>
@@
 </segment>
 </net>
-<net name="STM_SPI1_MISO" class="0">
-<segment>
-<wire x1="261.62" y1="147.32" x2="231.14" y2="147.32" width="0.1524" layer="91"/>
-<label x="231.14" y="147.32" size="1.27" layer="95" rot="MR0" xref="yes"/>
-<pinref part="IC1" gate="G$1" pin="IO_0"/>
-</segment>
-</net>
 <net name="STM_SPI1_SCK" class="0">
 <segment>
@@
 <text x="269.24" y="59.69" size="1.27" layer="95" rot="R90">FROM MAX2769</text>
 <text x="335.28" y="86.36" size="1.27" layer="95" rot="R90">TO MAX2769</text>
+<text x="245.11" y="58.42" size="1.27" layer="97">Don't need MISO!</text>
 </plain>
 <instances>
@@
 </instance>
 <instance part="3.3VD1" gate="3.3VD" x="322.58" y="170.18"/>
-<instance part="TP3" gate="G$1" x="149.86" y="96.52" smashed="yes">
-<attribute name="NAME" x="143.51" y="96.52" size="1.778" layer="95" font="vector"/>
-</instance>
-<instance part="TP6" gate="G$1" x="149.86" y="93.98" smashed="yes">
-<attribute name="NAME" x="143.51" y="93.98" size="1.778" layer="95" font="vector"/>
-</instance>
-<instance part="TP7" gate="G$1" x="149.86" y="91.44" smashed="yes">
-<attribute name="NAME" x="143.51" y="91.44" size="1.778" layer="95" font="vector"/>
-</instance>
 <instance part="X1" gate="C$1" x="254" y="189.23" smashed="yes" rot="R270">
 <attribute name="NAME" x="250.19" y="194.31" size="1.778" layer="95"/>
 <attribute name="VALUE" x="248.92" y="181.61" size="1.778" layer="96"/>
 </instance>
-<instance part="LED8" gate="LED" x="292.1" y="114.3" rot="R270"/>
+<instance part="LED3" gate="R" x="292.1" y="114.3" rot="R270"/>
+<instance part="LED3" gate="G" x="292.1" y="109.22" rot="R270"/>
+<instance part="LED3" gate="B" x="292.1" y="119.38" rot="R270"/>
 </instances>
 <busses>
@@
 </segment>
 <segment>
-<pinref part="LED8" gate="LED" pin="COMMON_ANODE"/>
 <pinref part="3.3VD3" gate="3.3VD" pin="3.3VD"/>
-<wire x1="294.64" y1="114.3" x2="299.72" y2="114.3" width="0.1524" layer="91"/>
 <wire x1="299.72" y1="114.3" x2="299.72" y2="119.38" width="0.1524" layer="91"/>
+<pinref part="LED3" gate="B" pin="A"/>
+<pinref part="LED3" gate="R" pin="A"/>
+<wire x1="294.64" y1="119.38" x2="294.64" y2="114.3" width="0.1524" layer="91"/>
+<pinref part="LED3" gate="G" pin="A"/>
+<wire x1="294.64" y1="114.3" x2="294.64" y2="109.22" width="0.1524" layer="91"/>
+<junction x="294.64" y="114.3"/>
+<wire x1="294.64" y1="114.3" x2="299.72" y2="114.3" width="0.1524" layer="91"/>
 </segment>
 </net>
@@
 </segment>
 </net>
-<net name="N$54" class="0">
-<segment>
-<pinref part="U2" gate="U" pin="PE5"/>
-<pinref part="TP7" gate="G$1" pin="1"/>
-<wire x1="160.02" y1="91.44" x2="149.86" y2="91.44" width="0.1524" layer="91"/>
-</segment>
-</net>
-<net name="N$55" class="0">
-<segment>
-<pinref part="TP6" gate="G$1" pin="1"/>
-<pinref part="U2" gate="U" pin="PE4"/>
-<wire x1="149.86" y1="93.98" x2="160.02" y2="93.98" width="0.1524" layer="91"/>
-</segment>
-</net>
-<net name="N$56" class="0">
-<segment>
-<pinref part="U2" gate="U" pin="PE3"/>
-<pinref part="TP3" gate="G$1" pin="1"/>
-<wire x1="160.02" y1="96.52" x2="149.86" y2="96.52" width="0.1524" layer="91"/>
-</segment>
-</net>
 <net name="DEBUG-PHY-MODWIRE" class="0">
 <segment>
@@
 </segment>
 </net>
-<net name="STM_SPI1_MISO" class="0">
-<segment>
-<pinref part="U2" gate="U" pin="PA6"/>
-<wire x1="243.84" y1="58.42" x2="274.32" y2="58.42" width="0.1524" layer="91"/>
-<label x="274.32" y="58.42" size="1.27" layer="95" xref="yes"/>
-</segment>
-</net>
 <net name="STM_SPI1_SCK" class="0">
 <segment>
@@
 </segment>
 </net>
-<net name="N$12" class="0">
-<segment>
-<pinref part="R38" gate="R" pin="1"/>
-<pinref part="LED8" gate="LED" pin="GK"/>
-<wire x1="287.02" y1="114.3" x2="284.48" y2="114.3" width="0.1524" layer="91"/>
-</segment>
-</net>
 <net name="N$18" class="0">
 <segment>
 <pinref part="R39" gate="R" pin="1"/>
-<pinref part="LED8" gate="LED" pin="BK"/>
 <wire x1="287.02" y1="109.22" x2="284.48" y2="109.22" width="0.1524" layer="91"/>
-</segment>
-</net>
-<net name="N$37" class="0">
-<segment>
-<pinref part="R40" gate="R" pin="1"/>
-<pinref part="LED8" gate="LED" pin="RK"/>
-<wire x1="287.02" y1="119.38" x2="284.48" y2="119.38" width="0.1524" layer="91"/>
+<pinref part="LED3" gate="G" pin="K"/>
 </segment>
 </net>
@@
 </segment>
 </net>
+<net name="N$12" class="0">
+<segment>
+<pinref part="R38" gate="R" pin="1"/>
+<pinref part="LED3" gate="R" pin="K"/>
+<wire x1="284.48" y1="114.3" x2="287.02" y2="114.3" width="0.1524" layer="91"/>
+</segment>
+</net>
+<net name="N$37" class="0">
+<segment>
+<pinref part="R40" gate="R" pin="1"/>
+<pinref part="LED3" gate="B" pin="K"/>
+<wire x1="284.48" y1="119.38" x2="287.02" y2="119.38" width="0.1524" layer="91"/>
+</segment>
+</net>
 </nets>
 </sheet>
@@
 <attribute name="VALUE" x="136.525" y="106.68" size="1.778" layer="96" rot="R180"/>
 </instance>
-<instance part="L3" gate="L" x="200.66" y="200.66" smashed="yes" rot="R90">
-<attribute name="NAME" x="198.755" y="205.105" size="1.778" layer="95"/>
-<attribute name="VALUE" x="193.04" y="203.2" size="1.27" layer="96"/>
+<instance part="L3" gate="L" x="203.2" y="200.66" smashed="yes">
+<attribute name="NAME" x="207.645" y="202.565" size="1.778" layer="95" rot="R270"/>
+<attribute name="VALUE" x="205.74" y="208.28" size="1.27" layer="96" rot="R270"/>
 </instance>
 <instance part="C28" gate="CE" x="218.44" y="190.5" smashed="yes" rot="MR180">
@@
 <attribute name="VALUE" x="176.784" y="159.131" size="1.778" layer="96"/>
 </instance>
-<instance part="TP16" gate="G$1" x="223.52" y="139.7" smashed="yes" rot="R180">
-<attribute name="NAME" x="226.06" y="138.43" size="1.778" layer="95" font="vector"/>
-</instance>
+<instance part="TP16" gate="TP" x="226.06" y="139.7"/>
 </instances>
 <busses>
@@
 <junction x="218.44" y="200.66"/>
 <pinref part="L3" gate="L" pin="2"/>
-<wire x1="200.66" y1="205.74" x2="213.36" y2="200.66" width="0.1524" layer="91"/>
+<wire x1="208.28" y1="200.66" x2="213.36" y2="200.66" width="0.1524" layer="91"/>
 <wire x1="213.36" y1="200.66" x2="218.44" y2="200.66" width="0.1524" layer="91"/>
 <junction x="213.36" y="200.66"/>
@@
 <wire x1="205.74" y1="167.64" x2="205.74" y2="180.34" width="0.1524" layer="91"/>
 <wire x1="205.74" y1="180.34" x2="208.28" y2="180.34" width="0.1524" layer="91"/>
-<wire x1="208.28" y1="180.34" x2="200.66" y2="205.74" width="0.1524" layer="91"/>
-<junction x="200.66" y="205.74"/>
+<wire x1="208.28" y1="180.34" x2="208.28" y2="200.66" width="0.1524" layer="91"/>
+<junction x="208.28" y="200.66"/>
 </segment>
 <segment>
@@
 <pinref part="L3" gate="L" pin="1"/>
 <pinref part="C32" gate="CE" pin="2"/>
-<wire x1="200.66" y1="193.04" x2="187.96" y2="200.66" width="0.1524" layer="91"/>
+<wire x1="195.58" y1="200.66" x2="187.96" y2="200.66" width="0.1524" layer="91"/>
 <wire x1="187.96" y1="200.66" x2="187.96" y2="195.58" width="0.1524" layer="91"/>
 <pinref part="C34" gate="CE" pin="2"/>
@@
 <wire x1="182.88" y1="200.66" x2="182.88" y2="195.58" width="0.1524" layer="91"/>
 <junction x="187.96" y="200.66"/>
-<wire x1="200.66" y1="193.04" x2="193.04" y2="180.34" width="0.1524" layer="91"/>
-<junction x="200.66" y="193.04"/>
+<wire x1="195.58" y1="200.66" x2="195.58" y2="180.34" width="0.1524" layer="91"/>
+<junction x="195.58" y="200.66"/>
 <pinref part="U3" gate="G$1" pin="VDDA_3.3"/>
-<wire x1="193.04" y1="180.34" x2="200.66" y2="180.34" width="0.1524" layer="91"/>
+<wire x1="195.58" y1="180.34" x2="200.66" y2="180.34" width="0.1524" layer="91"/>
 <wire x1="200.66" y1="180.34" x2="200.66" y2="167.64" width="0.1524" layer="91"/>
 <label x="187.96" y="177.8" size="1.778" layer="95"/>
@@
 <segment>
 <pinref part="U3" gate="G$1" pin="RXER"/>
-<pinref part="TP16" gate="G$1" pin="1"/>
 <wire x1="223.52" y1="139.7" x2="220.98" y2="139.7" width="0.1524" layer="91"/>
+<pinref part="TP16" gate="TP" pin="P"/>
 </segment>
 </net>
