File: v3-gps.sch (EAGLE design)
At the start: 180 parts, among them IC1 XC2C32A_VQ44_2, J1 1.27MM-SWD-CONNECTOR, J2 CON_SMA-ENDFIRE_EMERSON_EMERS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, J3 ROCKETNET-CONNECTOR-16M, J4 ZX62D-B-5P8, J7 CON_HIROSE_DM3D(MICROSD), Q1 NTR4101P, T1 ALT4532, T2 ALT4532, U1 MAX2769, U10 BP2G+, U11 MAX8510EXK29+T, U12 AVAGO-ALM-GPXX, U2 STM32F4V_100PIN_GPSBOARD, U3 KSZ8081, U4 7Q-16.368MBG-T, U6 MAX8510EXK29+T, U7 MAX8510EXK29+T, U8 LMZ12001, U9 VENUS638FLPX-L, X1 25 MHz

Commit message: Added link to the MAX2769 google doc, as well as renamed things to be BOM, and committed some minor changes in the layout and notes in the schematic.
Other:
- note added: "1.85V internal supply For CPLD"
- note added: "2.85V-S is the skytraq specific power supply. Meant to decouple from other analog and main digital supplies"
- note added: "DC BLOCKING CAP?"
- moved on the sheet: C24, C66, D1, R24
Changed lines of the file:
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@@
 <setting verticaltext="up"/>
 </settings>
-<grid distance="0.05" unitdist="inch" unit="inch" style="lines" multiple="2" display="no" altdistance="0.01" altunitdist="inch" altunit="inch"/>
+<grid distance="0.1" unitdist="inch" unit="inch" style="lines" multiple="1" display="no" altdistance="0.01" altunitdist="inch" altunit="inch"/>
 <layers>
 <layer number="1" name="Top" color="4" fill="1" visible="no" active="no"/>
@@
 <plain>
 <text x="55.88" y="217.17" size="1.778" layer="97">4.5 - 26 Vin</text>
-<text x="246.38" y="149.86" size="1.778" layer="97">2.85V Analog and Digital to MAX2769 GPS Receiver</text>
+<text x="248.92" y="210.82" size="1.778" layer="97">2.85V Analog and Digital to MAX2769 GPS Receiver</text>
 <text x="86.36" y="218.44" size="1.778" layer="97">Aux supply from USB debug</text>
-<text x="261.62" y="88.9" size="1.778" layer="97">2.85V For SkyTraq supply</text>
+<text x="264.16" y="134.62" size="1.778" layer="97">2.85V For SkyTraq supply</text>
 <text x="314.96" y="157.48" size="1.778" layer="94">THIS SHOULD BE AGND?!?!</text>
 <text x="313.69" y="111.76" size="1.778" layer="94">THIS SHOULD BE AGND?!?!</text>
+<text x="256.54" y="88.9" size="1.778" layer="97">1.85V internal supply For CPLD</text>
 </plain>
 <instances>
@@
 <text x="238.76" y="181.61" size="2.54" layer="97">WHERE SHOULD WE CONNECT GND/AGND</text>
 <text x="137.16" y="121.92" size="1.27" layer="97">1.2V LDO out</text>
-<text x="81.28" y="123.19" size="1.27" layer="97" rot="R90">DOUBLE CHECK THIS PACKAGE</text>
-<text x="91.44" y="134.62" size="1.778" layer="97">SuperCap</text>
+<text x="66.04" y="123.19" size="1.27" layer="97" rot="R90">DOUBLE CHECK THIS PACKAGE</text>
+<text x="76.2" y="134.62" size="1.778" layer="97">SuperCap</text>
+<text x="124.46" y="223.52" size="1.778" layer="97">2.85V-S is the skytraq specific power
+supply. Meant to decouple from other
+analog and main digital supplies</text>
+<text x="238.76" y="177.8" size="2.54" layer="97">DC BLOCKING CAP?</text>
 </plain>
 <instances>
@@
 <instance part="C19" gate="CE" x="124.46" y="187.96"/>
 <instance part="C22" gate="CE" x="132.08" y="187.96"/>
-<instance part="C24" gate="CE" x="111.76" y="167.64" rot="R180"/>
+<instance part="C24" gate="CE" x="111.76" y="170.18" rot="R180"/>
 <instance part="R21" gate="R" x="111.76" y="182.88" rot="MR90"/>
 <instance part="R22" gate="R" x="149.86" y="152.4" rot="MR90"/>
@@
 <attribute name="NAME" x="148.59" y="127" size="1.778" layer="95" font="vector"/>
 </instance>
-<instance part="D1" gate="G$1" x="86.36" y="157.48" smashed="yes" rot="R90">
-<attribute name="NAME" x="84.074" y="157.48" size="1.016" layer="95" rot="R90"/>
-<attribute name="VALUE" x="89.662" y="157.48" size="1.016" layer="96" rot="R90"/>
-</instance>
-<instance part="R24" gate="R" x="86.36" y="149.86" rot="MR90"/>
-<instance part="C66" gate="G$1" x="86.36" y="137.16"/>
+<instance part="D1" gate="G$1" x="71.12" y="157.48" smashed="yes" rot="R90">
+<attribute name="NAME" x="68.834" y="157.48" size="1.016" layer="95" rot="R90"/>
+<attribute name="VALUE" x="74.422" y="157.48" size="1.016" layer="96" rot="R90"/>
+</instance>
+<instance part="R24" gate="R" x="71.12" y="149.86" rot="MR90"/>
+<instance part="C66" gate="G$1" x="71.12" y="137.16"/>
 <instance part="SUPPLY2" gate="G$1" x="124.46" y="195.58"/>
 <instance part="SUPPLY3" gate="G$1" x="111.76" y="190.5"/>
-<instance part="SUPPLY4" gate="G$1" x="86.36" y="162.56"/>
+<instance part="SUPPLY4" gate="G$1" x="71.12" y="162.56"/>
 <instance part="SUPPLY5" gate="G$1" x="128.27" y="149.86"/>
-<instance part="GND44" gate="G1" x="86.36" y="129.54"/>
+<instance part="GND44" gate="G1" x="71.12" y="129.54"/>
 <instance part="GND24" gate="G1" x="154.94" y="99.06"/>
 <instance part="GND45" gate="G1" x="124.46" y="180.34"/>
 <instance part="GND46" gate="G1" x="132.08" y="180.34" rot="MR0"/>
 <instance part="GND47" gate="G1" x="149.86" y="144.78" rot="MR0"/>
-<instance part="GND48" gate="G1" x="111.76" y="162.56"/>
+<instance part="GND48" gate="G1" x="111.76" y="167.64"/>
 <instance part="C79" gate="CE" x="142.24" y="205.74"/>
 <instance part="C80" gate="CE" x="149.86" y="205.74"/>
@@
 <segment>
 <pinref part="C66" gate="G$1" pin="-"/>
-<wire x1="86.36" y1="132.08" x2="86.36" y2="129.54" width="0.1524" layer="91"/>
+<wire x1="71.12" y1="132.08" x2="71.12" y2="129.54" width="0.1524" layer="91"/>
 <pinref part="GND44" gate="G1" pin="GND"/>
 </segment>
@@
 <pinref part="C24" gate="CE" pin="1"/>
 <pinref part="GND48" gate="G1" pin="GND"/>
-<wire x1="111.76" y1="162.56" x2="111.76" y2="165.1" width="0.1524" layer="91"/>
 </segment>
 <segment>
@@
 <net name="STM_USART6_TX" class="0">
 <segment>
-<label x="143.51" y="162.56" size="1.27" layer="95" rot="MR0" xref="yes"/>
+<label x="100.33" y="162.56" size="1.27" layer="95" rot="MR0" xref="yes"/>
 <pinref part="U9" gate="G$1" pin="RXD0"/>
-<wire x1="143.51" y1="162.56" x2="154.94" y2="162.56" width="0.1524" layer="91"/>
+<wire x1="100.33" y1="162.56" x2="154.94" y2="162.56" width="0.1524" layer="91"/>
 <pinref part="TP25" gate="G$1" pin="1"/>
 <wire x1="154.94" y1="162.56" x2="160.02" y2="162.56" width="0.1524" layer="91"/>
@@
 <net name="STM_USART6_RX" class="0">
 <segment>
-<label x="143.51" y="160.02" size="1.27" layer="95" rot="MR0" xref="yes"/>
+<label x="100.33" y="160.02" size="1.27" layer="95" rot="MR0" xref="yes"/>
 <pinref part="U9" gate="G$1" pin="TXD0"/>
 <wire x1="160.02" y1="160.02" x2="154.94" y2="160.02" width="0.1524" layer="91"/>
 <pinref part="TP27" gate="G$1" pin="1"/>
-<wire x1="154.94" y1="160.02" x2="143.51" y2="160.02" width="0.1524" layer="91"/>
+<wire x1="154.94" y1="160.02" x2="100.33" y2="160.02" width="0.1524" layer="91"/>
 <junction x="154.94" y="160.02"/>
 </segment>
@@
 <wire x1="111.76" y1="175.26" x2="111.76" y2="177.8" width="0.1524" layer="91"/>
 <pinref part="C24" gate="CE" pin="2"/>
-<wire x1="111.76" y1="172.72" x2="111.76" y2="175.26" width="0.1524" layer="91"/>
 <junction x="111.76" y="175.26"/>
-<wire x1="111.76" y1="175.26" x2="93.98" y2="175.26" width="0.1524" layer="91"/>
-<label x="93.98" y="175.26" size="1.27" layer="95" rot="R180" xref="yes"/>
+<wire x1="111.76" y1="175.26" x2="101.6" y2="175.26" width="0.1524" layer="91"/>
+<label x="101.6" y="175.26" size="1.27" layer="95" rot="R180" xref="yes"/>
 <pinref part="TP28" gate="G$1" pin="1"/>
 <junction x="119.38" y="175.26"/>
@@
 <pinref part="U9" gate="G$1" pin="PPS"/>
 <wire x1="160.02" y1="127" x2="154.94" y2="127" width="0.1524" layer="91"/>
-<label x="144.78" y="127" size="1.27" layer="95" rot="R180" xref="yes"/>
+<label x="101.6" y="127" size="1.27" layer="95" rot="R180" xref="yes"/>
 <pinref part="TP30" gate="G$1" pin="1"/>
-<wire x1="154.94" y1="127" x2="144.78" y2="127" width="0.1524" layer="91"/>
+<wire x1="154.94" y1="127" x2="101.6" y2="127" width="0.1524" layer="91"/>
 <junction x="154.94" y="127"/>
 </segment>
@@
 <wire x1="160.02" y1="170.18" x2="119.38" y2="170.18" width="0.1524" layer="91"/>
 <wire x1="119.38" y1="170.18" x2="119.38" y2="142.24" width="0.1524" layer="91"/>
-<wire x1="119.38" y1="142.24" x2="86.36" y2="142.24" width="0.1524" layer="91"/>
+<wire x1="119.38" y1="142.24" x2="71.12" y2="142.24" width="0.1524" layer="91"/>
 <pinref part="R24" gate="R" pin="1"/>
-<wire x1="86.36" y1="144.78" x2="86.36" y2="142.24" width="0.1524" layer="91"/>
+<wire x1="71.12" y1="144.78" x2="71.12" y2="142.24" width="0.1524" layer="91"/>
 <pinref part="C66" gate="G$1" pin="+"/>
-<wire x1="86.36" y1="139.7" x2="86.36" y2="142.24" width="0.1524" layer="91"/>
-<junction x="86.36" y="142.24"/>
-</segment>
-</net>
+<wire x1="71.12" y1="139.7" x2="71.12" y2="142.24" width="0.1524" layer="91"/>
+<junction x="71.12" y="142.24"/>
+</segment>
+</net>

Commit message: 90% done! All analog routed, only 9 airwires left to the CPLD which is trivial (but should be rerouted for easy of routing and also for maybe power domains? In any case, it just needs: stiching, double checking, reduce size of board, tnames, and other pre-production checkouts.
Parts:
- added C82: 100n, rcl_custom:C-EU0402-C-NOSILK
- added SH1: BMI-S-202-SHIELD, hw-laird-bmi-s-202:BMI-S-202-SHIELD
Connections:
- net N$59 renamed Q1
- net N$60 renamed Q0
- net N$61 renamed I1
- net N$62 renamed I0
- net TCXO-OUT renamed N$54
- removed net N$63: IC1.IO_14
- net AGND: now also SH1.P$1
- net GND: now also C82.1
- net MAX-RF: now also U10.PORT1; no longer U10.PORT2
- net STQ-RF: now also U10.PORT2; no longer U10.PORT1
- net STQ-VBAT: now also C82.2
Other:
- note added: "ASSUME WE CAN USE CLKOUT AND NOT TCXO OUT?"
- note added: "Test point only"
Changed lines of the file:
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@@
 <class number="1" name="PWR" width="0" drill="0">
 </class>
-<class number="2" name="rf" width="0" drill="0">
-<clearance class="2" value="0.3302"/>
+<class number="2" name="RF" width="0" drill="0">
+<clearance class="2" value="0.635"/>
 </class>
 </classes>
@@
 <part name="TP16" library="apdm" deviceset="PAD+X" device="-0.7"/>
 <part name="LED3" library="apdm" deviceset="LED-RGB-SEPARATE-*" device="3528"/>
+<part name="C82" library="rcl_custom" deviceset="C-EU" device="0402-C-NOSILK" value="100n"/>
+<part name="GND51" library="supply" deviceset="GND" device=""/>
+<part name="SH1" library="hw-laird-bmi-s-202" deviceset="BMI-S-202-SHIELD" device=""/>
+<part name="AGND20" library="supply1" deviceset="AGND" device=""/>
 </parts>
 <sheets>
@@
 <attribute name="VALUE" x="124.46" y="127" size="1.778" layer="96"/>
 </instance>
+<instance part="SH1" gate="G$1" x="149.86" y="63.5"/>
+<instance part="AGND20" gate="VR1" x="149.86" y="55.88"/>
 </instances>
 <busses>
@@
 </segment>
 </net>
-<net name="STQ-RF" class="0">
-<segment>
-<wire x1="215.9" y1="104.14" x2="234.95" y2="104.14" width="0.1524" layer="91"/>
+<net name="STQ-RF" class="2">
+<segment>
+<wire x1="208.28" y1="104.14" x2="234.95" y2="104.14" width="0.1524" layer="91"/>
 <label x="234.95" y="104.14" size="1.778" layer="95" xref="yes"/>
-<wire x1="215.9" y1="104.14" x2="210.82" y2="109.22" width="0.1524" layer="91"/>
+<pinref part="U10" gate="G$1" pin="PORT2"/>
+</segment>
+</net>
+<net name="MAX-RF" class="2">
+<segment>
+<wire x1="208.28" y1="109.22" x2="234.95" y2="109.22" width="0.1524" layer="91"/>
+<label x="234.95" y="109.22" size="1.778" layer="95" xref="yes"/>
 <pinref part="U10" gate="G$1" pin="PORT1"/>
-<wire x1="210.82" y1="109.22" x2="208.28" y2="109.22" width="0.1524" layer="91"/>
-</segment>
-</net>
-<net name="MAX-RF" class="0">
-<segment>
-<wire x1="215.9" y1="109.22" x2="234.95" y2="109.22" width="0.1524" layer="91"/>
-<label x="234.95" y="109.22" size="1.778" layer="95" xref="yes"/>
-<wire x1="215.9" y1="109.22" x2="210.82" y2="104.14" width="0.1524" layer="91"/>
-<pinref part="U10" gate="G$1" pin="PORT2"/>
-<wire x1="210.82" y1="104.14" x2="208.28" y2="104.14" width="0.1524" layer="91"/>
-</segment>
-</net>
-<net name="N$14" class="0">
+</segment>
+</net>
+<net name="N$14" class="2">
 <segment>
 <pinref part="U10" gate="G$1" pin="SUM"/>
@@
 <wire x1="170.18" y1="121.92" x2="170.18" y2="120.65" width="0.1524" layer="91"/>
 </segment>
-</net>
-<net name="N$5" class="0">
+<segment>
+<pinref part="SH1" gate="G$1" pin="P$1"/>
+<pinref part="AGND20" gate="VR1" pin="AGND"/>
+</segment>
+</net>
+<net name="N$5" class="2">
 <segment>
 <pinref part="J2" gate="G$1" pin="SIG"/>
@@
 <wire x1="236.22" y1="165.1" x2="149.86" y2="165.1" width="0.1524" layer="97" style="shortdash"/>
 <text x="58.42" y="127" size="1.27" layer="95" rot="R90">MAX2769 SPI CONFIG PORT</text>
-<wire x1="215.9" y1="104.14" x2="215.9" y2="93.98" width="0.1524" layer="97"/>
-<wire x1="215.9" y1="93.98" x2="231.14" y2="93.98" width="0.1524" layer="97"/>
-<wire x1="231.14" y1="93.98" x2="231.14" y2="104.14" width="0.1524" layer="97"/>
-<wire x1="231.14" y1="104.14" x2="215.9" y2="104.14" width="0.1524" layer="97"/>
-<text x="215.9" y="97.79" size="1.778" layer="97">clock cleanup</text>
-<text x="173.99" y="114.3" size="1.778" layer="97">TODO: WHAT DO WE DO WITH CLKOUT?</text>
+<wire x1="220.98" y1="114.3" x2="220.98" y2="104.14" width="0.1524" layer="97"/>
+<wire x1="220.98" y1="104.14" x2="236.22" y2="104.14" width="0.1524" layer="97"/>
+<wire x1="236.22" y1="104.14" x2="236.22" y2="114.3" width="0.1524" layer="97"/>
+<wire x1="236.22" y1="114.3" x2="220.98" y2="114.3" width="0.1524" layer="97"/>
+<text x="220.98" y="107.95" size="1.778" layer="97">clock cleanup</text>
+<text x="201.93" y="101.6" size="1.778" layer="97">TODO: WHAT DO WE DO WITH CLKOUT?</text>
+<text x="191.77" y="99.06" size="1.778" layer="97">ASSUME WE CAN USE CLKOUT AND NOT TCXO OUT?</text>
 </plain>
 <instances>
@@
 </segment>
 </net>
-<net name="TCXO-OUT" class="0">
-<segment>
-<pinref part="C2" gate="CE" pin="1"/>
-<pinref part="U4" gate="U$1" pin="OUT"/>
-<wire x1="78.74" y1="106.68" x2="73.66" y2="106.68" width="0.15" layer="91"/>
-<wire x1="73.66" y1="106.68" x2="64.77" y2="106.68" width="0.15" layer="91"/>
-<wire x1="73.66" y1="106.68" x2="73.66" y2="30.48" width="0.1524" layer="91"/>
-<junction x="73.66" y="106.68"/>
-<wire x1="73.66" y1="30.48" x2="200.66" y2="30.48" width="0.1524" layer="91"/>
-<wire x1="200.66" y1="30.48" x2="200.66" y2="99.06" width="0.1524" layer="91"/>
-<wire x1="200.66" y1="99.06" x2="215.9" y2="99.06" width="0.1524" layer="91"/>
-</segment>
-</net>
 <net name="ANTFLAG" class="0">
 <segment>
@@
 </segment>
 </net>
-<net name="MAX-RF" class="0">
+<net name="MAX-RF" class="2">
 <segment>
 <wire x1="116.84" y1="88.9" x2="93.98" y2="88.9" width="0.1524" layer="91"/>
@@
 </segment>
 </net>
-<net name="N$59" class="0">
+<net name="Q1" class="0">
 <segment>
 <pinref part="U1" gate="G$1" pin="Q1"/>
@@
 </segment>
 </net>
-<net name="N$60" class="0">
+<net name="Q0" class="0">
 <segment>
 <pinref part="U1" gate="G$1" pin="Q0"/>
@@
 </segment>
 </net>
-<net name="N$61" class="0">
+<net name="I1" class="0">
 <segment>
 <pinref part="U1" gate="G$1" pin="I1"/>
@@
 </segment>
 </net>
-<net name="N$62" class="0">
+<net name="I0" class="0">
 <segment>
 <pinref part="U1" gate="G$1" pin="I0"/>
@@
 </segment>
 </net>
-<net name="N$63" class="0">
-<segment>
-<wire x1="231.14" y1="99.06" x2="248.92" y2="99.06" width="0.1524" layer="91"/>
-<wire x1="248.92" y1="99.06" x2="248.92" y2="109.22" width="0.1524" layer="91"/>
-<pinref part="IC1" gate="G$1" pin="IO_14"/>
-<wire x1="248.92" y1="109.22" x2="261.62" y2="109.22" width="0.1524" layer="91"/>
-</segment>
-</net>
 <net name="N$64" class="0">
 <segment>
@@
 <label x="231.14" y="139.7" size="1.27" layer="95" rot="MR0" xref="yes"/>
 <pinref part="IC1" gate="G$1" pin="IO_3"/>
+</segment>
+</net>
+<net name="N$54" class="0">
+<segment>
+<pinref part="U4" gate="U$1" pin="OUT"/>
+<pinref part="C2" gate="CE" pin="1"/>
+<wire x1="78.74" y1="106.68" x2="64.77" y2="106.68" width="0.15" layer="91"/>
 </segment>
 </net>
@@
 analog and main digital supplies</text>
 <text x="238.76" y="177.8" size="2.54" layer="97">DC BLOCKING CAP?</text>
+<text x="88.9" y="129.54" size="1.778" layer="97">Test point only</text>
+<text x="88.9" y="177.8" size="1.778" layer="97">Test point only</text>
 </plain>
 <instances>
@@
 <instance part="GND49" gate="G1" x="142.24" y="198.12"/>
 <instance part="GND50" gate="G1" x="149.86" y="198.12" rot="MR0"/>
+<instance part="C82" gate="CE" x="119.38" y="137.16" rot="R180"/>
+<instance part="GND51" gate="G1" x="119.38" y="134.62"/>
 </instances>
 <busses>
@@
 <pinref part="GND50" gate="G1" pin="GND"/>
 </segment>
-</net>
-<net name="STQ-RF" class="0">
+<segment>
+<pinref part="C82" gate="CE" pin="1"/>
+<pinref part="GND51" gate="G1" pin="GND"/>
+</segment>
+</net>
+<net name="STQ-RF" class="2">
 <segment>
 <pinref part="U9" gate="G$1" pin="RFIN"/>
@@
 <wire x1="71.12" y1="139.7" x2="71.12" y2="142.24" width="0.1524" layer="91"/>
 <junction x="71.12" y="142.24"/>
-</segment>
-</net>
+<pinref part="C82" gate="CE" pin="2"/>
+<junction x="119.38" y="142.24"/>
+</segment>
+</net>

Commit message: Couldn't help myself; wired all the things. Left to do: clean-up, mostly. Verify CPLD pins, verify MAX connections and SkyTraq connections, design review, etc.
Connections:
- net N$43 renamed VCAP_1
- net N$45 renamed VCAP_2
- net N$9 renamed BOOT0
- new net N$9: IC1.IO_22
- net N$64: now also IC1.IO_5; no longer IC1.IO_13
- net Q0: now also IC1.IO_7; no longer IC1.IO_11
- net Q1: now also IC1.IO_6; no longer IC1.IO_12
- net STM_SPI1_MOSI: now also IC1.IO_13; no longer IC1.IO_2
- net STM_SPI1_NSS: now also IC1.IO_12; no longer IC1.IO_3
- net STM_SPI1_SCK: now also IC1.IO_11; no longer IC1.IO_1
Other:
- moved on the sheet: C71, C72, C73, C74, IC1, JP1
