File: v3-gps.sch (EAGLE design)
At the start: 182 parts, among them IC1 XC2C32A_VQ44_2, J1 1.27MM-SWD-CONNECTOR, J2 CON_SMA-ENDFIRE_EMERSON_EMERS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, J3 ROCKETNET-CONNECTOR-16M, J4 ZX62D-B-5P8, J7 CON_HIROSE_DM3D(MICROSD), Q1 NTR4101P, T1 ALT4532, T2 ALT4532, U1 MAX2769, U10 BP2G+, U11 MAX8510EXK29+T, U12 AVAGO-ALM-GPXX, U2 STM32F4V_100PIN_GPSBOARD, U3 KSZ8081, U4 7Q-16.368MBG-T, U6 MAX8510EXK29+T, U7 MAX8510EXK29+T, U8 LMZ12001, U9 VENUS638FLPX-L, X1 25 MHz

Commit message: More tweaks, notes, board now almost done. Still to do: 42 MHz clock, double check power plane routing, 16MHz clock cleanup.
Parts:
- added R26: 10k, rcl_custom:R-US_0402-C-NOSILK
- C71, C72, C73, C74: value 100p -> 100n
Connections:
- net N$64 renamed MAX-CLKOUT
- net AGND: now also U12.GND
- net GND: now also R26.1
- net N$9: now also IC1.IN_32, R26.2; no longer IC1.IO_22
Other:
- note added: "MISSING HIGH SPEED CLOCK (50 Mhz or 42 MHz or whatever)!!!!!"
- moved on the sheet: C71, C72, C73, C74, LED3, R38, R39, R40

Commit message: Done! Removed power split plane because that was stupid on further reflection, added clock comparator, cleaned up ERCs and DRCs.
Parts:
- added C83, C84: 100n, rcl_custom:C-EU0402-C-NOSILK
- added R27: 10k, rcl_custom:R-US_0402-C-NOSILK
- added U5: LT1719S6, ic-comparator-linear-lt1719:IC_COMP_W_SDSOT23-6
- U2: value STM32F4V_100PIN_GPSBOARD -> STM32F407VG
Connections:
- net ANTFLAG renamed MAX_ANTFLAG
- net DEBUG-PHY-MODWIRE renamed ETH_DEBUG
- net EPHY_NRST renamed ETH_PHY_NRST
- net LD renamed MAX_LD
- net MAX_CFG_MOSI renamed MAX_CFG_SPI2_MOSI
- net MAX_CFG_SCLK renamed MAX_CFG_SPI2_SCLK
- net MCO1-ETH-CLK renamed ETH_MCO1_CLK
- net N$11 renamed RGB-B
- net N$34 renamed RGB-R
- net N$49 renamed LED4
- net N$50 renamed LED5
- net N$9 renamed CPLD_IN_ONLY
- net OTG_FS_DM renamed USB_FS_DM
- net OTG_FS_DP renamed USB_FS_DP
- net OTG_FS_VBUS renamed USB_FS_VBUS
- net PE0 renamed SDIO_PWR
- net STM_SPI1_SCK renamed MAX_OUT_SPI1_SCK
- removed net 3.3VD1: LED2.C, U2.PD8
- removed net STM_SPI1_MOSI: IC1.IO_13, U2.PB5
- removed net STM_SPI1_NSS: IC1.IO_12, U2.PA4
- new net MAX_OUT_SPI1_MOSI: IC1.IO_14, U2.PB5
- new net MAX_OUT_SPI1_NSS: IC1.IO_13, U2.PA4
- new net MAX_OUT_SPI_CLK: IC1.IO_12, U2.PB14
- new net N$43: C84.1, R27.1, U5A.-IN
- new net N$45: R27.2, U1.CLKOUT, U5A.+IN
- new net RGB-G: R39.2, U2.PD14
- net 3.3VD: now also C83.1, U5PWR.V+
- net GND: now also C83.2, C84.2, U5A.SD, U5PWR.V-
- net LED2: now also LED2.C, U2.PD8; no longer R39.2, U2.PD14
- net MAX-CLKOUT: now also U5A.OUT; no longer U1.CLKOUT
Other:
- note added: "(BOOT1)"
- note added: "(MCO1)"
- note added: "(MCO2)"
- note added: "TO SKYTRAQ GPS"
- note removed: "Clock to Eth PHY"
- note removed: "MISSING HIGH SPEED CLOCK (50 Mhz or 42 MHz or whatever)!!!!!"
- note removed: "STM32F407VG (LQFP100)"
- note removed: "clock cleanup"
- moved on the sheet: C10, C11, C20, C29, C30, C45, C46, C47, C48, C49, C50, C51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

Commit message: Forgot to add comparator library earlier. Added bzillions of test points, to CPLD and STM, for future mod wires :) Also left RF class isolate to 25 mils, forgot to reset that during the last commit. Nothing left as far as I can see.
Parts:
- added TP23, TP24, TP3, TP31, TP34, TP35, TP36, TP37, TP38, TP39, TP40, TP6, TP7: TEST-POINT15MIL-TEST-POINT, Tova:TEST-POINT15MIL-TEST-POINT
- TP1, TP10, TP11, TP12, TP13, TP14, TP15, TP17, TP18, TP19, TP20, TP21, TP22, TP25, TP26, TP27, TP28, TP29, TP30, TP32, TP33, TP8, TP9: value TEST-POINT -> TEST-POINT15MIL-TEST-POINT; device Tova:TEST-POINT -> Tova:TEST-POINT15MIL-TEST-POINT
Connections:
- net MAX_OUT_SPI1_MOSI renamed CPLD_OUT_SPI1_MOSI
- net MAX_OUT_SPI1_NSS renamed CPLD_OUT_SPI1_NSS
- net MAX_OUT_SPI1_SCK renamed CPLD_OUT_SPI1_SCK
- net MAX_OUT_SPI_CLK renamed CPLD_OUT_SPI_CLK
- new net CPLD_DEBUG: IC1.IO_15, U2.PD12
- new net N$11: IC1.IO_19, TP23.1
- new net N$34: IC1.IO_17, TP31.1
- new net N$49: IC1.IO_0, TP34.1
- new net N$50: TP35.1, U2.PD5
- new net N$55: TP36.1, U2.PD7
- new net N$56: TP37.1, U2.PD1
- new net N$59: TP38.1, U2.PB0
- new net N$60: TP39.1, U2.PE3
- new net N$61: TP40.1, U2.PE5
- new net N$9: IC1.IO_21, TP24.1
- net GND: now also TP3.1, TP6.1, TP7.1
Other:
- note added: "COVERED SHIELD"

Commit message: Added part numbers to some of the odder components. Found the supercap is no longer made, so switched it to an instock item. Also checked on other components, like the LNA and splitter. Cleaned up schematic notes, added comments, added stiching around RF lines (not necessary, but yay OCD) and ran ERC and DRCs again.
Parts:
- removed C66: (no value), SparkFun-Passives:CAP_POLEN_J2
- removed TP37: TEST-POINT15MIL-TEST-POINT, Tova:TEST-POINT15MIL-TEST-POINT
- added C85: DSK-3R3H334T-HL, cap-elna-ds:CAP-ELNA-DS
- LED3: value (none) -> SMLV56RGB1W1
- U12: value AVAGO-ALM-GPXX -> ALM-GP002
- U8: value LMZ12001 -> LMZ12001TZ-ADJ/NOPB
Connections:
- removed net N$56: TP37.1, U2.PD1
- net GND: now also C85.-; no longer C66.-
- net STQ-VBAT: now also C85.+; no longer C66.+
Other:
- note added: "2.85V analog supply for MAX2769"
- note added: "2.85V digital supply for MAX2769"
- note added: "Fsw = 1 MHz"
- note added: "GPS LNA +19 dB, NF = 1.66 dB"
- note added: "Low noise LDO supplies for RF ICs"
- note added: "Mini-Circuits L band Splitter"
- note added: "Power from USB port for debugging"
- note added: "Soldered down RF shield with cap"
- note added: "SuperCap!"
- note removed: "2.85V Analog and Digital to MAX2769 GPS Receiver"
- note removed: "ASSUME WE CAN USE CLKOUT AND NOT TCXO OUT?"
- note removed: "Aux supply from USB debug"
- note removed: "CHECK RFIN WITH NO INDUCTIVE PULLUP"
- note removed: "COVERED SHIELD"
- note removed: "DC BLOCKING CAP?"
- note removed: "DOUBLE CHECK THIS PACKAGE"
- note removed: "PB10: SPI2_SCK / AF=5"
- note removed: "Splitter"
- note removed: "SuperCap"
- note removed: "THIS SHOULD BE AGND?!?!"
- note removed: "TODO: WHAT DO WE DO WITH CLKOUT?"
- note removed: "WHERE SHOULD WE CONNECT GND/AGND"
- moved on the sheet: C1, C56, C67, C68, C69, C70, C75, C76, C77, C78, C81, J2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

Commit message: So many little tweaks: updated ground planes, created BOM and then found out that everything doesn't exist anymore, so found new part numbers and in some cases (like the supercap) found new parts, arranged TNAMES, stitched RF lines, updated values for LED Rs, and more that I've forgotten already.
Parts:
- C19, C79: device rcl_custom:C-EU0402-C-NOSILK -> rcl_custom:C-EU0603-C-NOSILK
- C62: value 100n 50V -> 1n 2kv
- R12: value 1.5k -> 10k
- R14, R16, R20: value 1k -> 3.32k
- R38: value 400 -> 3.32k
- R39: value 110 -> 3.32k
- R40: value 900 -> 3.32k
- TP16: value (none) -> TPTP06R; device apdm:PAD+X-0.7 -> testpad:TPTP06R
- U1: value MAX2769 -> MAX2769ETI+
- U14: value MIC5025-1.8V -> MIC5319-1.8V
- renumbered IC1 to U13, VR1 to U14
Connections:
- net CPLD_OUT_SPI_CLK renamed CPLD_OUT_SPI_CLK_SRC
- net N$22 renamed LED/GPIO
- net N$25 renamed RTC
- net N$2: now also TP16.TP; no longer TP16.P
Other:
- moved on the sheet: C23, C36, C62

Commit message: OK now it's really done. tnames cleaned up more, ERC and DRC gone over, BOM updated and price calculated, found lack of stock on certain items, etc.
Other:
- note added: "115k UART"
- note added: "42 Mbps SPI"
- note added: "SkyTraq Venus638 GPS"
- note added: "Xylinx CoolRunner2 CPLD"
- note removed: "25 Mbps SPI"
- note removed: "SkyTraq GPS"
- note removed: "UART"
- note removed: "Xylinx CoolRunner2"

Commit message: Added 1.8V library, cleaned up power layer after seeing gerbers, added more comments on schematic after viewing PDF, and commited both for those folks without EAGLE.
Connections:
- net V18 renamed 1.8V
Other:
- note added: ""RocketNet" Power + Ethernet (not PoE!) distribution bus"
- note added: "0.8V clipped sign"
- note added: "1.8V core and 2.85V low noise analog supplies"
- note added: "1.8V internal supply For CPLD"
- note added: "10 - 20 V system power"
- note added: "16.384 MHz TCXO"
- note added: "4 bits I/Q data @ 4.096 Msps"
- note added: "4.5V (Vusb) to 20V (Shore power) Power in from RocketNet Connector"
- note added: "42 Mbps SPI to STM32"
- note added: "Block Diagram"
- note added: "Ethernet PHY + RocketNet"
- note added: "From passive -8 dBi cylindrical linear patch antenna"
- note added: "JTAG Programming header"
- note added: "LMZ12001TZ 3.3V SPS"
- note added: "MAX2769 + CPLD interface"
- note added: "MAX2769 SPI CONFIG port"
- note added: "Microcontroller"
- note added: "NMEA / Binary UART to STM32"
- note added: "Power Supplies"
- note added: "RF front end"
- note added: "SMA and coax to to L1 band linearly polarized "wrap around" cylindrical patch antennas on rocket aeroshell (-8 dBi typical)."
- note added: "SPI reference clock from STM32"
- note added: "STM32 RMII Interface"
- note added: "SkyTraq VENUS638 GPS"
- note removed: "1.85V internal supply For CPLD"
- note removed: "4.5 - 26 Vin"
- note removed: "MAX2769 SPI CONFIG PORT"
- note removed: "Test point only"
- moved on the sheet: C12, C13, C14, C15, C16, C17, C18, C19, C2, C22, C24, C3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

Commit message: Widended interface between digital and RF sections, added spacing to high speed MAX outputs, Added THads for scope ground clips and silk area for board #. Added GPS_RESET, and cleaned up STM scehamtic a bit.
Connections:
- net N$45 renamed MAX_CLK_OUT
- net VDD_1.2_ETH_SUPP renamed VDD_1.2
- new net CPLD_RESET: U13.IO_30, U2.PA10
Other:
- note added: "16.368 MHz TCXO"
- note added: "4 bits I/Q data @ 4.092 Msps"
- note added: "Fsw = 410 kHz"
- note added: "SAW + LNA"
- note removed: "16.384 MHz TCXO"
- note removed: "4 bits I/Q data @ 4.096 Msps"
- note removed: "Don't need MISO!"
- note removed: "FROM MAX2769"
- note removed: "Fsw = 1 MHz"
- note removed: "LNA"
