File: v3-gps.sch (EAGLE design)
At the start: 199 parts, among them J1 1.27MM-SWD-CONNECTOR, J2 CON_SMA-ENDFIRE_EMERSON_EMERS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, J3 ROCKETNET-CONNECTOR-16M, J4 ZX62D-B-5P8, J7 CON_HIROSE_DM3D(MICROSD), Q1 NTR4101P, T1 ALT4532, T2 ALT4532, U1 MAX2769ETI+, U10 BP2G+, U11 MAX8510EXK29+T, U12 ALM-GP002, U13 XC2C32A_VQ44_2, U14 MIC5319-1.8V, U2 STM32F407VG, U3 KSZ8081, U4 7Q-16.368MBG-T, U5 LT1719S6, U6 MAX8510EXK29+T, U7 MAX8510EXK29+T, U8 LMZ12001TZ-ADJ/NOPB, U9 VENUS638FLPX-L, X1 25 MHz

Commit message: Added Xilinx docs, and changed the SAW/LNA to the *correct* part number
Parts:
- U12: value ALM-GP002 -> ALM-GP003
Changed lines of the file:
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@@
 <part name="GND49" library="supply" deviceset="GND" device=""/>
 <part name="GND50" library="supply" deviceset="GND" device=""/>
-<part name="U12" library="ic-lna-ALM-GPxx-Avago" deviceset="AVAGO-ALM-GPXX" device="" value="ALM-GP002"/>
+<part name="U12" library="ic-lna-ALM-GPxx-Avago" deviceset="AVAGO-ALM-GPXX" device="" value="ALM-GP003"/>
 <part name="C1" library="rcl_custom" deviceset="C-EU" device="0402-C-NOSILK" value="330p"/>
 <part name="AGND24" library="supply1" deviceset="AGND" device=""/>

Commit message: Updated Schematic and BOM with problems, wrong values, etc.
Parts:
- C76: value 1u -> 2.2u
- C77: value 10n -> 100n
- R21: value 10k -> 33k
- R24: value 10k -> 1k
- U13: value XC2C32A_VQ44_2 -> XC2C64A-5VQG44C
- U9: value VENUS638FLPX-L -> VENUS838FLPX-L
Changed lines of the file:
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@@
 <?xml version="1.0" encoding="utf-8"?>
 <!DOCTYPE eagle SYSTEM "eagle.dtd">
-<eagle version="7.1.0">
+<eagle version="7.3.0">
 <drawing>
 <settings>
@@
 <part name="TP19" library="Tova" deviceset="TEST-POINT" device="15MIL-TEST-POINT" value="TEST-POINT15MIL-TEST-POINT"/>
 <part name="TP20" library="Tova" deviceset="TEST-POINT" device="15MIL-TEST-POINT" value="TEST-POINT15MIL-TEST-POINT"/>
-<part name="U9" library="SparkFun-RF" deviceset="VENUS638FLPX-L" device=""/>
+<part name="U9" library="SparkFun-RF" deviceset="VENUS638FLPX-L" device="" value="VENUS838FLPX-L"/>
 <part name="U10" library="minicircuits-splitter" deviceset="MINICIRCUITS-BP2G" device="" value="BP2G+"/>
 <part name="AGND1" library="supply1" deviceset="AGND" device=""/>
@@
 <part name="C22" library="rcl_custom" deviceset="C-EU" device="0402-C-NOSILK" value="100p"/>
 <part name="C24" library="rcl_custom" deviceset="C-EU" device="0402-C-NOSILK" value="100n"/>
-<part name="R21" library="rcl_custom" deviceset="R-US_" device="0402-C-NOSILK" value="10k"/>
+<part name="R21" library="rcl_custom" deviceset="R-US_" device="0402-C-NOSILK" value="33k"/>
 <part name="R22" library="rcl_custom" deviceset="R-US_" device="0402-C-NOSILK" value="10k"/>
 <part name="R23" library="rcl_custom" deviceset="R-US_" device="0402-C-NOSILK" value="1k"/>
@@
 <part name="TP30" library="Tova" deviceset="TEST-POINT" device="15MIL-TEST-POINT" value="TEST-POINT15MIL-TEST-POINT"/>
 <part name="D1" library="diode-0603" deviceset="DIODE-0603" device=""/>
-<part name="R24" library="rcl_custom" deviceset="R-US_" device="0402-C-NOSILK" value="10k"/>
+<part name="R24" library="rcl_custom" deviceset="R-US_" device="0402-C-NOSILK" value="1k"/>
 <part name="TP1" library="Tova" deviceset="TEST-POINT" device="15MIL-TEST-POINT" value="TEST-POINT15MIL-TEST-POINT"/>
 <part name="U11" library="SparkFun-PowerIC" deviceset="V_REG_LDO" device="SMD2" value="MAX8510EXK29+T"/>
@@
 <part name="AGND17" library="supply1" deviceset="AGND" device=""/>
 <part name="AGND18" library="supply1" deviceset="AGND" device=""/>
-<part name="U13" library="dp_devices" deviceset="XC2C32A_VQ44_2" device=""/>
+<part name="U13" library="dp_devices" deviceset="XC2C32A_VQ44_2" device="" value="XC2C64A-5VQG44C"/>
 <part name="U$10" library="SparkFun-Aesthetics" deviceset="3.3VD" device=""/>
 <part name="C71" library="rcl_custom" deviceset="C-EU" device="0402-C-NOSILK" value="100n"/>
@@
 <part name="C75" library="rcl_custom" deviceset="C-EU" device="0603-B-NOSILK" value="1u"/>
 <part name="GND41" library="SparkFun-Aesthetics" deviceset="GND" device=""/>
-<part name="C76" library="rcl_custom" deviceset="C-EU" device="0603-B-NOSILK" value="1u"/>
-<part name="C77" library="rcl_custom" deviceset="C-EU" device="0402-C-NOSILK" value="10n"/>
+<part name="C76" library="rcl_custom" deviceset="C-EU" device="0603-B-NOSILK" value="2.2u"/>
+<part name="C77" library="rcl_custom" deviceset="C-EU" device="0402-C-NOSILK" value="100n"/>
 <part name="GND42" library="SparkFun-Aesthetics" deviceset="GND" device=""/>
 <part name="C78" library="rcl_custom" deviceset="C-EU" device="0402-C-NOSILK" value="100n"/>
@@
 <part name="SUPPLY7" library="1.8V" deviceset="1.8V" device=""/>
 <part name="SUPPLY8" library="1.8V" deviceset="1.8V" device=""/>
+<part name="GND77" library="SparkFun-Aesthetics" deviceset="GND" device=""/>
 </parts>
 <sheets>
@@
 <text x="107.95" y="160.02" size="1.778" layer="97">Fsw = 410 kHz</text>
 <text x="327.66" y="26.67" size="5.08" layer="94">Power Supplies</text>
+<wire x1="290.83" y1="82.55" x2="293.37" y2="82.55" width="0.1524" layer="102"/>
+<wire x1="293.37" y1="82.55" x2="293.37" y2="71.12" width="0.1524" layer="102"/>
+<wire x1="289.56" y1="83.82" x2="292.1" y2="82.55" width="0.1524" layer="102"/>
+<wire x1="292.1" y1="83.82" x2="289.56" y2="82.55" width="0.1524" layer="102"/>
 </plain>
 <instances>
@@
 <instance part="FRAME3" gate="G$2" x="325.12" y="0"/>
 <instance part="SUPPLY8" gate="G$1" x="320.04" y="86.36"/>
+<instance part="GND77" gate="1" x="293.37" y="68.58" smashed="yes">
+<attribute name="VALUE" x="290.83" y="66.04" size="1.778" layer="96"/>
+</instance>
 </instances>
 <busses>
