File: GPS-USB_Front_End_Board/kicad_board_design/usb_gps.sch (KiCad schematic (older format))
At the start: 1 part, among them P1 CONN_02X12

Commit message: Completed, reviewed usb_gps board design.
Connections:
- net MAX_2769/+5V: now also P1.1 (P1); no longer P1.4 (P4)
- net MAX_2769/GND: now also P1.4 (P4); no longer P1.1 (P1)
Changed lines of the file:
@@
 LIBS:93LC46B-E_SN
 LIBS:OscillatorTaitien
+LIBS:maxim
+LIBS:MAX8510EXK21
+LIBS:LT1719
+LIBS:LT1719S6B
+LIBS:LT1719CS6TRPBF
 LIBS:usb_gps-cache
 EELAYER 25 0
@@
 F16 "GPIO2" I R 3600 5100 60
 F17 "GPIO3" I R 3600 5300 60
+F18 "VCC3V3" O R 3600 5425 60
 $EndSheet
 $Sheet
@@
 F14 "SHDN#" I L 7000 5100 60
 F15 "IDLE#" I L 7000 5300 60
+F16 "VCC3V3" I L 7000 5425 60
 $EndSheet
 $Comp
@@
 NoConn ~ 5500 3700
 Wire Wire Line
+	3600 3100 5000 3100
+Wire Wire Line
+	3600 3200 3950 3200
+Wire Wire Line
+	3600 3300 4050 3300
+Wire Wire Line
+	3600 3400 4150 3400
+Wire Wire Line
+	4150 3400 4150 3300
+Wire Wire Line
+	4150 3300 5000 3300
+Wire Wire Line
+	3600 3600 4250 3600
+Wire Wire Line
+	4250 3600 4250 3400
+Wire Wire Line
+	4250 3400 5000 3400
+Wire Wire Line
+	3600 3700 4350 3700
+Wire Wire Line
+	4350 3700 4350 3500
+Wire Wire Line
+	4350 3500 5000 3500
+Wire Wire Line
+	3600 4100 4450 4100
+Wire Wire Line
+	4450 4100 4450 3600
+Wire Wire Line
+	4450 3600 5000 3600
+Wire Wire Line
+	3600 4200 4550 4200
+Wire Wire Line
+	4550 4200 4550 3700
+Wire Wire Line
+	4550 3700 5000 3700
+Wire Wire Line
+	3600 4300 4650 4300
+Wire Wire Line
+	4650 4300 4650 3800
+Wire Wire Line
+	4650 3800 5000 3800
+Wire Wire Line
+	3600 4400 4750 4400
+Wire Wire Line
+	4750 4400 4750 3900
+Wire Wire Line
+	4750 3900 5000 3900
+Wire Wire Line
+	7000 3100 6750 3100
+Wire Wire Line
+	6750 3100 6750 3000
+Wire Wire Line
+	6750 3000 5500 3000
+Wire Wire Line
+	7000 3200 6650 3200
+Wire Wire Line
+	6650 3200 6650 3100
+Wire Wire Line
+	6650 3100 5500 3100
+Wire Wire Line
+	7000 3300 6550 3300
+Wire Wire Line
+	6550 3300 6550 3200
+Wire Wire Line
+	6550 3200 5500 3200
+Wire Wire Line
+	7000 3400 6450 3400
+Wire Wire Line
+	6450 3400 6450 3300
+Wire Wire Line
+	6450 3300 5500 3300
+Wire Wire Line
+	7000 3700 6250 3700
+Wire Wire Line
+	6250 3700 6250 3500
+Wire Wire Line
+	6250 3500 5500 3500
+Wire Wire Line
+	7000 4100 6150 4100
+Wire Wire Line
+	6150 4100 6150 3600
+Wire Wire Line
+	6150 3600 5500 3600
+Wire Wire Line
+	7000 4300 5950 4300
+Wire Wire Line
+	5950 4300 5950 3800
+Wire Wire Line
+	5950 3800 5500 3800
+Wire Wire Line
+	7000 4400 5850 4400
+Wire Wire Line
+	5850 4400 5850 3900
+Wire Wire Line
+	5850 3900 5500 3900
+Wire Wire Line
+	3600 4700 7000 4700
+Wire Wire Line
+	3600 4900 7000 4900
+Wire Wire Line
+	3600 5100 7000 5100
+Wire Wire Line
+	3600 5300 7000 5300
+Wire Wire Line
+	4050 3300 4050 3200
+Wire Wire Line
+	4050 3200 5000 3200
+Wire Wire Line
+	3950 3200 3950 3000
+Wire Wire Line
+	3950 3000 5000 3000
+Wire Wire Line
 	3600 2900 5000 2900
 Wire Wire Line
-	5000 2800 4900 2800
-Wire Wire Line
-	4900 2800 4900 2900
-Connection ~ 4900 2900
-Wire Wire Line
-	3600 2800 4700 2800
-Wire Wire Line
-	4700 2800 4700 2550
-Wire Wire Line
-	4700 2550 5700 2550
-Wire Wire Line
-	5700 2550 5700 2900
-Wire Wire Line
-	5700 2900 5500 2900
+	5500 2900 7000 2900
+Wire Wire Line
+	4700 2900 4700 2450
+Wire Wire Line
+	4700 2450 5800 2450
+Wire Wire Line
+	5800 2450 5800 2900
+Connection ~ 5800 2900
+Connection ~ 4700 2900
+Wire Wire Line
+	3600 2800 5000 2800
 Wire Wire Line
 	5500 2800 7000 2800
+Wire Wire Line
+	4800 2800 4800 2550
+Wire Wire Line
+	4800 2550 5700 2550
+Wire Wire Line
+	5700 2550 5700 2800
 Connection ~ 5700 2800
-Wire Wire Line
-	3600 3100 5000 3100
-Wire Wire Line
-	3600 3200 3950 3200
-Wire Wire Line
-	3600 3300 4050 3300
-Wire Wire Line
-	3600 3400 4150 3400
-Wire Wire Line
-	4150 3400 4150 3300
-Wire Wire Line
-	4150 3300 5000 3300
-Wire Wire Line
-	3600 3600 4250 3600
-Wire Wire Line
-	4250 3600 4250 3400
-Wire Wire Line
-	4250 3400 5000 3400
-Wire Wire Line
-	3600 3700 4350 3700
-Wire Wire Line
-	4350 3700 4350 3500
-Wire Wire Line
-	4350 3500 5000 3500
-Wire Wire Line
-	3600 4100 4450 4100
-Wire Wire Line
-	4450 4100 4450 3600
-Wire Wire Line
-	4450 3600 5000 3600
-Wire Wire Line
-	3600 4200 4550 4200
-Wire Wire Line
-	4550 4200 4550 3700
-Wire Wire Line
-	4550 3700 5000 3700
-Wire Wire Line
-	3600 4300 4650 4300
-Wire Wire Line
-	4650 4300 4650 3800
-Wire Wire Line
-	4650 3800 5000 3800
-Wire Wire Line
-	3600 4400 4750 4400
-Wire Wire Line
-	4750 4400 4750 3900
-Wire Wire Line
-	4750 3900 5000 3900
-Wire Wire Line
-	4500 2900 4500 2450
-Wire Wire Line
-	4500 2450 5850 2450
-Wire Wire Line
-	5850 2450 5850 2900
-Wire Wire Line
-	5850 2900 7000 2900
-Connection ~ 4500 2900
-Wire Wire Line
-	7000 3100 6750 3100
-Wire Wire Line
-	6750 3100 6750 3000
-Wire Wire Line
-	6750 3000 5500 3000
-Wire Wire Line
-	7000 3200 6650 3200
-Wire Wire Line
-	6650 3200 6650 3100
-Wire Wire Line
-	6650 3100 5500 3100
-Wire Wire Line
-	7000 3300 6550 3300
-Wire Wire Line
-	6550 3300 6550 3200
-Wire Wire Line
-	6550 3200 5500 3200
-Wire Wire Line
-	7000 3400 6450 3400
-Wire Wire Line
-	6450 3400 6450 3300
-Wire Wire Line
-	6450 3300 5500 3300
-Wire Wire Line
-	7000 3700 6250 3700
-Wire Wire Line
-	6250 3700 6250 3500
-Wire Wire Line
-	6250 3500 5500 3500
-Wire Wire Line
-	7000 4100 6150 4100
-Wire Wire Line
-	6150 4100 6150 3600
-Wire Wire Line
-	6150 3600 5500 3600
-Wire Wire Line
-	7000 4300 5950 4300
-Wire Wire Line
-	5950 4300 5950 3800
-Wire Wire Line
-	5950 3800 5500 3800
-Wire Wire Line
-	7000 4400 5850 4400
-Wire Wire Line
-	5850 4400 5850 3900
-Wire Wire Line
-	5850 3900 5500 3900
-Wire Wire Line
-	3600 4700 7000 4700
-Wire Wire Line
-	3600 4900 7000 4900
-Wire Wire Line
-	3600 5100 7000 5100
-Wire Wire Line
-	3600 5300 7000 5300
-Wire Wire Line
-	4050 3300 4050 3200
-Wire Wire Line
-	4050 3200 5000 3200
-Wire Wire Line
-	3950 3200 3950 3000
-Wire Wire Line
-	3950 3000 5000 3000
+Connection ~ 4800 2800
+Wire Wire Line
+	3600 5425 7000 5425
 $EndSCHEMATC
