File: GPS-USB_Front_End_Board/kicad_board_design/usb_gps.kicad_pcb (KiCad board)
At the start: 4 copper layers, 99.1 x 53.3 mm, 85 parts, among them J1 10118192-0001LF, J2 Edge Launch SMA, J3 Edge Launch SMA, P1 CONN_02X12, U1 93LCxxB, U2 FT2232HL-REEL, U3 L4931ABD33-TR, U4 SAWTEK-855969, U5 AP131-30, U6 MAX2769CETI+, U7 SAWTEK-855969, X1 TCXO3, Y1 Crystal_GND24

Commit message: Completed, reviewed usb_gps board design.
Parts:
- removed F1: Polyfuse_Small, fuse:0805L_Littelfuse
- removed FB2: BLM18PG471SN1D, digikey-footprints:0603
- removed G***: LOGO, logo:logo_combined_components
- removed J2: Edge Launch SMA, digikey-footprints:RF_SMA_Receptical_Vertical_CONSMA001-SMD-G
- removed L1: NC, Choke_SMD:Choke_SMD_1206_Handsoldering
- removed L2: 6.2nH, Capacitors_SMD:C_0603_HandSoldering
- removed L3: 4.3nH, Capacitors_SMD:C_0402
- removed REF1, REF2, REF3, REF4: MountingHole_2.5mm, Mounting_Holes:MountingHole_2.5mm
- added C36: .1uF, Capacitors_SMD:C_0402, F.Cu at (133.2, 66.7)
- added C37: 100nF, Capacitors_SMD:C_0402, F.Cu at (117.3, 68.7)
- added C38: .1uF, Capacitors_SMD:C_0402, F.Cu at (124.7, 68.3)
- added R19: 0, Resistors_SMD:R_0603_HandSoldering, F.Cu at (121.7, 74.5)
- added R20: NC, Resistors_SMD:R_0603_HandSoldering, F.Cu at (117.9, 72.0)
- added U8: LT1719S6 -- Not Populated, rf:TSOT-23_S6, F.Cu at (122.4, 71.4)
- added W1: EECS, Measurement_Points:Measurement_Point_Round-TH_Small, F.Cu at (87.0, 88.3)
- added W2: D0, Measurement_Points:Measurement_Point_Round-TH_Small, F.Cu at (87.0, 95.9)
- added W3: D1, Measurement_Points:Measurement_Point_Round-TH_Small, F.Cu at (87.0, 93.3)
- added W4: PWREN, Measurement_Points:Measurement_Point_Round-TH_Small, F.Cu at (99.7, 97.2)
- added W5: SUSPEND, Measurement_Points:Measurement_Point_Round-TH_Small, F.Cu at (119.1, 80.9)
- added W6: EECLK, Measurement_Points:Measurement_Point_Round-TH_Small, F.Cu at (87.0, 90.8)
- C10: value NC -> 10uF; footprint Capacitors_SMD:C_0805_HandSoldering -> Capacitors_SMD:C_0603_HandSoldering
- C12: value 33pF -> 1uF
- C17: value 100pF -> 10nF; footprint Capacitors_SMD:C_0805_HandSoldering -> Capacitors_SMD:C_0402
- C24: value 10uF -> 10nF; footprint Capacitors_SMD:C_0805_HandSoldering -> Capacitors_SMD:C_0402
- C9: value NC -> 100 nF; footprint Capacitors_SMD:C_0805_HandSoldering -> Capacitors_SMD:C_0402
- J1: value 10118192-0001LF -> Micro-USB Connector
- TP2, TP3, TP4, TP5, TP6: footprint Measurement_Points:Test_Point -> Measurement_Points:Measurement_Point_Round-TH_Small
- U3: value L4931ABD33-TR -> L4931 LDO
- U4: value SAWTEK-855969 -> MAX8510; footprint rf:Sawtek_855969 -> rf:21-0076E
- U5: value AP131-30 -> MAX8510; footprint TO_SOT_Packages_SMD:SOT-23-5 -> rf:21-0076E
- X1: value TCXO3 -> 13.368MHz TCXO; footprint oscillator:CTS_405_xtal -> rf:TCXO_Taitien
- Y1: value Crystal_GND24 -> 12MHz Crystal
- moved C9 62.1 mm to (91.6, 66.3)
- moved C10 57.8 mm to (102.6, 68.3), turned to 270 degrees
- moved R15 26.5 mm to (162.0, 98.5), turned to 270 degrees
- moved R16 26.2 mm to (165.8, 96.4), turned to 270 degrees
- moved TP5 24.6 mm to (120.4, 66.2)
- moved C4 22.5 mm to (99.7, 102.2), turned to 180 degrees
- moved C26 18.2 mm to (160.9, 78.4)
- moved R10 15.8 mm to (135.8, 100.9)
- moved TP4 14.2 mm to (96.5, 65.0)
- moved TP6 11.9 mm to (107.3, 109.2)
- moved C24 9.03 mm to (131.4, 66.7)
- moved C33 8.89 mm to (104.1, 99.1)
- moved U5 7.30 mm to (128.8, 66.7)
- moved R9 6.35 mm to (135.9, 110.4)
- moved TP1 5.25 mm to (135.2, 71.3)
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Connections:
- C1 pad 1: /USB_FT2232/VCC3V3 -> /MAX_2769/VCC3V3
- C10 pad 1: /MAX_2769/VCC3V -> /MAX_2769/+5V
- C11 pad 1: /MAX_2769/VCC3V -> /MAX_2769/VCCA
- C12 pad 1: Net-(C12-Pad1) -> /MAX_2769/+5V
- C12 pad 2: Net-(C12-Pad2) -> GND
- C13 pad 1: /MAX_2769/VCC3V -> /MAX_2769/VCCA
- C14 pad 1: /MAX_2769/VCC3V -> /MAX_2769/VCCA
- C15 pad 1: /MAX_2769/VCC3V -> /MAX_2769/VCCD
- C16 pad 1: /MAX_2769/VCC3V -> /MAX_2769/VCCA
- C17 pad 1: Net-(C12-Pad2) -> /MAX_2769/VCCA
- C19 pad 1: /MAX_2769/VCC3V -> /MAX_2769/VCCA
- C2 pad 1: /USB_FT2232/VCC3V3 -> /MAX_2769/VCC3V3
- C21 pad 1: /MAX_2769/VCC3V -> /MAX_2769/VCCA
- C22 pad 1: /MAX_2769/VCC3V -> /MAX_2769/VCCA
- C23 pad 1: Net-(C23-Pad1) -> /MAX_2769/VCCA
- C24 pad 1: /MAX_2769/VCC3V -> /MAX_2769/VCCD
- C24 pad 2: GND -> Net-(C24-Pad2)
- C26 pad 2: /MAX_2769/CLKOUT -> Net-(C26-Pad2)
- C34 pad 1: /USB_FT2232/VCC3V3 -> /MAX_2769/VCC3V3
- C35 pad 1: /USB_FT2232/VCC3V3 -> /MAX_2769/VCC3V3
- C7 pad 1: /USB_FT2232/VCC3V3 -> /MAX_2769/VCC3V3
- C9 pad 1: Net-(C12-Pad1) -> Net-(C9-Pad1)
- D1 pad 4: /USB_FT2232/Data- -> /USB_FT2232/Data+
- D1 pad 6: /USB_FT2232/Data+ -> /USB_FT2232/Data-
- FB1 pad 2: Net-(F1-Pad1) -> /USB_FT2232/VBUS
- J1 pad 2: Net-(D1-Pad3) -> Net-(D1-Pad1)
- J1 pad 3: Net-(D1-Pad1) -> Net-(D1-Pad3)
- J1 pad 6: Net-(J1-Pad6) -> Net-(C9-Pad1)
- P1 pad 1: GND -> /MAX_2769/+5V
- P1 pad 4: /MAX_2769/+5V -> GND
- R1 pad 1: /USB_FT2232/VCC3V3 -> /MAX_2769/VCC3V3
- R11 pad 2: /MAX_2769/VCC3V -> /MAX_2769/VCCA
- R14 pad 1: /MAX_2769/WR# -> /MAX_2769/CLKOUT
- R14 pad 2: /MAX_2769/CLKOUT -> /MAX_2769/WR#
- R15 pad 1: /MAX_2769/D3 -> /MAX_2769/Q1
- R15 pad 2: /MAX_2769/Q1 -> /MAX_2769/D3
- R16 pad 1: /MAX_2769/D2 -> /MAX_2769/Q0
- R16 pad 2: /MAX_2769/Q0 -> /MAX_2769/D2
- R17 pad 1: /MAX_2769/D1 -> /MAX_2769/I0
- R17 pad 2: /MAX_2769/I0 -> /MAX_2769/D1
- R18 pad 1: /MAX_2769/D0 -> /MAX_2769/I1
- R18 pad 2: /MAX_2769/I1 -> /MAX_2769/D0
- R3 pad 1: /USB_FT2232/VCC3V3 -> /MAX_2769/VCC3V3
- R4 pad 1: /USB_FT2232/VCC3V3 -> /MAX_2769/VCC3V3
- R5 pad 1: /USB_FT2232/VCC3V3 -> /MAX_2769/VCC3V3
- R7 pad 2: /MAX_2769/VCC3V -> /MAX_2769/VCCA
- TP5 pad 1: /USB_FT2232/VCC3V3 -> /MAX_2769/VCC3V3
- U1 pad 8: /USB_FT2232/VCC3V3 -> /MAX_2769/VCC3V3
- U2 pad 20: /USB_FT2232/VCC3V3 -> /MAX_2769/VCC3V3
- U2 pad 31: /USB_FT2232/VCC3V3 -> /MAX_2769/VCC3V3
- U2 pad 4: /USB_FT2232/VCC3V3 -> /MAX_2769/VCC3V3
- U2 pad 42: /USB_FT2232/VCC3V3 -> /MAX_2769/VCC3V3
- U2 pad 50: /USB_FT2232/VCC3V3 -> /MAX_2769/VCC3V3
- U2 pad 56: /USB_FT2232/VCC3V3 -> /MAX_2769/VCC3V3
- U2 pad 9: /USB_FT2232/VCC3V3 -> /MAX_2769/VCC3V3
- U3 pad 1: Net-(FB2-Pad2) -> /MAX_2769/VCC3V3
- U4 pad 1: GND -> /MAX_2769/+5V
- U4 pad 2: Net-(C12-Pad2) -> GND
- U4 pad 3: GND -> /MAX_2769/+5V
- U4 pad 4: GND -> Net-(C17-Pad2)
- U4 pad 5: Net-(C17-Pad2) -> /MAX_2769/VCCA
- U5 pad 4: Net-(C23-Pad1) -> Net-(C24-Pad2)
- U5 pad 5: /MAX_2769/VCC3V -> /MAX_2769/VCCD
- U6 pad 11: /MAX_2769/VCC3V -> /MAX_2769/VCCA
- U6 pad 13: /MAX_2769/VCC3V -> /MAX_2769/VCCA
- U6 pad 14: /MAX_2769/VCC3V -> /MAX_2769/VCCA
- U6 pad 19: /MAX_2769/VCC3V -> /MAX_2769/VCCD
- U6 pad 23: /MAX_2769/VCC3V -> /MAX_2769/VCCA
- U6 pad 27: /MAX_2769/LNA1 -> Net-(U6-Pad27)
- U6 pad 4: /MAX_2769/VCC3V -> /MAX_2769/VCCA
- X1 pad 4: /MAX_2769/VCC3V -> /MAX_2769/VCCA
Routing:
- net /MAX_2769/VCC3V: track 363.5 -> 0.00 mm, vias 16 -> 0
- net /USB_FT2232/VCC3V3: track 77.9 -> 0.00 mm, vias 18 -> 0
- net /USB_FT2232/GPIO3: track 41.0 -> 110.5 mm, vias 2 -> 4
- net /MAX_2769/VCCD: track 0.00 -> 65.0 mm, vias 0 -> 2
- net Net-(C26-Pad2): track 0.00 -> 48.7 mm
- net /MAX_2769/LNA1: track 47.2 -> 0.00 mm
- net /MAX_2769/VCCA: track 0.00 -> 43.8 mm, vias 0 -> 20
- net GND: track 145.8 -> 102.1 mm, vias 47 -> 26
- net /MAX_2769/D2: track 10.8 -> 52.2 mm, vias 0 -> 1
- net /MAX_2769/VCC3V3: track 0.00 -> 35.9 mm, vias 0 -> 21
- net Net-(C12-Pad1): track 28.3 -> 0.00 mm
- net /MAX_2769/D3: track 9.23 -> 33.7 mm, vias 0 -> 1
- net Net-(C12-Pad2): track 21.7 -> 0.00 mm
- net Net-(R6-Pad1): track 21.9 -> 43.5 mm, vias 0 -> 1
- net Net-(C9-Pad1): track 0.00 -> 21.4 mm
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- added copper zone on In2.Cu, net /MAX_2769/VCC3V3
- added copper zone on In2.Cu, net /MAX_2769/VCCA
- removed copper zone on In2.Cu, net /USB_FT2232/VCC3V3
- removed copper zone on In2.Cu, net GND
Other:
- net class Default: trace_width 0.127 -> 0.2032
- rule trace_min: 0.127 -> 0.2032

Commit message: Re-add the mounting holes.
Parts:
- added G***: LOGO, logo:logo_combined_components, F.Cu at (174.0, 101.6)
- added REF**: MountingHole_2.2mm_M2_Pad_Via, Mounting_Holes:MountingHole_2.2mm_M2_Pad_Via, F.Cu at (177.8, 64.8)
- added REF**: MountingHole_2.2mm_M2_Pad_Via, Mounting_Holes:MountingHole_2.2mm_M2_Pad_Via, F.Cu at (177.8, 110.5)
- added REF**: MountingHole_2.2mm_M2_Pad_Via, Mounting_Holes:MountingHole_2.2mm_M2_Pad_Via, F.Cu at (86.4, 110.5)
- added REF**: MountingHole_2.2mm_M2_Pad_Via, Mounting_Holes:MountingHole_2.2mm_M2_Pad_Via, F.Cu at (86.4, 64.8)
