File: GPS-USB_Front_End_Board/kicad_board_design/USB_FT2232.sch (KiCad schematic (older format))
At the start: 32 parts, among them J1 10118192-0001LF, U1 93LCxxB, U2 FT2232HL-REEL, U3 L4931ABD33-TR, Y1 Crystal_GND24

Commit message: Completed, reviewed usb_gps board design.
Parts:
- removed F1: Polyfuse_Small, fuse:0805L_Littelfuse, symbol Polyfuse_Small
- removed FB2: BLM18PG471SN1D, digikey-footprints:0603, symbol BLM18PG471SN1D
- added C10: 10uF, Capacitors_SMD:C_0603_HandSoldering, symbol C_Small
- added C9: 100 nF, Capacitors_SMD:C_0402, symbol C_Small
- added W1: EECS, Measurement_Points:Measurement_Point_Round-TH_Small, symbol TEST_1P
- added W2: D0, Measurement_Points:Measurement_Point_Round-TH_Small, symbol TEST_1P
- added W3: D1, Measurement_Points:Measurement_Point_Round-TH_Small, symbol TEST_1P
- added W4: PWREN, Measurement_Points:Measurement_Point_Round-TH_Small, symbol TEST_1P
- added W5: SUSPEND, Measurement_Points:Measurement_Point_Round-TH_Small, symbol TEST_1P
- added W6: EECLK, Measurement_Points:Measurement_Point_Round-TH_Small, symbol TEST_1P
- J1: value 10118192-0001LF -> Micro-USB Connector
- TP2, TP3, TP4, TP5, TP6: footprint Measurement_Points:Test_Point -> Measurement_Points:Measurement_Point_Round-TH_Small
- U3: value L4931ABD33-TR -> L4931 LDO
- Y1: value Crystal_GND24 -> 12MHz Crystal
Connections:
- net +5V: now also C10.1
- net Data+: now also D1.4; no longer D1.6
- net Data-: now also D1.6; no longer D1.4
- net EECLK: now also W6.1
- net EECS: now also W1.1
- net GND: now also C10.2, C9.2
- net VBUS: now also FB1.2
- net VCC3V3: now also U3.1 (VOUT)
- net at J1.2 (Data-): now also D1.1; no longer D1.3
- net at J1.3 (Data+): now also D1.3; no longer D1.1
- net at J1.6: now also C9.1
- net at U2.36 (SUSPEND): now also W5.1
- net at U2.60 (PWREN): now also W4.1
- net at R6.1, U1.3 (DI), U2.61 (EEDATA): now also W3.1
- net at R5.2, R6.2, U1.4 (DO): now also W2.1
- no-connect marks 25 -> 22
Other:
- note added: "Off-Sheet Signals\n"

Commit message: schematic cleanup
Parts:
- C1: MFR (none) -> Samsung; MPN (none) -> CL10B105KP8NNNC; SPN (none) -> 1276-1946-1-ND; SPR (none) -> Digikey; SPURL (none) -> -
- C10: MFR (none) -> Samsung; MPN (none) -> CL10B106MQ8NRNC; SPN (none) -> 1276-1948-1-ND; SPR (none) -> Digikey; SPURL (none) -> -
- C2, C33, C35, C6, C8, C9: MFR (none) -> TDK; MPN (none) -> CGA2B1X7R1C104K050BC; SPN (none) -> 445-5613-1-ND; SPR (none) -> Digikey; SPURL (none) -> -
- C3, C5: MFR (none) -> Kemet; MPN (none) -> C0805C100K5RAC7800; SPN (none) -> 399-17612-1-ND; SPR (none) -> Digikey; SPURL (none) -> -
- C34, C4: MFR (none) -> TDK; MPN (none) -> C2012X7R1C335K125AB; SPN (none) -> 445-7582-1-ND; SPR (none) -> Digikey; SPURL (none) -> -
- C7: MFR (none) -> TDK; MPN (none) -> C2012X7R1C225K125AB; SPN (none) -> 445-1420-1-ND; SPR (none) -> Digikey; SPURL (none) -> -
- D1: MFR (none) -> STMicro; SPN (none) -> 497-5235-1-ND USB; SPR (none) -> Digikey; SPURL (none) -> -
- FB1: MFR (none) -> Taiyo Yuden; MPN BLM18PG471SN1D -> BK0603HS330-T; SPN (none) -> 587-1828-1-ND; SPR (none) -> Digikey; SPURL (none) -> -
- J1: MFR (none) -> Amphenol; SPN (none) -> 609-4613-1-ND; SPR (none) -> Digikey; SPURL (none) -> -
- R1, R3, R4, R5: MFR (none) -> TE Connectivity; MPN (none) -> CRGH0805F10K; SPN (none) -> A126417DKR-ND; SPR (none) -> Digikey; SPURL (none) -> -
- R2: MFR (none) -> TE Connectivity; MPN (none) -> CPF0603B12KE1; SPN (none) -> A103037CT-ND; SPR (none) -> Digikey; SPURL (none) -> -
- R6: MFR (none) -> Yageo; MPN (none) -> AC0603FR-072KL; SPN (none) -> YAG3590CT-ND; SPR (none) -> Digikey; SPURL (none) -> -
- TP1, TP2, TP3, TP4, TP5, TP6, W1, W2, W3, W4, W5, W6: MFR (none) -> -; MPN (none) -> -; SPN (none) -> -; SPR (none) -> -; SPURL (none) -> -
- U1: MFR (none) -> MicroChip; MPN (none) -> 93LC46B-I/SN; SPN (none) -> 93LC46B-I/SN-ND; SPR (none) -> Digikey; SPURL (none) -> -
- U2: MFR (none) -> FTDI; SPN (none) -> 768-1024-1-ND; SPR (none) -> Digikey; SPURL (none) -> -
- U3: MFR (none) -> STMicro; SPN (none) -> 497-1155-1-ND; SPR (none) -> Digikey; SPURL (none) -> -
- Y1: MFR (none) -> CTS; MPN (none) -> 405C35E12M00000; SPN (none) -> CTX819DKR-ND; SPR (none) -> Digikey; SPURL (none) -> -
